File: Extruder.sch (KiCad schematic (older format))
At the start: 0 parts

Commit message: Add 3 axis and 2 extruders. Basic thermistor temperature sensing and MOSFET heaters in the extruders.
Parts:
- added J7: Probe, symbol Connector_Generic:Conn_02x01
- added J8: Extruder Heater, symbol Connector_Specialized:Screw_Terminal_01x02
Connections:
- new net Fimalent Detect/SENSOR: J7.2 (Pin_2)
- new net GND: J7.1 (Pin_1)
- new net Heating/HEATER: J8.2 (Pin_2)
- new net V_MOTORS: J8.1 (Pin_1)
Changed lines of the file:
@@
 $Descr A4 11693 8268
 encoding utf-8
-Sheet 6 6
+Sheet 25 29
 Title ""
 Date ""
@@
 Comment4 ""
 $EndDescr
+$Sheet
+S 2700 1950 950  1650
+U 5AD4B0F5
+F0 "Driver" 50
+F1 "MotorDriver_TMC2660.sch" 50
+F2 "V_IO" I R 3650 2100 50
+F3 "V_MOTORS" I R 3650 2300 50
+F4 "MOT1B" O L 2700 2150 50
+F5 "MOT1A" O L 2700 2050 50
+F6 "MOT2A" O L 2700 2250 50
+F7 "MOT2B" O L 2700 2350 50
+F8 "STEP" I L 2700 2600 50
+F9 "DIR" I L 2700 2700 50
+F10 "~CS" I L 2700 2850 50
+F11 "SCK" I L 2700 2950 50
+F12 "MOSI" I L 2700 3050 50
+F13 "MISO" O L 2700 3150 50
+F14 "~ENABLE" I L 2700 3300 50
+F15 "SG_TST" O L 2700 3450 50
+$EndSheet
+Text HLabel 2600 2600 0    50   Input ~ 0
+STEP
+Text HLabel 2600 2700 0    50   Input ~ 0
+DIR
+Text HLabel 2600 2850 0    50   Input ~ 0
+~CS
+Text HLabel 2600 2950 0    50   Input ~ 0
+SCK
+Text HLabel 2600 3050 0    50   Input ~ 0
+MOSI
+Text HLabel 2600 3150 0    50   Output ~ 0
+MISO
+Text HLabel 2600 3300 0    50   Input ~ 0
+~ENABLE
+Text HLabel 2600 3450 0    50   Output ~ 0
+SG_TST
+Text HLabel 4050 2100 2    50   Input ~ 0
+V_IO
+Text HLabel 4050 2300 2    50   Input ~ 0
+V_MOTORS
+Wire Wire Line
+	2700 2600 2600 2600
+Wire Wire Line
+	2700 2700 2600 2700
+Wire Wire Line
+	2700 2850 2600 2850
+Wire Wire Line
+	2700 2950 2600 2950
+Wire Wire Line
+	2700 3050 2600 3050
+Wire Wire Line
+	2700 3150 2600 3150
+Wire Wire Line
+	2700 3300 2600 3300
+Wire Wire Line
+	2700 3450 2600 3450
+$Sheet
+S 2700 3850 950  600
+U 5AD4BBBB
+F0 "Fimalent Detect" 50
+F1 "Endstop.sch" 50
+F2 "SENSOR" I L 2700 4000 50
+F3 "OUT" O L 2700 4250 50
+F4 "V_IO" I R 3650 3950 50
+$EndSheet
+Wire Wire Line
+	3650 3950 3750 3950
+Wire Wire Line
+	3750 3950 3750 2100
+Connection ~ 3750 2100
+Wire Wire Line
+	3750 2100 3650 2100
+Text HLabel 2600 4250 0    50   Output ~ 0
+FILAMENT
+Wire Wire Line
+	2600 4250 2700 4250
+$Comp
+L Connector_Generic:Conn_02x01 J7
+U 1 1 5AD4BF35
+P 2300 4000
+AR Path="/5AC337B6/5ACBE919/5AD4BF35" Ref="J7"  Part="1"
+AR Path="/5AC337B6/5AD9F95A/5AD4BF35" Ref="J15"  Part="1"
+F 0 "J15" H 2350 4217 50  0000 C CNN
+F 1 "Probe" H 2350 4126 50  0000 C CNN
+F 2 "" H 2300 4000 50  0001 C CNN
+F 3 "~" H 2300 4000 50  0001 C CNN
+	1    2300 4000
+	1    0    0    -1
+$EndComp
+Wire Wire Line
+	2600 4000 2700 4000
+$Comp
+L power:GND #PWR04
+U 1 1 5AD4C143
+P 2100 4100
+AR Path="/5AC337B6/5ACBE919/5AD4C143" Ref="#PWR04"  Part="1"
+AR Path="/5AC337B6/5AD9F95A/5AD4C143" Ref="#PWR043"  Part="1"
+F 0 "#PWR043" H 2100 3850 50  0001 C CNN
+F 1 "GND" H 2105 3927 50  0000 C CNN
+F 2 "" H 2100 4100 50  0001 C CNN
+F 3 "" H 2100 4100 50  0001 C CNN
+	1    2100 4100
+	1    0    0    -1
+$EndComp
+Wire Wire Line
+	2100 4100 2100 4000
+$Sheet
+S 1850 1950 700  550
+U 5AD4C411
+F0 "Motor" 50
+F1 "MotorConnect.sch" 50
+F2 "MOT1B" I R 2550 2150 50
+F3 "MOT1A" I R 2550 2050 50
+F4 "MOT2A" I R 2550 2250 50
+F5 "MOT2B" I R 2550 2350 50
+$EndSheet
+Wire Wire Line
+	2550 2050 2700 2050
+Wire Wire Line
+	2700 2150 2550 2150
+Wire Wire Line
+	2700 2250 2550 2250
+Wire Wire Line
+	2700 2350 2550 2350
+$Sheet
+S 5300 2550 700  550
+U 5AD4D269
+F0 "Heating" 50
+F1 "BasicHeater.sch" 50
+F2 "AVREF" I L 5300 2700 50
+F3 "TEMP" O L 5300 2850 50
+F4 "PWM" I R 6000 2900 50
+F5 "V_HEAT" I R 6000 2700 50
+F6 "HEATER" O R 6000 2800 50
+$EndSheet
+Text HLabel 5200 2700 0    50   Input ~ 0
+AVREF
+Text HLabel 5200 2850 0    50   Output ~ 0
+ETEMP
+Wire Wire Line
+	5200 2700 5300 2700
+Wire Wire Line
+	5300 2850 5200 2850
+Text HLabel 6150 2900 2    50   Input ~ 0
+PWM
+Wire Wire Line
+	3650 2300 3950 2300
+Wire Wire Line
+	3750 2100 4050 2100
+Wire Wire Line
+	3950 2300 3950 2200
+Wire Wire Line
+	3950 2200 6150 2200
+Wire Wire Line
+	6150 2200 6150 2700
+Wire Wire Line
+	6150 2700 6000 2700
+Connection ~ 3950 2300
+Wire Wire Line
+	3950 2300 4050 2300
+Wire Wire Line
+	6000 2900 6150 2900
+$Comp
+L Connector_Specialized:Screw_Terminal_01x02 J8
+U 1 1 5AD53BDD
+P 6750 2700
+AR Path="/5AC337B6/5ACBE919/5AD53BDD" Ref="J8"  Part="1"
+AR Path="/5AC337B6/5AD9F95A/5AD53BDD" Ref="J16"  Part="1"
+F 0 "J16" H 6829 2692 50  0000 L CNN
+F 1 "Extruder Heater" H 6829 2601 50  0000 L CNN
+F 2 "" H 6750 2700 50  0001 C CNN
+F 3 "~" H 6750 2700 50  0001 C CNN
+	1    6750 2700
+	1    0    0    -1
+$EndComp
+Wire Wire Line
+	6000 2800 6550 2800
+Wire Wire Line
+	6550 2700 6150 2700
+Connection ~ 6150 2700
 $EndSCHEMATC

Commit message: Added the rest of the printer parts. Should be complete more or less.
Parts:
- renumbered J7 to J1, J8 to J2
Changed lines of the file:
@@
 EESchema Schematic File Version 4
+LIBS:PrntrBoardV1-cache
 EELAYER 26 0
 EELAYER END
 $Descr A4 11693 8268
 encoding utf-8
-Sheet 25 29
+Sheet 25 35
 Title ""
 Date ""
@@
 	2600 4250 2700 4250
 $Comp
-L Connector_Generic:Conn_02x01 J7
+L Connector_Generic:Conn_02x01 J1
 U 1 1 5AD4BF35
 P 2300 4000
-AR Path="/5AC337B6/5ACBE919/5AD4BF35" Ref="J7"  Part="1"
+AR Path="/5AC337B6/5ACBE919/5AD4BF35" Ref="J1"  Part="1"
 AR Path="/5AC337B6/5AD9F95A/5AD4BF35" Ref="J15"  Part="1"
 F 0 "J15" H 2350 4217 50  0000 C CNN
@@
 	2600 4000 2700 4000
 $Comp
-L power:GND #PWR04
+L power:GND #PWR01
 U 1 1 5AD4C143
 P 2100 4100
-AR Path="/5AC337B6/5ACBE919/5AD4C143" Ref="#PWR04"  Part="1"
-AR Path="/5AC337B6/5AD9F95A/5AD4C143" Ref="#PWR043"  Part="1"
-F 0 "#PWR043" H 2100 3850 50  0001 C CNN
+AR Path="/5AC337B6/5ACBE919/5AD4C143" Ref="#PWR01"  Part="1"
+AR Path="/5AC337B6/5AD9F95A/5AD4C143" Ref="#PWR046"  Part="1"
+F 0 "#PWR046" H 2100 3850 50  0001 C CNN
 F 1 "GND" H 2105 3927 50  0000 C CNN
 F 2 "" H 2100 4100 50  0001 C CNN
@@
 	6000 2900 6150 2900
 $Comp
-L Connector_Specialized:Screw_Terminal_01x02 J8
+L Connector_Specialized:Screw_Terminal_01x02 J2
 U 1 1 5AD53BDD
 P 6750 2700
-AR Path="/5AC337B6/5ACBE919/5AD53BDD" Ref="J8"  Part="1"
+AR Path="/5AC337B6/5ACBE919/5AD53BDD" Ref="J2"  Part="1"
 AR Path="/5AC337B6/5AD9F95A/5AD53BDD" Ref="J16"  Part="1"
 F 0 "J16" H 6829 2692 50  0000 L CNN

Commit message: Finish the schematics. All pins are assinged to the NUCLEO-64 board.
Parts:
- renumbered J1 to J10, J2 to J11
Changed lines of the file:
@@
 $Descr A4 11693 8268
 encoding utf-8
-Sheet 25 35
+Sheet 3 35
 Title ""
 Date ""
@@
 	2600 4250 2700 4250
 $Comp
-L Connector_Generic:Conn_02x01 J1
+L Connector_Generic:Conn_02x01 J10
 U 1 1 5AD4BF35
 P 2300 4000
-AR Path="/5AC337B6/5ACBE919/5AD4BF35" Ref="J1"  Part="1"
-AR Path="/5AC337B6/5AD9F95A/5AD4BF35" Ref="J15"  Part="1"
-F 0 "J15" H 2350 4217 50  0000 C CNN
+AR Path="/5AC337B6/5ACBE919/5AD4BF35" Ref="J10"  Part="1"
+AR Path="/5AC337B6/5AD9F95A/5AD4BF35" Ref="J24"  Part="1"
+F 0 "J10" H 2350 4217 50  0000 C CNN
 F 1 "Probe" H 2350 4126 50  0000 C CNN
 F 2 "" H 2300 4000 50  0001 C CNN
@@
 	2600 4000 2700 4000
 $Comp
-L power:GND #PWR01
+L power:GND #PWR011
 U 1 1 5AD4C143
 P 2100 4100
-AR Path="/5AC337B6/5ACBE919/5AD4C143" Ref="#PWR01"  Part="1"
-AR Path="/5AC337B6/5AD9F95A/5AD4C143" Ref="#PWR046"  Part="1"
-F 0 "#PWR046" H 2100 3850 50  0001 C CNN
+AR Path="/5AC337B6/5ACBE919/5AD4C143" Ref="#PWR011"  Part="1"
+AR Path="/5AC337B6/5AD9F95A/5AD4C143" Ref="#PWR056"  Part="1"
+F 0 "#PWR011" H 2100 3850 50  0001 C CNN
 F 1 "GND" H 2105 3927 50  0000 C CNN
 F 2 "" H 2100 4100 50  0001 C CNN
@@
 	6000 2900 6150 2900
 $Comp
-L Connector_Specialized:Screw_Terminal_01x02 J2
+L Connector_Specialized:Screw_Terminal_01x02 J11
 U 1 1 5AD53BDD
 P 6750 2700
-AR Path="/5AC337B6/5ACBE919/5AD53BDD" Ref="J2"  Part="1"
-AR Path="/5AC337B6/5AD9F95A/5AD53BDD" Ref="J16"  Part="1"
-F 0 "J16" H 6829 2692 50  0000 L CNN
+AR Path="/5AC337B6/5ACBE919/5AD53BDD" Ref="J11"  Part="1"
+AR Path="/5AC337B6/5AD9F95A/5AD53BDD" Ref="J25"  Part="1"
+F 0 "J11" H 6829 2692 50  0000 L CNN
 F 1 "Extruder Heater" H 6829 2601 50  0000 L CNN
 F 2 "" H 6750 2700 50  0001 C CNN

Commit message: Split the bed heater in separate schematics.
Changed lines of the file:
@@
 $Descr A4 11693 8268
 encoding utf-8
-Sheet 3 35
+Sheet 25 35
 Title ""
 Date ""
@@
 AR Path="/5AC337B6/5ACBE919/5AD4BF35" Ref="J10"  Part="1"
 AR Path="/5AC337B6/5AD9F95A/5AD4BF35" Ref="J24"  Part="1"
-F 0 "J10" H 2350 4217 50  0000 C CNN
+F 0 "J24" H 2350 4217 50  0000 C CNN
 F 1 "Probe" H 2350 4126 50  0000 C CNN
 F 2 "" H 2300 4000 50  0001 C CNN
@@
 AR Path="/5AC337B6/5ACBE919/5AD4C143" Ref="#PWR011"  Part="1"
 AR Path="/5AC337B6/5AD9F95A/5AD4C143" Ref="#PWR056"  Part="1"
-F 0 "#PWR011" H 2100 3850 50  0001 C CNN
+F 0 "#PWR056" H 2100 3850 50  0001 C CNN
 F 1 "GND" H 2105 3927 50  0000 C CNN
 F 2 "" H 2100 4100 50  0001 C CNN
@@
 AR Path="/5AC337B6/5ACBE919/5AD53BDD" Ref="J11"  Part="1"
 AR Path="/5AC337B6/5AD9F95A/5AD53BDD" Ref="J25"  Part="1"
-F 0 "J11" H 6829 2692 50  0000 L CNN
+F 0 "J25" H 6829 2692 50  0000 L CNN
 F 1 "Extruder Heater" H 6829 2601 50  0000 L CNN
 F 2 "" H 6750 2700 50  0001 C CNN

Commit message: Assigned footprints for all components. Inductors are approximate size. MOSFETs dont agree with the footprints. Saved pcb netlist report as report.txt.
Parts:
- J10: footprint (none) -> Connector_PinHeader_2.54mm:PinHeader_1x02_P2.54mm_Vertical
- J11: footprint (none) -> TerminalBlock_Phoenix:TerminalBlock_Phoenix_MPT-0,5-2-2.54_1x02_P2.54mm_Horizontal
Changed lines of the file:
@@
 $Descr A4 11693 8268
 encoding utf-8
-Sheet 25 35
+Sheet 3 35
 Title ""
 Date ""
@@
 AR Path="/5AC337B6/5ACBE919/5AD4BF35" Ref="J10"  Part="1"
 AR Path="/5AC337B6/5AD9F95A/5AD4BF35" Ref="J24"  Part="1"
-F 0 "J24" H 2350 4217 50  0000 C CNN
+F 0 "J10" H 2350 4217 50  0000 C CNN
 F 1 "Probe" H 2350 4126 50  0000 C CNN
-F 2 "" H 2300 4000 50  0001 C CNN
+F 2 "Connector_PinHeader_2.54mm:PinHeader_1x02_P2.54mm_Vertical" H 2300 4000 50  0001 C CNN
 F 3 "~" H 2300 4000 50  0001 C CNN
 	1    2300 4000
@@
 AR Path="/5AC337B6/5ACBE919/5AD53BDD" Ref="J11"  Part="1"
 AR Path="/5AC337B6/5AD9F95A/5AD53BDD" Ref="J25"  Part="1"
-F 0 "J25" H 6829 2692 50  0000 L CNN
+F 0 "J11" H 6829 2692 50  0000 L CNN
 F 1 "Extruder Heater" H 6829 2601 50  0000 L CNN
-F 2 "" H 6750 2700 50  0001 C CNN
+F 2 "TerminalBlock_Phoenix:TerminalBlock_Phoenix_MPT-0,5-2-2.54_1x02_P2.54mm_Horizontal" H 6750 2700 50  0001 C CNN
 F 3 "~" H 6750 2700 50  0001 C CNN
 	1    6750 2700

Commit message: Updated components. Removed power supply. Component layout on PCB.
Changed lines of the file:
@@
 $Descr A4 11693 8268
 encoding utf-8
-Sheet 3 35
+Sheet 3 34
 Title ""
 Date ""
@@
 AR Path="/5AC337B6/5ACBE919/5AD4BF35" Ref="J10"  Part="1"
 AR Path="/5AC337B6/5AD9F95A/5AD4BF35" Ref="J24"  Part="1"
-F 0 "J10" H 2350 4217 50  0000 C CNN
+F 0 "J24" H 2350 4217 50  0000 C CNN
 F 1 "Probe" H 2350 4126 50  0000 C CNN
 F 2 "Connector_PinHeader_2.54mm:PinHeader_1x02_P2.54mm_Vertical" H 2300 4000 50  0001 C CNN
@@
 AR Path="/5AC337B6/5ACBE919/5AD53BDD" Ref="J11"  Part="1"
 AR Path="/5AC337B6/5AD9F95A/5AD53BDD" Ref="J25"  Part="1"
-F 0 "J11" H 6829 2692 50  0000 L CNN
+F 0 "J25" H 6829 2692 50  0000 L CNN
 F 1 "Extruder Heater" H 6829 2601 50  0000 L CNN
 F 2 "TerminalBlock_Phoenix:TerminalBlock_Phoenix_MPT-0,5-2-2.54_1x02_P2.54mm_Horizontal" H 6750 2700 50  0001 C CNN

Commit message: First routing complete. DRC pass.
Parts:
- J11: footprint TerminalBlock_Phoenix:TerminalBlock_Phoenix_MPT-0,5-2-2.54_1x02_P2.54mm_Horizontal -> TerminalBlock_Phoenix:TerminalBlock_Phoenix_PT-1,5-2-3.5-H_1x02_P3.50mm_Horizontal
Changed lines of the file:
@@
 F 0 "J25" H 6829 2692 50  0000 L CNN
 F 1 "Extruder Heater" H 6829 2601 50  0000 L CNN
-F 2 "TerminalBlock_Phoenix:TerminalBlock_Phoenix_MPT-0,5-2-2.54_1x02_P2.54mm_Horizontal" H 6750 2700 50  0001 C CNN
+F 2 "TerminalBlock_Phoenix:TerminalBlock_Phoenix_PT-1,5-2-3.5-H_1x02_P3.50mm_Horizontal" H 6750 2700 50  0001 C CNN
 F 3 "~" H 6750 2700 50  0001 C CNN
 	1    6750 2700
