File: Extruder.sch (KiCad schematic (older format))
At the start: 2 parts, among them J10 Probe, J11 Extruder Heater

Commit message: Update schematics to use TMC5130/TMC2130 drivers.
Connections:
- net labels added: 5V
- wire segments 30 -> 31
Changed lines of the file:
@@
 $Descr A4 11693 8268
 encoding utf-8
-Sheet 3 34
+Sheet 25 34
 Title ""
 Date ""
@@
 U 5AD4B0F5
 F0 "Driver" 50
-F1 "MotorDriver_TMC2660.sch" 50
+F1 "MotorDriver_TMC5130.sch" 50
 F2 "V_IO" I R 3650 2100 50
 F3 "V_MOTORS" I R 3650 2300 50
@@
 F14 "~ENABLE" I L 2700 3300 50
 F15 "SG_TST" O L 2700 3450 50
+F16 "5V" I R 3650 2500 50
 $EndSheet
 Text HLabel 2600 2600 0    50   Input ~ 0
@@
 	6550 2700 6150 2700
 Connection ~ 6150 2700
+Text HLabel 4050 2500 2    50   Input ~ 0
+5V
+Wire Wire Line
+	4050 2500 3650 2500
 $EndSCHEMATC

Commit message: Added motor clock source.
Connections:
- net labels added: CLOCK
- wire segments 31 -> 32
Changed lines of the file:
@@
 $EndDescr
 $Sheet
-S 2700 1950 950  1650
+S 2700 1950 950  1750
 U 5AD4B0F5
 F0 "Driver" 50
@@
 F15 "SG_TST" O L 2700 3450 50
 F16 "5V" I R 3650 2500 50
+F17 "CLOCK" I L 2700 3550 50
 $EndSheet
 Text HLabel 2600 2600 0    50   Input ~ 0
@@
 AR Path="/5AC337B6/5ACBE919/5AD4BF35" Ref="J10"  Part="1"
 AR Path="/5AC337B6/5AD9F95A/5AD4BF35" Ref="J24"  Part="1"
-F 0 "J10" H 2350 4217 50  0000 C CNN
+F 0 "J24" H 2350 4217 50  0000 C CNN
 F 1 "Probe" H 2350 4126 50  0000 C CNN
 F 2 "Connector_PinHeader_2.54mm:PinHeader_1x02_P2.54mm_Vertical" H 2300 4000 50  0001 C CNN
@@
 AR Path="/5AC337B6/5ACBE919/5AD53BDD" Ref="J11"  Part="1"
 AR Path="/5AC337B6/5AD9F95A/5AD53BDD" Ref="J25"  Part="1"
-F 0 "J11" H 6829 2692 50  0000 L CNN
+F 0 "J25" H 6829 2692 50  0000 L CNN
 F 1 "Extruder Heater" H 6829 2601 50  0000 L CNN
 F 2 "TerminalBlock_Phoenix:TerminalBlock_Phoenix_PT-1,5-2-3.5-H_1x02_P3.50mm_Horizontal" H 6750 2700 50  0001 C CNN
@@
 Wire Wire Line
 	4050 2500 3650 2500
+Text HLabel 2600 3550 0    50   Input ~ 0
+CLOCK
+Wire Wire Line
+	2600 3550 2700 3550
 $EndSCHEMATC

Commit message: Switched to local foorprints for terminals and LED. Switched to local foorprint for the printer driver ship - it has larger thermal pad ares.
Placement V1 complete.
Parts:
- J11: footprint TerminalBlock_Phoenix:TerminalBlock_Phoenix_PT-1,5-2-3.5-H_1x02_P3.50mm_Horizontal -> PrntrBoardV1:TerminalBlock_Phoenix_PT-1,5-2-3.5-H_1x02_P3.50mm_Horizontal
Changed lines of the file:
@@
 L Connector_Generic:Conn_02x01 J10
 U 1 1 5AD4BF35
-P 2300 4000
+P 2400 4000
 AR Path="/5AC337B6/5ACBE919/5AD4BF35" Ref="J10"  Part="1"
 AR Path="/5AC337B6/5AD9F95A/5AD4BF35" Ref="J24"  Part="1"
-F 0 "J24" H 2350 4217 50  0000 C CNN
-F 1 "Probe" H 2350 4126 50  0000 C CNN
-F 2 "Connector_PinHeader_2.54mm:PinHeader_1x02_P2.54mm_Vertical" H 2300 4000 50  0001 C CNN
-F 3 "~" H 2300 4000 50  0001 C CNN
-	1    2300 4000
-	1    0    0    -1
+F 0 "J24" H 2450 4217 50  0000 C CNN
+F 1 "Probe" H 2450 4126 50  0000 C CNN
+F 2 "Connector_PinHeader_2.54mm:PinHeader_1x02_P2.54mm_Vertical" H 2400 4000 50  0001 C CNN
+F 3 "~" H 2400 4000 50  0001 C CNN
+	1    2400 4000
+	-1   0    0    -1
 $EndComp
 Wire Wire Line
@@
 F 0 "J25" H 6829 2692 50  0000 L CNN
 F 1 "Extruder Heater" H 6829 2601 50  0000 L CNN
-F 2 "TerminalBlock_Phoenix:TerminalBlock_Phoenix_PT-1,5-2-3.5-H_1x02_P3.50mm_Horizontal" H 6750 2700 50  0001 C CNN
+F 2 "PrntrBoardV1:TerminalBlock_Phoenix_PT-1,5-2-3.5-H_1x02_P3.50mm_Horizontal" H 6750 2700 50  0001 C CNN
 F 3 "~" H 6750 2700 50  0001 C CNN
 	1    6750 2700

Commit message: Updated motor connector pinout.
Changed lines of the file:
@@
 F2 "V_IO" I R 3650 2100 50
 F3 "V_MOTORS" I R 3650 2300 50
-F4 "MOT1B" O L 2700 2150 50
-F5 "MOT1A" O L 2700 2050 50
-F6 "MOT2A" O L 2700 2250 50
-F7 "MOT2B" O L 2700 2350 50
-F8 "STEP" I L 2700 2600 50
-F9 "DIR" I L 2700 2700 50
-F10 "~CS" I L 2700 2850 50
-F11 "SCK" I L 2700 2950 50
-F12 "MOSI" I L 2700 3050 50
-F13 "MISO" O L 2700 3150 50
-F14 "~ENABLE" I L 2700 3300 50
-F15 "SG_TST" O L 2700 3450 50
-F16 "5V" I R 3650 2500 50
-F17 "CLOCK" I L 2700 3550 50
+F4 "STEP" I L 2700 2600 50
+F5 "DIR" I L 2700 2700 50
+F6 "~CS" I L 2700 2850 50
+F7 "SCK" I L 2700 2950 50
+F8 "MOSI" I L 2700 3050 50
+F9 "MISO" O L 2700 3150 50
+F10 "~ENABLE" I L 2700 3300 50
+F11 "SG_TST" O L 2700 3450 50
+F12 "5V" I R 3650 2500 50
+F13 "CLOCK" I L 2700 3550 50
+F14 "MOTB1" O L 2700 2050 50
+F15 "MOTA1" O L 2700 2250 50
+F16 "MOTA2" O L 2700 2350 50
+F17 "MOTB2" O L 2700 2150 50
 $EndSheet
 Text HLabel 2600 2600 0    50   Input ~ 0
@@
 F0 "Motor" 50
 F1 "MotorConnect.sch" 50
-F2 "MOT1B" I R 2550 2150 50
-F3 "MOT1A" I R 2550 2050 50
-F4 "MOT2A" I R 2550 2250 50
-F5 "MOT2B" I R 2550 2350 50
+F2 "MOTB1" I R 2550 2050 50
+F3 "MOTB2" I R 2550 2150 50
+F4 "MOTA2" I R 2550 2350 50
+F5 "MOTA1" I R 2550 2250 50
 $EndSheet
 Wire Wire Line

Commit message: Movet top FID to the top right corner. Added PCB origin. Switched 0.1uF 50V cpas to 0402 size.
Parts:
- J11: symbol Connector_Specialized:Screw_Terminal_01x02 -> PrntrBoardV1-rescue:Screw_Terminal_01x02-Connector_Specialized
Changed lines of the file:
@@
 	6000 2900 6150 2900
 $Comp
-L Connector_Specialized:Screw_Terminal_01x02 J11
+L PrntrBoardV1-rescue:Screw_Terminal_01x02-Connector_Specialized J11
 U 1 1 5AD53BDD
 P 6750 2700

Commit message: Some useless changes, I'll remove the SD_MODE wire soon.
Connections:
- net labels added: SD_MODE
- wire segments 32 -> 33
Changed lines of the file:
@@
 $Descr A4 11693 8268
 encoding utf-8
-Sheet 25 34
+Sheet 3 34
 Title ""
 Date ""
@@
 F16 "MOTA2" O L 2700 2350 50
 F17 "MOTB2" O L 2700 2150 50
+F18 "SD_MODE" I L 2700 3650 50
 $EndSheet
 Text HLabel 2600 2600 0    50   Input ~ 0
@@
 Wire Wire Line
 	2600 3550 2700 3550
+Text HLabel 2600 3650 0    50   Input ~ 0
+SD_MODE
+Wire Wire Line
+	2600 3650 2700 3650
 $EndSCHEMATC

Commit message: Removed SD_MODE wire. Added motor clock oscillator. Wired the clock on the internal layer to reduce EMI.
Connections:
- net labels removed: SD_MODE
- wire segments 33 -> 32
Changed lines of the file:
@@
 F16 "MOTA2" O L 2700 2350 50
 F17 "MOTB2" O L 2700 2150 50
-F18 "SD_MODE" I L 2700 3650 50
 $EndSheet
 Text HLabel 2600 2600 0    50   Input ~ 0
@@
 Wire Wire Line
 	2600 3550 2700 3550
-Text HLabel 2600 3650 0    50   Input ~ 0
-SD_MODE
-Wire Wire Line
-	2600 3650 2700 3650
 $EndSCHEMATC
