File: MotorConnect.sch (KiCad schematic (older format))
At the start: 1 part, among them J9 Stepper

Commit message: Added the rest of the printer parts. Should be complete more or less.
Parts:
- renumbered J9 to J3
Changed lines of the file:
@@
 EESchema Schematic File Version 4
+LIBS:PrntrBoardV1-cache
 EELAYER 26 0
 EELAYER END
 $Descr A4 11693 8268
 encoding utf-8
-Sheet 24 29
+Sheet 24 35
 Title ""
 Date ""
@@
 $EndDescr
 $Comp
-L Connector_Generic:Conn_01x04 J9
+L Connector_Generic:Conn_01x04 J3
 U 1 1 5AD04DCC
 P 4400 2700
-AR Path="/5AC337B6/5ACBE919/5AD4C411/5AD04DCC" Ref="J9"  Part="1"
+AR Path="/5AC337B6/5ACBE919/5AD4C411/5AD04DCC" Ref="J3"  Part="1"
 AR Path="/5AC337B6/5AD04C54/5AD04DCC" Ref="J11"  Part="1"
 AR Path="/5AC337B6/5AD0CC96/5AD04DCC" Ref="J12"  Part="1"

Commit message: Finish the schematics. All pins are assinged to the NUCLEO-64 board.
Parts:
- renumbered J3 to J12
Changed lines of the file:
@@
 $EndDescr
 $Comp
-L Connector_Generic:Conn_01x04 J3
+L Connector_Generic:Conn_01x04 J12
 U 1 1 5AD04DCC
 P 4400 2700
-AR Path="/5AC337B6/5ACBE919/5AD4C411/5AD04DCC" Ref="J3"  Part="1"
-AR Path="/5AC337B6/5AD04C54/5AD04DCC" Ref="J11"  Part="1"
-AR Path="/5AC337B6/5AD0CC96/5AD04DCC" Ref="J12"  Part="1"
-AR Path="/5AC337B6/5AD1664A/5AD1665B/5AD04DCC" Ref="J13"  Part="1"
-AR Path="/5AC337B6/5AD1664A/5AD1665E/5AD04DCC" Ref="J14"  Part="1"
-AR Path="/5AC337B6/5AD9F95A/5AD4C411/5AD04DCC" Ref="J17"  Part="1"
-F 0 "J17" H 4480 2692 50  0000 L CNN
+AR Path="/5AC337B6/5ACBE919/5AD4C411/5AD04DCC" Ref="J12"  Part="1"
+AR Path="/5AC337B6/5AD04C54/5AD04DCC" Ref="J20"  Part="1"
+AR Path="/5AC337B6/5AD0CC96/5AD04DCC" Ref="J21"  Part="1"
+AR Path="/5AC337B6/5AD1664A/5AD1665B/5AD04DCC" Ref="J22"  Part="1"
+AR Path="/5AC337B6/5AD1664A/5AD1665E/5AD04DCC" Ref="J23"  Part="1"
+AR Path="/5AC337B6/5AD9F95A/5AD4C411/5AD04DCC" Ref="J26"  Part="1"
+F 0 "J26" H 4480 2692 50  0000 L CNN
 F 1 "Stepper" H 4480 2601 50  0000 L CNN
 F 2 "" H 4400 2700 50  0001 C CNN

Commit message: Assigned footprints for all components. Inductors are approximate size. MOSFETs dont agree with the footprints. Saved pcb netlist report as report.txt.
Parts:
- J12: footprint (none) -> Connector_PinHeader_2.54mm:PinHeader_1x03_P2.54mm_Vertical
Changed lines of the file:
@@
 F 0 "J26" H 4480 2692 50  0000 L CNN
 F 1 "Stepper" H 4480 2601 50  0000 L CNN
-F 2 "" H 4400 2700 50  0001 C CNN
+F 2 "Connector_PinHeader_2.54mm:PinHeader_1x03_P2.54mm_Vertical" H 4400 2700 50  0001 C CNN
 F 3 "~" H 4400 2700 50  0001 C CNN
 	1    4400 2700

Commit message: Updated components. Removed power supply. Component layout on PCB.
Parts:
- J12: footprint Connector_PinHeader_2.54mm:PinHeader_1x03_P2.54mm_Vertical -> Connector_PinHeader_2.54mm:PinHeader_1x04_P2.54mm_Vertical
Changed lines of the file:
@@
 $Descr A4 11693 8268
 encoding utf-8
-Sheet 24 35
+Sheet 24 34
 Title ""
 Date ""
@@
 F 0 "J26" H 4480 2692 50  0000 L CNN
 F 1 "Stepper" H 4480 2601 50  0000 L CNN
-F 2 "Connector_PinHeader_2.54mm:PinHeader_1x03_P2.54mm_Vertical" H 4400 2700 50  0001 C CNN
+F 2 "Connector_PinHeader_2.54mm:PinHeader_1x04_P2.54mm_Vertical" H 4400 2700 50  0001 C CNN
 F 3 "~" H 4400 2700 50  0001 C CNN
 	1    4400 2700

Commit message: Routed most of the power traces.
Connections:
- net MOT2A: now also J12.4 (Pin_4); no longer J12.3 (Pin_3)
- net MOT2B: now also J12.3 (Pin_3); no longer J12.4 (Pin_4)
Changed lines of the file:
@@
 $Descr A4 11693 8268
 encoding utf-8
-Sheet 24 34
+Sheet 6 34
 Title ""
 Date ""
@@
 AR Path="/5AC337B6/5AD1664A/5AD1665E/5AD04DCC" Ref="J23"  Part="1"
 AR Path="/5AC337B6/5AD9F95A/5AD4C411/5AD04DCC" Ref="J26"  Part="1"
-F 0 "J26" H 4480 2692 50  0000 L CNN
+F 0 "J20" H 4480 2692 50  0000 L CNN
 F 1 "Stepper" H 4480 2601 50  0000 L CNN
 F 2 "Connector_PinHeader_2.54mm:PinHeader_1x04_P2.54mm_Vertical" H 4400 2700 50  0001 C CNN
@@
 Text HLabel 3900 2700 0    50   Input ~ 0
 MOT1A
+Text HLabel 3900 2900 0    50   Input ~ 0
+MOT2A
 Text HLabel 3900 2800 0    50   Input ~ 0
-MOT2A
-Text HLabel 3900 2900 0    50   Input ~ 0
 MOT2B
 Wire Wire Line

Commit message: First routing complete. DRC pass.
Changed lines of the file:
@@
 AR Path="/5AC337B6/5AD1664A/5AD1665E/5AD04DCC" Ref="J23"  Part="1"
 AR Path="/5AC337B6/5AD9F95A/5AD4C411/5AD04DCC" Ref="J26"  Part="1"
-F 0 "J20" H 4480 2692 50  0000 L CNN
+F 0 "J26" H 4480 2692 50  0000 L CNN
 F 1 "Stepper" H 4480 2601 50  0000 L CNN
 F 2 "Connector_PinHeader_2.54mm:PinHeader_1x04_P2.54mm_Vertical" H 4400 2700 50  0001 C CNN

Commit message: Added mounting holes and fiducials. Placed all components labels so they are readable.
Changed lines of the file:
@@
 AR Path="/5AC337B6/5AD1664A/5AD1665E/5AD04DCC" Ref="J23"  Part="1"
 AR Path="/5AC337B6/5AD9F95A/5AD4C411/5AD04DCC" Ref="J26"  Part="1"
-F 0 "J26" H 4480 2692 50  0000 L CNN
+F 0 "J21" H 4480 2692 50  0000 L CNN
 F 1 "Stepper" H 4480 2601 50  0000 L CNN
 F 2 "Connector_PinHeader_2.54mm:PinHeader_1x04_P2.54mm_Vertical" H 4400 2700 50  0001 C CNN

Commit message: Placed motor drivers and some endstops.
Changed lines of the file:
@@
 AR Path="/5AC337B6/5AD1664A/5AD1665E/5AD04DCC" Ref="J23"  Part="1"
 AR Path="/5AC337B6/5AD9F95A/5AD4C411/5AD04DCC" Ref="J26"  Part="1"
-F 0 "J21" H 4480 2692 50  0000 L CNN
+F 0 "J22" H 4480 2692 50  0000 L CNN
 F 1 "Stepper" H 4480 2601 50  0000 L CNN
 F 2 "Connector_PinHeader_2.54mm:PinHeader_1x04_P2.54mm_Vertical" H 4400 2700 50  0001 C CNN
