File: MotorConnect.sch (KiCad schematic (older format))
At the start: 1 part, among them J12 Stepper

Commit message: Update schematics to use TMC5130/TMC2130 drivers.
Changed lines of the file:
@@
 AR Path="/5AC337B6/5AD1664A/5AD1665E/5AD04DCC" Ref="J23"  Part="1"
 AR Path="/5AC337B6/5AD9F95A/5AD4C411/5AD04DCC" Ref="J26"  Part="1"
-F 0 "J22" H 4480 2692 50  0000 L CNN
+F 0 "J26" H 4480 2692 50  0000 L CNN
 F 1 "Stepper" H 4480 2601 50  0000 L CNN
 F 2 "Connector_PinHeader_2.54mm:PinHeader_1x04_P2.54mm_Vertical" H 4400 2700 50  0001 C CNN

Commit message: Updated motor connector pinout.
Connections:
- net MOT1A renamed MOTB2
- net MOT1B renamed MOTB1
- net MOT2A renamed MOTA2
- net MOT2B renamed MOTA1
Changed lines of the file:
@@
 $Descr A4 11693 8268
 encoding utf-8
-Sheet 6 34
+Sheet 28 34
 Title ""
 Date ""
@@
 $EndComp
 Text HLabel 3900 2600 0    50   Input ~ 0
-MOT1B
+MOTB1
 Text HLabel 3900 2700 0    50   Input ~ 0
-MOT1A
+MOTB2
 Text HLabel 3900 2900 0    50   Input ~ 0
-MOT2A
+MOTA2
 Text HLabel 3900 2800 0    50   Input ~ 0
-MOT2B
+MOTA1
 Wire Wire Line
 	3900 2600 4200 2600

Commit message: Reset schematics for tmc2660. Clean the board layout.
Parts:
- renumbered J12 to J19
Changed lines of the file:
@@
 $EndDescr
 $Comp
-L Connector_Generic:Conn_01x04 J12
+L Connector_Generic:Conn_01x04 J19
 U 1 1 5AD04DCC
 P 4400 2700
-AR Path="/5AC337B6/5ACBE919/5AD4C411/5AD04DCC" Ref="J12"  Part="1"
-AR Path="/5AC337B6/5AD04C54/5AD04DCC" Ref="J20"  Part="1"
-AR Path="/5AC337B6/5AD0CC96/5AD04DCC" Ref="J21"  Part="1"
-AR Path="/5AC337B6/5AD1664A/5AD1665B/5AD04DCC" Ref="J22"  Part="1"
-AR Path="/5AC337B6/5AD1664A/5AD1665E/5AD04DCC" Ref="J23"  Part="1"
-AR Path="/5AC337B6/5AD9F95A/5AD4C411/5AD04DCC" Ref="J26"  Part="1"
-F 0 "J26" H 4480 2692 50  0000 L CNN
+AR Path="/5AC337B6/5ACBE919/5AD4C411/5AD04DCC" Ref="J19"  Part="1"
+AR Path="/5AC337B6/5AD04C54/5AD04DCC" Ref="J27"  Part="1"
+AR Path="/5AC337B6/5AD0CC96/5AD04DCC" Ref="J28"  Part="1"
+AR Path="/5AC337B6/5AD1664A/5AD1665B/5AD04DCC" Ref="J29"  Part="1"
+AR Path="/5AC337B6/5AD1664A/5AD1665E/5AD04DCC" Ref="J30"  Part="1"
+AR Path="/5AC337B6/5AD9F95A/5AD4C411/5AD04DCC" Ref="J33"  Part="1"
+F 0 "J33" H 4480 2692 50  0000 L CNN
 F 1 "Stepper" H 4480 2601 50  0000 L CNN
 F 2 "Connector_PinHeader_2.54mm:PinHeader_1x04_P2.54mm_Vertical" H 4400 2700 50  0001 C CNN

Commit message: Updated motor connectors to Molex SL style.
Parts:
- J19: footprint Connector_PinHeader_2.54mm:PinHeader_1x04_P2.54mm_Vertical -> kicad-molex-sl-footprints:Molex-SL-4POS
Changed lines of the file:
@@
 $Descr A4 11693 8268
 encoding utf-8
-Sheet 28 35
+Sheet 6 35
 Title ""
 Date ""
@@
 AR Path="/5AC337B6/5AD1664A/5AD1665E/5AD04DCC" Ref="J30"  Part="1"
 AR Path="/5AC337B6/5AD9F95A/5AD4C411/5AD04DCC" Ref="J33"  Part="1"
-F 0 "J33" H 4480 2692 50  0000 L CNN
+F 0 "J19" H 4480 2692 50  0000 L CNN
 F 1 "Stepper" H 4480 2601 50  0000 L CNN
-F 2 "Connector_PinHeader_2.54mm:PinHeader_1x04_P2.54mm_Vertical" H 4400 2700 50  0001 C CNN
+F 2 "kicad-molex-sl-footprints:Molex-SL-4POS" H 4400 2700 50  0001 C CNN
 F 3 "~" H 4400 2700 50  0001 C CNN
 	1    4400 2700

Commit message: Add reverse polarity protection diode.
Changed lines of the file:
@@
 AR Path="/5AC337B6/5AD1664A/5AD1665E/5AD04DCC" Ref="J30"  Part="1"
 AR Path="/5AC337B6/5AD9F95A/5AD4C411/5AD04DCC" Ref="J33"  Part="1"
-F 0 "J19" H 4480 2692 50  0000 L CNN
+F 0 "J33" H 4480 2692 50  0000 L CNN
 F 1 "Stepper" H 4480 2601 50  0000 L CNN
 F 2 "kicad-molex-sl-footprints:Molex-SL-4POS" H 4400 2700 50  0001 C CNN
