File: BasicHeater.sch (KiCad schematic (older format))
At the start: 10 parts, among them J13 Thermistor

Commit message: Change 10uF capacitor footprints to 1206.
Parts:
- C17: value 10uF 35V -> 10uF 50V; footprint Capacitor_SMD:CP_Elec_4x5.3 -> Capacitor_SMD:C_1206_3216Metric; symbol Device:CP1_Small -> Device:C
Changed lines of the file:
@@
 	5550 3600 5550 3650
 $Comp
-L Device:CP1_Small C17
+L Device:C C17
 U 1 1 5AD51206
-P 4950 2450
+P 4950 2400
 AR Path="/5AC337B6/5ACBE919/5AD4D269/5AD51206" Ref="C17"  Part="1"
 AR Path="/5AC337B6/5AD9F95A/5AD4D269/5AD51206" Ref="C70"  Part="1"
 AR Path="/5AB8F10D/5AD51206" Ref="C72"  Part="1"
 F 0 "C70" H 4750 2500 50  0000 L CNN
-F 1 "10uF 35V" H 4500 2400 50  0000 L CNN
-F 2 "Capacitor_SMD:CP_Elec_4x5.3" H 4950 2450 50  0001 C CNN
-F 3 "~" H 4950 2450 50  0001 C CNN
-	1    4950 2450
+F 1 "10uF 50V" H 4550 2300 50  0000 L CNN
+F 2 "Capacitor_SMD:C_1206_3216Metric" H 4950 2400 50  0001 C CNN
+F 3 "~" H 4950 2400 50  0001 C CNN
+	1    4950 2400
 	1    0    0    -1
 $EndComp
@@
 	4950 2550 4950 2700
 Wire Wire Line
-	4950 2350 4950 1950
+	4950 2250 4950 1950
 Wire Wire Line
 	4950 1950 5250 1950

Commit message: Updated TR3 foor print and re-routed tracks.
Parts:
- D17: footprint Diode_SMD:D_SOD-323F -> Diode_SMD:D_SOD-323_HandSoldering
Changed lines of the file:
@@
 F 0 "D17" V 5554 2329 50  0000 L CNN
 F 1 "1N4148" V 5645 2329 50  0000 L CNN
-F 2 "Diode_SMD:D_SOD-323F" H 5600 2250 50  0001 C CNN
+F 2 "Diode_SMD:D_SOD-323_HandSoldering" H 5600 2250 50  0001 C CNN
 F 3 "~" H 5600 2250 50  0001 C CNN
 	1    5600 2250
