File: PrntrBoardV1.sch (KiCad schematic (older format))
At the start: 25 parts, among them J1 EXT 5V, J2 Bed Heater, J29 12-24V, J3 Z Probe, J4 E0 Cool, J5 E0 Part, J6 E1 Cool, J7 E1 Part, J8 Always On Fan 1, J9 Always On Fan 2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

Commit message: Update schematics to use TMC5130/TMC2130 drivers.
Parts:
- removed J1: EXT 5V, Connector_PinHeader_2.54mm:PinHeader_1x02_P2.54mm_Vertical, symbol Connector_Generic:Conn_01x02
- added J1: EXT 5V, TerminalBlock_Phoenix:TerminalBlock_Phoenix_PT-1,5-2-3.5-H_1x02_P3.50mm_Horizontal, symbol Connector_Specialized:Screw_Terminal_01x02
Connections:
- wire segments 207 -> 209
Changed lines of the file:
@@
 F39 "E1_TEMP" O L 6050 2250 50
 F40 "E1_PWM" I L 6050 2600 50
+F41 "5V" I L 6050 1350 50
 $EndSheet
 $Comp
@@
 	5900 800  2550 800
 Connection ~ 5900 800
-$Comp
-L Connector_Generic:Conn_01x02 J1
-U 1 1 5AD9E37F
-P 3500 1950
-F 0 "J1" H 3420 1625 50  0000 C CNN
-F 1 "EXT 5V" H 3420 1716 50  0000 C CNN
-F 2 "Connector_PinHeader_2.54mm:PinHeader_1x02_P2.54mm_Vertical" H 3500 1950 50  0001 C CNN
-F 3 "~" H 3500 1950 50  0001 C CNN
-	1    3500 1950
-	-1   0    0    1
-$EndComp
 $Comp
 L power:GND #PWR01
@@
 $EndComp
 NoConn ~ 1950 1400
+$Comp
+L Connector_Specialized:Screw_Terminal_01x02 J1
+U 1 1 5AEDA4A7
+P 3500 1950
+F 0 "J1" H 3420 1625 50  0000 C CNN
+F 1 "EXT 5V" H 3420 1716 50  0000 C CNN
+F 2 "TerminalBlock_Phoenix:TerminalBlock_Phoenix_PT-1,5-2-3.5-H_1x02_P3.50mm_Horizontal" H 3500 1950 50  0001 C CNN
+F 3 "~" H 3500 1950 50  0001 C CNN
+	1    3500 1950
+	-1   0    0    1
+$EndComp
+Wire Wire Line
+	6050 1350 4100 1350
+Wire Wire Line
+	4100 1350 4100 1850
+Connection ~ 4100 1850
 $EndSCHEMATC

Commit message: Added motor clock source.
Parts:
- added J30: Ext Motor Clock, Connector_PinHeader_2.54mm:PinHeader_1x04_P2.54mm_Vertical, symbol Connector_Generic:Conn_01x02
- added JP2: Motor Clock Select, Jumper:SolderJumper-3_P1.3mm_Open_Pad1.0x1.5mm, symbol Jumper:Jumper_3_Bridged12
Connections:
- net labels added: MOT_CLOCK
- wire segments 209 -> 217
Changed lines of the file:
@@
 F40 "E1_PWM" I L 6050 2600 50
 F41 "5V" I L 6050 1350 50
+F42 "CLOCK" I L 6050 3400 50
 $EndSheet
 $Comp
 L my_4xxx:4078 U1
 U 1 1 5AB8C4A5
-P 5400 3200
-F 0 "U1" H 5600 3650 50  0000 C CNN
-F 1 "4078" H 5550 3750 50  0000 C CNN
-F 2 "Package_SO:TSSOP-14_4.4x5mm_P0.65mm" H 5400 3200 50  0001 C CNN
-F 3 "" H 5400 3200 50  0001 C CNN
-	1    5400 3200
+P 5250 3200
+F 0 "U1" H 5450 3650 50  0000 C CNN
+F 1 "4078" H 5400 3750 50  0000 C CNN
+F 2 "Package_SO:TSSOP-14_4.4x5mm_P0.65mm" H 5250 3200 50  0001 C CNN
+F 3 "" H 5250 3200 50  0001 C CNN
+	1    5250 3200
 	-1   0    0    1
 $EndComp
 Wire Wire Line
-	6050 2850 5900 2850
-Wire Wire Line
-	6050 2950 5900 2950
-Wire Wire Line
-	6050 3050 5900 3050
-Wire Wire Line
-	6050 3150 5900 3150
-Wire Wire Line
-	6050 3250 5900 3250
-Wire Wire Line
-	5900 3350 5900 3450
-Connection ~ 5900 3450
-Wire Wire Line
-	5900 3450 5900 3550
+	6050 2850 5750 2850
+Wire Wire Line
+	6050 2950 5750 2950
+Wire Wire Line
+	6050 3050 5750 3050
+Wire Wire Line
+	6050 3150 5750 3150
+Wire Wire Line
+	6050 3250 5750 3250
+Wire Wire Line
+	5750 3350 5750 3450
+Connection ~ 5750 3450
+Wire Wire Line
+	5750 3450 5750 3550
 $Comp
 L power:GND #PWR04
 U 1 1 5AB8C5FB
-P 5900 3800
-F 0 "#PWR04" H 5900 3550 50  0001 C CNN
-F 1 "GND" H 5905 3627 50  0000 C CNN
-F 2 "" H 5900 3800 50  0001 C CNN
-F 3 "" H 5900 3800 50  0001 C CNN
-	1    5900 3800
-	1    0    0    -1
-$EndComp
-Connection ~ 5900 3550
+P 5750 3800
+F 0 "#PWR04" H 5750 3550 50  0001 C CNN
+F 1 "GND" H 5755 3627 50  0000 C CNN
+F 2 "" H 5750 3800 50  0001 C CNN
+F 3 "" H 5750 3800 50  0001 C CNN
+	1    5750 3800
+	1    0    0    -1
+$EndComp
+Connection ~ 5750 3550
 Wire Wire Line
 	5400 1050 6050 1050
@@
 Pin budget:\n17 GPIO out\n7 GPIO PWM out\n12 GPIO in\n3 ADC in\n1 SPI
 Wire Wire Line
-	4900 3350 4500 3350
-Text Label 4600 3350 0    50   ~ 0
+	4750 3350 4650 3350
+Text Label 4700 3350 0    50   ~ 0
 STALL
 $Sheet
@@
 Text Label 10050 5200 2    50   ~ 0
 Z_PROBE_IN
-NoConn ~ 4900 3200
+NoConn ~ 4750 3200
 $Comp
 L NUCLEO-64:NUCLEO-64 U11
@@
 NoConn ~ 1750 3000
 Wire Wire Line
-	5900 3550 5900 3800
-Wire Wire Line
-	5400 2800 5400 2450
-Wire Wire Line
-	5400 2450 5150 2450
+	5750 3550 5750 3800
+Wire Wire Line
+	5250 2800 5250 2450
+Wire Wire Line
+	5250 2450 5150 2450
 Connection ~ 5150 2450
 Wire Wire Line
-	5400 3600 5400 3900
-Wire Wire Line
-	5400 3900 4400 3900
+	5250 3600 5250 3900
+Wire Wire Line
+	5250 3900 4400 3900
 Wire Wire Line
 	4400 3900 4400 3400
@@
 	4100 1350 4100 1850
 Connection ~ 4100 1850
+Wire Wire Line
+	6050 3400 5850 3400
+Wire Wire Line
+	5850 3400 5850 4050
+Text Label 5850 3950 0    50   ~ 0
+MOT_CLOCK
+$Comp
+L Jumper:Jumper_3_Bridged12 JP2
+U 1 1 5AE5CEDD
+P 4400 6250
+F 0 "JP2" H 4250 6350 50  0000 C CNN
+F 1 "Motor Clock Select" H 4550 6050 50  0000 C CNN
+F 2 "Jumper:SolderJumper-3_P1.3mm_Open_Pad1.0x1.5mm" H 4400 6250 50  0001 C CNN
+F 3 "~" H 4400 6250 50  0001 C CNN
+	1    4400 6250
+	1    0    0    -1
+$EndComp
+Wire Wire Line
+	3250 6250 4150 6250
+Wire Wire Line
+	4400 6400 4400 6900
+Text Label 4400 6700 0    50   ~ 0
+MOT_CLOCK
+$Comp
+L Connector_Generic:Conn_01x02 J30
+U 1 1 5AE7F628
+P 4300 5800
+F 0 "J30" H 4220 5475 50  0000 C CNN
+F 1 "Ext Motor Clock" H 4220 5566 50  0000 C CNN
+F 2 "Connector_PinHeader_2.54mm:PinHeader_1x04_P2.54mm_Vertical" H 4300 5800 50  0001 C CNN
+F 3 "~" H 4300 5800 50  0001 C CNN
+	1    4300 5800
+	-1   0    0    1
+$EndComp
+$Comp
+L power:GND #PWR086
+U 1 1 5AE7F7F3
+P 4500 5900
+F 0 "#PWR086" H 4500 5650 50  0001 C CNN
+F 1 "GND" H 4650 5800 50  0000 C CNN
+F 2 "" H 4500 5900 50  0001 C CNN
+F 3 "" H 4500 5900 50  0001 C CNN
+	1    4500 5900
+	1    0    0    -1
+$EndComp
+Wire Wire Line
+	4500 5800 4500 5900
+Wire Wire Line
+	4500 5700 4750 5700
+Wire Wire Line
+	4750 5700 4750 6250
+Wire Wire Line
+	4750 6250 4650 6250
 $EndSCHEMATC

Commit message: Switched to local foorprints for terminals and LED. Switched to local foorprint for the printer driver ship - it has larger thermal pad ares.
Placement V1 complete.
Parts:
- removed F1: Mini blade fuse, Fuse:Fuse_Blade_Mini_directSolder, symbol Device:Fuse
- added C88: 100uF, Capacitor_SMD:CP_Elec_6.3x7.7, symbol Device:CP
- added C89: 0.001uF, Capacitor_SMD:C_0603_1608Metric, symbol Device:C
- added MK4: Mounting_Hole, MountingHole:MountingHole_3.2mm_M3, symbol Mechanical:Mounting_Hole
- J1, J4, J5, J6, J7, J8, J9: footprint TerminalBlock_Phoenix:TerminalBlock_Phoenix_PT-1,5-2-3.5-H_1x02_P3.50mm_Horizontal -> PrntrBoardV1:TerminalBlock_Phoenix_PT-1,5-2-3.5-H_1x02_P3.50mm_Horizontal
- J2, J29: footprint TerminalBlock_Phoenix:TerminalBlock_Phoenix_MKDS-1,5-2_1x02_P5.00mm_Horizontal -> PrntrBoardV1:TerminalBlock_Phoenix_MKDS-1,5-2-5.08_1x02_P5.08mm_Horizontal
- J30: footprint Connector_PinHeader_2.54mm:PinHeader_1x04_P2.54mm_Vertical -> Connector_PinHeader_2.54mm:PinHeader_1x02_P2.54mm_Vertical
Connections:
- wire segments 217 -> 222
- no-connect marks 32 -> 33
Changed lines of the file:
@@
 F 0 "J2" H 8180 4042 50  0000 L CNN
 F 1 "Bed Heater" H 8180 3951 50  0000 L CNN
-F 2 "TerminalBlock_Phoenix:TerminalBlock_Phoenix_MKDS-1,5-2_1x02_P5.00mm_Horizontal" H 8100 4050 50  0001 C CNN
+F 2 "PrntrBoardV1:TerminalBlock_Phoenix_MKDS-1,5-2-5.08_1x02_P5.08mm_Horizontal" H 8100 4050 50  0001 C CNN
 F 3 "~" H 8100 4050 50  0001 C CNN
 	1    8100 4050
@@
 F 0 "J7" H 9479 3342 50  0000 L CNN
 F 1 "E1 Part" H 9479 3251 50  0000 L CNN
-F 2 "TerminalBlock_Phoenix:TerminalBlock_Phoenix_PT-1,5-2-3.5-H_1x02_P3.50mm_Horizontal" H 9400 3350 50  0001 C CNN
+F 2 "PrntrBoardV1:TerminalBlock_Phoenix_PT-1,5-2-3.5-H_1x02_P3.50mm_Horizontal" H 9400 3350 50  0001 C CNN
 F 3 "~" H 9400 3350 50  0001 C CNN
 	1    9400 3350
@@
 F 0 "J6" H 9479 2792 50  0000 L CNN
 F 1 "E1 Cool" H 9479 2701 50  0000 L CNN
-F 2 "TerminalBlock_Phoenix:TerminalBlock_Phoenix_PT-1,5-2-3.5-H_1x02_P3.50mm_Horizontal" H 9400 2800 50  0001 C CNN
+F 2 "PrntrBoardV1:TerminalBlock_Phoenix_PT-1,5-2-3.5-H_1x02_P3.50mm_Horizontal" H 9400 2800 50  0001 C CNN
 F 3 "~" H 9400 2800 50  0001 C CNN
 	1    9400 2800
@@
 F 0 "J5" H 9479 2192 50  0000 L CNN
 F 1 "E0 Part" H 9479 2101 50  0000 L CNN
-F 2 "TerminalBlock_Phoenix:TerminalBlock_Phoenix_PT-1,5-2-3.5-H_1x02_P3.50mm_Horizontal" H 9400 2200 50  0001 C CNN
+F 2 "PrntrBoardV1:TerminalBlock_Phoenix_PT-1,5-2-3.5-H_1x02_P3.50mm_Horizontal" H 9400 2200 50  0001 C CNN
 F 3 "~" H 9400 2200 50  0001 C CNN
 	1    9400 2200
@@
 F 0 "J4" H 9479 1642 50  0000 L CNN
 F 1 "E0 Cool" H 9479 1551 50  0000 L CNN
-F 2 "TerminalBlock_Phoenix:TerminalBlock_Phoenix_PT-1,5-2-3.5-H_1x02_P3.50mm_Horizontal" H 9400 1650 50  0001 C CNN
+F 2 "PrntrBoardV1:TerminalBlock_Phoenix_PT-1,5-2-3.5-H_1x02_P3.50mm_Horizontal" H 9400 1650 50  0001 C CNN
 F 3 "~" H 9400 1650 50  0001 C CNN
 	1    9400 1650
@@
 	1    0    0    -1
 $EndComp
-$Comp
-L Device:Fuse F1
-U 1 1 5AB99299
-P 8450 1050
-F 0 "F1" V 8350 1000 50  0000 C CNN
-F 1 "Mini blade fuse" V 8550 1000 50  0000 C CNN
-F 2 "Fuse:Fuse_Blade_Mini_directSolder" V 8380 1050 50  0001 C CNN
-F 3 "~" H 8450 1050 50  0001 C CNN
-	1    8450 1050
-	0    1    1    0
-$EndComp
-Wire Wire Line
-	8300 1050 7900 1050
 Connection ~ 7900 1050
 Wire Wire Line
 	7900 1050 7900 3950
-Wire Wire Line
-	8600 1050 8700 1050
 Wire Wire Line
 	8950 1200 8950 1250
@@
 F 0 "J8" H 10229 1642 50  0000 L CNN
 F 1 "Always On Fan 1" H 10229 1551 50  0000 L CNN
-F 2 "TerminalBlock_Phoenix:TerminalBlock_Phoenix_PT-1,5-2-3.5-H_1x02_P3.50mm_Horizontal" H 10150 1650 50  0001 C CNN
+F 2 "PrntrBoardV1:TerminalBlock_Phoenix_PT-1,5-2-3.5-H_1x02_P3.50mm_Horizontal" H 10150 1650 50  0001 C CNN
 F 3 "~" H 10150 1650 50  0001 C CNN
 	1    10150 1650
@@
 F 0 "J9" H 10229 2042 50  0000 L CNN
 F 1 "Always On Fan 2" H 10229 1951 50  0000 L CNN
-F 2 "TerminalBlock_Phoenix:TerminalBlock_Phoenix_PT-1,5-2-3.5-H_1x02_P3.50mm_Horizontal" H 10150 2050 50  0001 C CNN
+F 2 "PrntrBoardV1:TerminalBlock_Phoenix_PT-1,5-2-3.5-H_1x02_P3.50mm_Horizontal" H 10150 2050 50  0001 C CNN
 F 3 "~" H 10150 2050 50  0001 C CNN
 	1    10150 2050
@@
 F 0 "J29" H 2270 575 50  0000 C CNN
 F 1 "12-24V" H 2270 666 50  0000 C CNN
-F 2 "TerminalBlock_Phoenix:TerminalBlock_Phoenix_MKDS-1,5-2_1x02_P5.00mm_Horizontal" H 2350 900 50  0001 C CNN
+F 2 "PrntrBoardV1:TerminalBlock_Phoenix_MKDS-1,5-2-5.08_1x02_P5.08mm_Horizontal" H 2350 900 50  0001 C CNN
 F 3 "~" H 2350 900 50  0001 C CNN
 	1    2350 900
@@
 F 0 "J1" H 3420 1625 50  0000 C CNN
 F 1 "EXT 5V" H 3420 1716 50  0000 C CNN
-F 2 "TerminalBlock_Phoenix:TerminalBlock_Phoenix_PT-1,5-2-3.5-H_1x02_P3.50mm_Horizontal" H 3500 1950 50  0001 C CNN
+F 2 "PrntrBoardV1:TerminalBlock_Phoenix_PT-1,5-2-3.5-H_1x02_P3.50mm_Horizontal" H 3500 1950 50  0001 C CNN
 F 3 "~" H 3500 1950 50  0001 C CNN
 	1    3500 1950
@@
 $EndComp
 Wire Wire Line
-	6050 1350 4100 1350
+	6050 1350 5050 1350
 Wire Wire Line
 	4100 1350 4100 1850
@@
 F 0 "J30" H 4220 5475 50  0000 C CNN
 F 1 "Ext Motor Clock" H 4220 5566 50  0000 C CNN
-F 2 "Connector_PinHeader_2.54mm:PinHeader_1x04_P2.54mm_Vertical" H 4300 5800 50  0001 C CNN
+F 2 "Connector_PinHeader_2.54mm:PinHeader_1x02_P2.54mm_Vertical" H 4300 5800 50  0001 C CNN
 F 3 "~" H 4300 5800 50  0001 C CNN
 	1    4300 5800
@@
 Wire Wire Line
 	4750 6250 4650 6250
+Wire Wire Line
+	7900 1050 8700 1050
+$Comp
+L Device:CP C88
+U 1 1 5ADECB62
+P 4700 1500
+F 0 "C88" H 4500 1500 50  0000 L CNN
+F 1 "100uF" H 4450 1400 50  0000 L CNN
+F 2 "Capacitor_SMD:CP_Elec_6.3x7.7" H 4738 1350 50  0001 C CNN
+F 3 "~" H 4700 1500 50  0001 C CNN
+	1    4700 1500
+	1    0    0    -1
+$EndComp
+Connection ~ 4700 1350
+Wire Wire Line
+	4700 1350 4100 1350
+$Comp
+L Device:C C89
+U 1 1 5ADECC47
+P 5050 1500
+F 0 "C89" H 5165 1546 50  0000 L CNN
+F 1 "0.001uF" H 5050 1400 50  0000 L CNN
+F 2 "Capacitor_SMD:C_0603_1608Metric" H 5088 1350 50  0001 C CNN
+F 3 "~" H 5050 1500 50  0001 C CNN
+	1    5050 1500
+	1    0    0    -1
+$EndComp
+Connection ~ 5050 1350
+Wire Wire Line
+	5050 1350 4700 1350
+Wire Wire Line
+	3850 1950 4700 1950
+Wire Wire Line
+	4700 1950 4700 1650
+Connection ~ 3850 1950
+Wire Wire Line
+	5050 1650 5050 1950
+Wire Wire Line
+	5050 1950 4700 1950
+Connection ~ 4700 1950
+$Comp
+L Mechanical:Mounting_Hole MK4
+U 1 1 5AE11BDF
+P 1000 1350
+F 0 "MK4" H 1100 1396 50  0000 L CNN
+F 1 "Mounting_Hole" H 1100 1305 50  0000 L CNN
+F 2 "MountingHole:MountingHole_3.2mm_M3" H 1000 1350 50  0001 C CNN
+F 3 "" H 1000 1350 50  0001 C CNN
+	1    1000 1350
+	1    0    0    -1
+$EndComp
+NoConn ~ 1000 1350
 $EndSCHEMATC

Commit message: Movet top FID to the top right corner. Added PCB origin. Switched 0.1uF 50V cpas to 0402 size.
Parts:
- J1, J2, J29, J4, J5, J6, J7, J8, J9: symbol Connector_Specialized:Screw_Terminal_01x02 -> PrntrBoardV1-rescue:Screw_Terminal_01x02-Connector_Specialized
Changed lines of the file:
@@
 $EndSheet
 $Comp
-L Connector_Specialized:Screw_Terminal_01x02 J2
+L PrntrBoardV1-rescue:Screw_Terminal_01x02-Connector_Specialized J2
 U 1 1 5AB8F2FF
 P 8100 4050
@@
 $EndSheet
 $Comp
-L Connector_Specialized:Screw_Terminal_01x02 J7
+L PrntrBoardV1-rescue:Screw_Terminal_01x02-Connector_Specialized J7
 U 1 1 5AB92C7F
 P 9400 3350
@@
 $EndComp
 $Comp
-L Connector_Specialized:Screw_Terminal_01x02 J6
+L PrntrBoardV1-rescue:Screw_Terminal_01x02-Connector_Specialized J6
 U 1 1 5AB92D01
 P 9400 2800
@@
 $EndComp
 $Comp
-L Connector_Specialized:Screw_Terminal_01x02 J5
+L PrntrBoardV1-rescue:Screw_Terminal_01x02-Connector_Specialized J5
 U 1 1 5AB92D3C
 P 9400 2200
@@
 $EndComp
 $Comp
-L Connector_Specialized:Screw_Terminal_01x02 J4
+L PrntrBoardV1-rescue:Screw_Terminal_01x02-Connector_Specialized J4
 U 1 1 5AB92D90
 P 9400 1650
@@
 	7150 5450 7150 5100
 $Comp
-L Connector_Specialized:Screw_Terminal_01x02 J8
+L PrntrBoardV1-rescue:Screw_Terminal_01x02-Connector_Specialized J8
 U 1 1 5AC9DA10
 P 10150 1650
@@
 $EndComp
 $Comp
-L Connector_Specialized:Screw_Terminal_01x02 J9
+L PrntrBoardV1-rescue:Screw_Terminal_01x02-Connector_Specialized J9
 U 1 1 5AC9DAC8
 P 10150 2050
@@
 Connection ~ 4100 2900
 $Comp
-L Connector_Specialized:Screw_Terminal_01x02 J29
+L PrntrBoardV1-rescue:Screw_Terminal_01x02-Connector_Specialized J29
 U 1 1 5ACB9063
 P 2350 900
@@
 NoConn ~ 1950 1400
 $Comp
-L Connector_Specialized:Screw_Terminal_01x02 J1
+L PrntrBoardV1-rescue:Screw_Terminal_01x02-Connector_Specialized J1
 U 1 1 5AEDA4A7
 P 3500 1950

Commit message: Updated TR3 foor print and re-routed tracks.
Parts:
- added JP8: Use VIn, Connector_PinHeader_2.54mm:PinHeader_1x02_P2.54mm_Vertical, symbol Jumper:Jumper_2_Open
- added JP9: Use USB, Connector_PinHeader_2.54mm:PinHeader_1x02_P2.54mm_Vertical, symbol Jumper:Jumper_2_Open
- C89: value 0.001uF -> 1000pF
Connections:
- wire segments 222 -> 228
- no-connect marks 33 -> 32
Changed lines of the file:
@@
 5V
 Wire Wire Line
-	5900 800  2550 800
+	5900 800  3350 800
 Connection ~ 5900 800
 $Comp
@@
 NoConn ~ 1750 4300
 NoConn ~ 3250 3200
-NoConn ~ 3250 3800
 NoConn ~ 1750 3000
 Wire Wire Line
@@
 	3700 1850 4100 1850
 Wire Wire Line
-	4100 1850 4100 2900
+	4100 1850 4100 2500
 Wire Wire Line
 	3850 2050 3850 1950
@@
 P 5050 1500
 F 0 "C89" H 5165 1546 50  0000 L CNN
-F 1 "0.001uF" H 5050 1400 50  0000 L CNN
+F 1 "1000pF" H 5050 1400 50  0000 L CNN
 F 2 "Capacitor_SMD:C_0603_1608Metric" H 5088 1350 50  0001 C CNN
 F 3 "~" H 5050 1500 50  0001 C CNN
@@
 $EndComp
 NoConn ~ 1000 1350
+$Comp
+L Jumper:Jumper_2_Open JP8
+U 1 1 5AF4F08D
+P 3350 1350
+F 0 "JP8" V 3304 1448 50  0000 L CNN
+F 1 "Use VIn" V 3395 1448 50  0000 L CNN
+F 2 "Connector_PinHeader_2.54mm:PinHeader_1x02_P2.54mm_Vertical" H 3350 1350 50  0001 C CNN
+F 3 "~" H 3350 1350 50  0001 C CNN
+	1    3350 1350
+	0    1    1    0
+$EndComp
+Wire Wire Line
+	3350 1150 3350 800
+Connection ~ 3350 800
+Wire Wire Line
+	3350 800  2550 800
+Wire Wire Line
+	3350 1550 3350 3800
+Wire Wire Line
+	3350 3800 3250 3800
+$Comp
+L Jumper:Jumper_2_Open JP9
+U 1 1 5AF74BAA
+P 3900 2500
+F 0 "JP9" H 4200 2500 50  0000 C CNN
+F 1 "Use USB" H 3900 2644 50  0000 C CNN
+F 2 "Connector_PinHeader_2.54mm:PinHeader_1x02_P2.54mm_Vertical" H 3900 2500 50  0001 C CNN
+F 3 "~" H 3900 2500 50  0001 C CNN
+	1    3900 2500
+	1    0    0    -1
+$EndComp
+Connection ~ 4100 2500
+Wire Wire Line
+	4100 2500 4100 2900
+Wire Wire Line
+	3700 2500 3450 2500
+Text Label 3500 2500 0    50   ~ 0
+VBUS
 $EndSCHEMATC

Commit message: Added 10k pullups to control inputs for heaters, to disable heaters when control module is not installed.
Parts:
- added R22, R23, R28, R29: 10k, Resistor_SMD:R_0603_1608Metric, symbol Device:R
Connections:
- wire segments 228 -> 236
Changed lines of the file:
@@
 Wire Wire Line
 	5150 2450 5150 2500
-Text Notes 4800 4750 0    50   ~ 0
+Text Notes 4250 4750 0    50   ~ 0
 Pin budget:\n17 GPIO out\n7 GPIO PWM out\n12 GPIO in\n3 ADC in\n1 SPI
 Wire Wire Line
@@
 Z_PROBE_MOD_BUF
 Wire Wire Line
-	5450 6850 4850 6850
+	5450 6850 4750 6850
 Text Label 5350 6850 2    50   ~ 0
 Z_PROBE_MOD
@@
 P 4400 6250
 F 0 "JP2" H 4250 6350 50  0000 C CNN
-F 1 "Motor Clock Select" H 4550 6050 50  0000 C CNN
+F 1 "Motor Clock Select" H 4350 6450 50  0000 C CNN
 F 2 "Jumper:SolderJumper-3_P1.3mm_Open_Pad1.0x1.5mm" H 4400 6250 50  0001 C CNN
 F 3 "~" H 4400 6250 50  0001 C CNN
@@
 Wire Wire Line
 	4400 6400 4400 6900
-Text Label 4400 6700 0    50   ~ 0
+Text Label 4400 6850 1    50   ~ 0
 MOT_CLOCK
 $Comp
@@
 Text Label 3500 2500 0    50   ~ 0
 VBUS
+$Comp
+L Device:R R29
+U 1 1 5AFAB4C8
+P 4900 4900
+F 0 "R29" H 4970 4946 50  0000 L CNN
+F 1 "10k" H 4970 4855 50  0000 L CNN
+F 2 "Resistor_SMD:R_0603_1608Metric" V 4830 4900 50  0001 C CNN
+F 3 "~" H 4900 4900 50  0001 C CNN
+	1    4900 4900
+	1    0    0    -1
+$EndComp
+$Comp
+L Device:R R23
+U 1 1 5AFAB5E3
+P 4850 5600
+F 0 "R23" H 4920 5646 50  0000 L CNN
+F 1 "10k" H 4920 5555 50  0000 L CNN
+F 2 "Resistor_SMD:R_0603_1608Metric" V 4780 5600 50  0001 C CNN
+F 3 "~" H 4850 5600 50  0001 C CNN
+	1    4850 5600
+	1    0    0    -1
+$EndComp
+$Comp
+L Device:R R28
+U 1 1 5AFAB683
+P 4850 6100
+F 0 "R28" H 4920 6146 50  0000 L CNN
+F 1 "10k" H 4920 6055 50  0000 L CNN
+F 2 "Resistor_SMD:R_0603_1608Metric" V 4780 6100 50  0001 C CNN
+F 3 "~" H 4850 6100 50  0001 C CNN
+	1    4850 6100
+	1    0    0    -1
+$EndComp
+$Comp
+L Device:R R22
+U 1 1 5AFAB73E
+P 4750 6650
+F 0 "R22" H 4820 6696 50  0000 L CNN
+F 1 "10k" H 4820 6605 50  0000 L CNN
+F 2 "Resistor_SMD:R_0603_1608Metric" V 4680 6650 50  0001 C CNN
+F 3 "~" H 4750 6650 50  0001 C CNN
+	1    4750 6650
+	1    0    0    -1
+$EndComp
+Wire Wire Line
+	4750 6800 4750 6850
+Wire Wire Line
+	4850 6250 4850 6350
+Wire Wire Line
+	4850 5750 4850 5850
+Wire Wire Line
+	4900 5050 4900 5100
+Wire Wire Line
+	4750 6500 4750 6350
+Wire Wire Line
+	4850 5950 5050 5950
+Wire Wire Line
+	4850 5450 4850 5250
+Wire Wire Line
+	4900 4750 4900 4550
+Text Label 4900 4650 0    50   ~ 0
+3.3V
+Text Label 4850 5350 0    50   ~ 0
+3.3V
+Text Label 4850 5950 0    50   ~ 0
+3.3V
+Text Label 4750 6450 0    50   ~ 0
+3.3V
 $EndSCHEMATC

Commit message: Some useless changes, I'll remove the SD_MODE wire soon.
Parts:
- added JP11: Use Ramp Generator, symbol Jumper:Jumper_2_Open
Connections:
- net labels added: SD_MODE
- wire segments 236 -> 240
Changed lines of the file:
@@
 F41 "5V" I L 6050 1350 50
 F42 "CLOCK" I L 6050 3400 50
+F43 "SD_MODE" I L 6050 2000 50
 $EndSheet
 $Comp
@@
 Text Label 4750 6450 0    50   ~ 0
 3.3V
+Wire Wire Line
+	6050 2000 5500 2000
+Text Label 5550 2000 0    50   ~ 0
+SD_MODE
+$Comp
+L Jumper:Jumper_2_Open JP11
+U 1 1 5AFFD02A
+P 8450 5850
+F 0 "JP11" V 8496 5948 50  0000 L CNN
+F 1 "Use Ramp Generator" V 8405 5948 50  0000 L CNN
+F 2 "" H 8450 5850 50  0001 C CNN
+F 3 "~" H 8450 5850 50  0001 C CNN
+	1    8450 5850
+	0    1    -1   0
+$EndComp
+Wire Wire Line
+	8450 6050 8450 6150
+Wire Wire Line
+	8450 6150 7650 6150
+Wire Wire Line
+	8450 5650 8450 5350
+Text Label 8450 5450 0    50   ~ 0
+SD_MODE
 $EndSCHEMATC

Commit message: Removed SD_MODE wire. Added motor clock oscillator. Wired the clock on the internal layer to reduce EMI.
Parts:
- removed J30: Ext Motor Clock, Connector_PinHeader_2.54mm:PinHeader_1x02_P2.54mm_Vertical, symbol Connector_Generic:Conn_01x02
- removed JP11: Use Ramp Generator, symbol Jumper:Jumper_2_Open
- removed JP2: Motor Clock Select, Jumper:SolderJumper-3_P1.3mm_Open_Pad1.0x1.5mm, symbol Jumper:Jumper_3_Bridged12
Connections:
- net labels removed: MOT_CLOCK, SD_MODE
- wire segments 240 -> 228
Changed lines of the file:
@@
 F40 "E1_PWM" I L 6050 2600 50
 F41 "5V" I L 6050 1350 50
-F42 "CLOCK" I L 6050 3400 50
-F43 "SD_MODE" I L 6050 2000 50
 $EndSheet
 $Comp
@@
 Connection ~ 4100 1850
 Wire Wire Line
-	6050 3400 5850 3400
-Wire Wire Line
-	5850 3400 5850 4050
-Text Label 5850 3950 0    50   ~ 0
-MOT_CLOCK
-$Comp
-L Jumper:Jumper_3_Bridged12 JP2
-U 1 1 5AE5CEDD
-P 4400 6250
-F 0 "JP2" H 4250 6350 50  0000 C CNN
-F 1 "Motor Clock Select" H 4350 6450 50  0000 C CNN
-F 2 "Jumper:SolderJumper-3_P1.3mm_Open_Pad1.0x1.5mm" H 4400 6250 50  0001 C CNN
-F 3 "~" H 4400 6250 50  0001 C CNN
-	1    4400 6250
-	1    0    0    -1
-$EndComp
-Wire Wire Line
-	3250 6250 4150 6250
-Wire Wire Line
-	4400 6400 4400 6900
-Text Label 4400 6850 1    50   ~ 0
-MOT_CLOCK
-$Comp
-L Connector_Generic:Conn_01x02 J30
-U 1 1 5AE7F628
-P 4300 5800
-F 0 "J30" H 4220 5475 50  0000 C CNN
-F 1 "Ext Motor Clock" H 4220 5566 50  0000 C CNN
-F 2 "Connector_PinHeader_2.54mm:PinHeader_1x02_P2.54mm_Vertical" H 4300 5800 50  0001 C CNN
-F 3 "~" H 4300 5800 50  0001 C CNN
-	1    4300 5800
-	-1   0    0    1
-$EndComp
-$Comp
-L power:GND #PWR086
-U 1 1 5AE7F7F3
-P 4500 5900
-F 0 "#PWR086" H 4500 5650 50  0001 C CNN
-F 1 "GND" H 4650 5800 50  0000 C CNN
-F 2 "" H 4500 5900 50  0001 C CNN
-F 3 "" H 4500 5900 50  0001 C CNN
-	1    4500 5900
-	1    0    0    -1
-$EndComp
-Wire Wire Line
-	4500 5800 4500 5900
-Wire Wire Line
-	4500 5700 4750 5700
-Wire Wire Line
-	4750 5700 4750 6250
-Wire Wire Line
-	4750 6250 4650 6250
-Wire Wire Line
 	7900 1050 8700 1050
 $Comp
@@
 Text Label 4750 6450 0    50   ~ 0
 3.3V
-Wire Wire Line
-	6050 2000 5500 2000
-Text Label 5550 2000 0    50   ~ 0
-SD_MODE
-$Comp
-L Jumper:Jumper_2_Open JP11
-U 1 1 5AFFD02A
-P 8450 5850
-F 0 "JP11" V 8496 5948 50  0000 L CNN
-F 1 "Use Ramp Generator" V 8405 5948 50  0000 L CNN
-F 2 "" H 8450 5850 50  0001 C CNN
-F 3 "~" H 8450 5850 50  0001 C CNN
-	1    8450 5850
-	0    1    -1   0
-$EndComp
-Wire Wire Line
-	8450 6050 8450 6150
-Wire Wire Line
-	8450 6150 7650 6150
-Wire Wire Line
-	8450 5650 8450 5350
-Text Label 8450 5450 0    50   ~ 0
-SD_MODE
 $EndSCHEMATC
