File: PrntrBoardV1.sch (KiCad schematic (older format))
At the start: 33 parts, among them J1 EXT 5V, J2 Bed Heater, J29 12-24V, J3 Z Probe, J4 E0 Cool, J5 E0 Part, J6 E1 Cool, J7 E1 Part, J8 Always On Fan 1, J9 Always On Fan 2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

Commit message: Added led on all power busses.
Parts:
- added D19, D20, D21, D22: LED, PrntrBoardV1:LED_0603_1608Metric, symbol Device:LED
- added R30, R31, R36: 10k, Resistor_SMD:R_0603_1608Metric, symbol Device:R
- added R37: 1k, Resistor_SMD:R_0603_1608Metric, symbol Device:R
Connections:
- wire segments 228 -> 240
Changed lines of the file:
@@
 P 10150 1650
 F 0 "J8" H 10229 1642 50  0000 L CNN
-F 1 "Always On Fan 1" H 10229 1551 50  0000 L CNN
+F 1 "Always On Fan 1" H 9900 1450 50  0000 L CNN
 F 2 "PrntrBoardV1:TerminalBlock_Phoenix_PT-1,5-2-3.5-H_1x02_P3.50mm_Horizontal" H 10150 1650 50  0001 C CNN
 F 3 "~" H 10150 1650 50  0001 C CNN
@@
 P 10150 2050
 F 0 "J9" H 10229 2042 50  0000 L CNN
-F 1 "Always On Fan 2" H 10229 1951 50  0000 L CNN
+F 1 "Always On Fan 2" H 9950 1850 50  0000 L CNN
 F 2 "PrntrBoardV1:TerminalBlock_Phoenix_PT-1,5-2-3.5-H_1x02_P3.50mm_Horizontal" H 10150 2050 50  0001 C CNN
 F 3 "~" H 10150 2050 50  0001 C CNN
@@
 	6400 4700 6400 5100
 Wire Wire Line
-	6400 5100 7150 5100
+	6400 5100 6750 5100
 Connection ~ 7150 5100
 Wire Wire Line
@@
 Connection ~ 4400 3400
 Wire Wire Line
-	4400 3400 4400 1250
+	4400 3400 4400 2750
 Connection ~ 4100 2900
 $Comp
@@
 U 1 1 5ADECB62
 P 4700 1500
-F 0 "C88" H 4500 1500 50  0000 L CNN
+F 0 "C88" H 4450 1550 50  0000 L CNN
 F 1 "100uF" H 4450 1400 50  0000 L CNN
 F 2 "Capacitor_SMD:CP_Elec_6.3x7.7" H 4738 1350 50  0001 C CNN
@@
 Wire Wire Line
 	5050 1350 4700 1350
-Wire Wire Line
-	3850 1950 4700 1950
 Wire Wire Line
 	4700 1950 4700 1650
@@
 Connection ~ 3350 800
 Wire Wire Line
-	3350 800  2550 800
+	3350 800  3000 800
 Wire Wire Line
 	3350 1550 3350 3800
@@
 Text Label 4750 6450 0    50   ~ 0
 3.3V
+$Comp
+L Device:LED D19
+U 1 1 5AF9C2B5
+P 3000 950
+F 0 "D19" V 3038 833 50  0000 R CNN
+F 1 "LED" V 2947 833 50  0000 R CNN
+F 2 "PrntrBoardV1:LED_0603_1608Metric" H 3000 950 50  0001 C CNN
+F 3 "~" H 3000 950 50  0001 C CNN
+	1    3000 950
+	0    -1   -1   0
+$EndComp
+Connection ~ 3000 800
+Wire Wire Line
+	3000 800  2550 800
+$Comp
+L Device:LED D21
+U 1 1 5AF9C4CA
+P 10750 1400
+F 0 "D21" V 10788 1283 50  0000 R CNN
+F 1 "LED" V 10697 1283 50  0000 R CNN
+F 2 "PrntrBoardV1:LED_0603_1608Metric" H 10750 1400 50  0001 C CNN
+F 3 "~" H 10750 1400 50  0001 C CNN
+	1    10750 1400
+	0    -1   -1   0
+$EndComp
+$Comp
+L Device:LED D20
+U 1 1 5AF9C705
+P 6750 5250
+F 0 "D20" V 6788 5133 50  0000 R CNN
+F 1 "LED" V 6697 5133 50  0000 R CNN
+F 2 "PrntrBoardV1:LED_0603_1608Metric" H 6750 5250 50  0001 C CNN
+F 3 "~" H 6750 5250 50  0001 C CNN
+	1    6750 5250
+	0    -1   -1   0
+$EndComp
+$Comp
+L Device:R R31
+U 1 1 5AF9C901
+P 6750 5600
+F 0 "R31" H 6820 5646 50  0000 L CNN
+F 1 "10k" H 6820 5555 50  0000 L CNN
+F 2 "Resistor_SMD:R_0603_1608Metric" V 6680 5600 50  0001 C CNN
+F 3 "~" H 6750 5600 50  0001 C CNN
+	1    6750 5600
+	1    0    0    -1
+$EndComp
+$Comp
+L Device:R R30
+U 1 1 5AF9C9AB
+P 3000 1300
+F 0 "R30" H 3070 1346 50  0000 L CNN
+F 1 "10k" H 3070 1255 50  0000 L CNN
+F 2 "Resistor_SMD:R_0603_1608Metric" V 2930 1300 50  0001 C CNN
+F 3 "~" H 3000 1300 50  0001 C CNN
+	1    3000 1300
+	1    0    0    -1
+$EndComp
+$Comp
+L Device:R R36
+U 1 1 5AF9CA87
+P 10750 1750
+F 0 "R36" H 10820 1796 50  0000 L CNN
+F 1 "10k" H 10820 1705 50  0000 L CNN
+F 2 "Resistor_SMD:R_0603_1608Metric" V 10680 1750 50  0001 C CNN
+F 3 "~" H 10750 1750 50  0001 C CNN
+	1    10750 1750
+	1    0    0    -1
+$EndComp
+Wire Wire Line
+	9850 1250 10750 1250
+Connection ~ 9850 1250
+Wire Wire Line
+	10750 1550 10750 1600
+Wire Wire Line
+	3000 1100 3000 1150
+Wire Wire Line
+	6750 5400 6750 5450
+$Comp
+L power:GND #PWR087
+U 1 1 5AFEB104
+P 6750 5800
+F 0 "#PWR087" H 6750 5550 50  0001 C CNN
+F 1 "GND" H 6755 5627 50  0000 C CNN
+F 2 "" H 6750 5800 50  0001 C CNN
+F 3 "" H 6750 5800 50  0001 C CNN
+	1    6750 5800
+	1    0    0    -1
+$EndComp
+$Comp
+L power:GND #PWR086
+U 1 1 5AFEB1AA
+P 3000 1500
+F 0 "#PWR086" H 3000 1250 50  0001 C CNN
+F 1 "GND" H 3005 1327 50  0000 C CNN
+F 2 "" H 3000 1500 50  0001 C CNN
+F 3 "" H 3000 1500 50  0001 C CNN
+	1    3000 1500
+	1    0    0    -1
+$EndComp
+$Comp
+L power:GND #PWR088
+U 1 1 5AFEB250
+P 10750 1950
+F 0 "#PWR088" H 10750 1700 50  0001 C CNN
+F 1 "GND" H 10755 1777 50  0000 C CNN
+F 2 "" H 10750 1950 50  0001 C CNN
+F 3 "" H 10750 1950 50  0001 C CNN
+	1    10750 1950
+	1    0    0    -1
+$EndComp
+Wire Wire Line
+	10750 1900 10750 1950
+Wire Wire Line
+	6750 5750 6750 5800
+Wire Wire Line
+	3000 1450 3000 1500
+Connection ~ 6750 5100
+Wire Wire Line
+	6750 5100 7150 5100
+Wire Wire Line
+	3850 1950 4700 1950
+$Comp
+L Device:R R37
+U 1 1 5B04FD2D
+P 4700 2350
+F 0 "R37" H 4500 2450 50  0000 L CNN
+F 1 "1k" H 4550 2350 50  0000 L CNN
+F 2 "Resistor_SMD:R_0603_1608Metric" V 4630 2350 50  0001 C CNN
+F 3 "~" H 4700 2350 50  0001 C CNN
+	1    4700 2350
+	1    0    0    -1
+$EndComp
+$Comp
+L Device:LED D22
+U 1 1 5B04FE03
+P 4550 2750
+F 0 "D22" H 4542 2495 50  0000 C CNN
+F 1 "LED" H 4542 2586 50  0000 C CNN
+F 2 "PrntrBoardV1:LED_0603_1608Metric" H 4550 2750 50  0001 C CNN
+F 3 "~" H 4550 2750 50  0001 C CNN
+	1    4550 2750
+	-1   0    0    1
+$EndComp
+Connection ~ 4400 2750
+Wire Wire Line
+	4400 2750 4400 1250
+Wire Wire Line
+	4700 2750 4700 2500
+Wire Wire Line
+	4700 2200 4700 1950
 $EndSCHEMATC

Commit message: Added LCD screen. Updated REDME.
Connections:
- net labels added: LCD_A0, MOSI_BUF, SCK_BUF, ~LCD_CS, ~LCD_RESET
- wire segments 240 -> 256
- no-connect marks 32 -> 30
Changed lines of the file:
@@
 $Descr A4 11693 8268
 encoding utf-8
-Sheet 1 34
+Sheet 1 35
 Title ""
 Date ""
@@
 F30 "E0_SG" O L 6050 3150 50
 F31 "E0_FLMT" O R 7350 3000 50
-F32 "E0_TEMP" O L 6050 2150 50
+F32 "E0_TEMP" O L 6050 2250 50
 F33 "E0_PWM" I L 6050 2500 50
 F34 "E1_STEP" I R 7350 1450 50
@@
 F37 "E1_SG" O L 6050 3250 50
 F38 "E1_FLMT" O R 7350 3100 50
-F39 "E1_TEMP" O L 6050 2250 50
+F39 "E1_TEMP" O L 6050 2350 50
 F40 "E1_PWM" I L 6050 2600 50
 F41 "5V" I L 6050 1350 50
+F42 "MOSI_BUF" O L 6050 2000 50
+F43 "SCK_BUF" O L 6050 2100 50
 $EndSheet
 $Comp
@@
 	6050 1900 5600 1900
 Wire Wire Line
-	6050 2150 5600 2150
-Wire Wire Line
-	6050 2250 5600 2250
-Wire Wire Line
 	6600 4300 6050 4300
 Text Label 6150 4300 0    50   ~ 0
 BED_TEMP
-Text Label 5650 2150 0    50   ~ 0
+Text Label 5650 2250 0    50   ~ 0
 E0_TEMP
-Text Label 5650 2250 0    50   ~ 0
+Text Label 5650 2350 0    50   ~ 0
 E1_TEMP
 Text Label 5500 1500 0    50   ~ 0
@@
 Wire Wire Line
 	3850 1950 3700 1950
-NoConn ~ 1750 3900
-NoConn ~ 1750 4000
 $Comp
 L Mechanical:Mounting_Hole MK1
@@
 Wire Wire Line
 	4700 2200 4700 1950
+$Sheet
+S 10000 3650 950  1200
+U 5AFA5DB1
+F0 "LCD Display" 50
+F1 "ST7735 LCD.sch" 50
+F2 "SDA" I L 10000 3800 50
+F3 "SCL" I L 10000 3900 50
+F4 "A0" I L 10000 4000 50
+F5 "~RESET" I L 10000 4100 50
+F6 "3.3V" I L 10000 4350 50
+F7 "LED+" I L 10000 4500 50
+F8 "LED-" I L 10000 4650 50
+F9 "~CS" I L 10000 4200 50
+$EndSheet
+$Comp
+L power:GND #PWR089
+U 1 1 5AFBABF4
+P 9800 4700
+F 0 "#PWR089" H 9800 4450 50  0001 C CNN
+F 1 "GND" H 9805 4527 50  0000 C CNN
+F 2 "" H 9800 4700 50  0001 C CNN
+F 3 "" H 9800 4700 50  0001 C CNN
+	1    9800 4700
+	1    0    0    -1
+$EndComp
+Wire Wire Line
+	9800 4700 9800 4650
+Wire Wire Line
+	9800 4650 10000 4650
+Wire Wire Line
+	10000 4500 9750 4500
+Wire Wire Line
+	9750 4500 9750 4350
+Wire Wire Line
+	9750 4350 10000 4350
+Wire Wire Line
+	9750 4350 9400 4350
+Connection ~ 9750 4350
+Text Label 9450 4350 0    50   ~ 0
+3.3V
+Wire Wire Line
+	10000 3800 9400 3800
+Wire Wire Line
+	10000 3900 9400 3900
+Wire Wire Line
+	10000 4000 9400 4000
+Wire Wire Line
+	10000 4100 9400 4100
+Text Label 9450 4100 0    50   ~ 0
+~LCD_RESET
+Text Label 9450 4000 0    50   ~ 0
+LCD_A0
+Text Label 9450 3900 0    50   ~ 0
+SCK_BUF
+Text Label 9450 3800 0    50   ~ 0
+MOSI_BUF
+Wire Wire Line
+	3250 6250 3950 6250
+Text Label 3900 6250 2    50   ~ 0
+~LCD_RESET
+Wire Wire Line
+	1750 3900 1000 3900
+Text Label 1050 3900 0    50   ~ 0
+LCD_A0
+Wire Wire Line
+	10000 4200 9400 4200
+Text Label 9450 4200 0    50   ~ 0
+~LCD_CS
+Wire Wire Line
+	1750 4000 1000 4000
+Text Label 1050 4000 0    50   ~ 0
+~LCD_CS
+Wire Wire Line
+	6050 2350 5600 2350
+Wire Wire Line
+	6050 2250 5600 2250
+Wire Wire Line
+	6050 2000 5600 2000
+Wire Wire Line
+	6050 2100 5600 2100
+Text Label 5650 2000 0    50   ~ 0
+MOSI_BUF
+Text Label 5650 2100 0    50   ~ 0
+SCK_BUF
 $EndSCHEMATC

Commit message: Change the LCD power to 5V, keep the 3.3V only for the backlight LED.
Connections:
- wire segments 256 -> 254
Changed lines of the file:
@@
 F4 "A0" I L 10000 4000 50
 F5 "~RESET" I L 10000 4100 50
-F6 "3.3V" I L 10000 4350 50
-F7 "LED+" I L 10000 4500 50
-F8 "LED-" I L 10000 4650 50
-F9 "~CS" I L 10000 4200 50
+F6 "LED+" I L 10000 4500 50
+F7 "LED-" I L 10000 4650 50
+F8 "~CS" I L 10000 4200 50
+F9 "VCC" I L 10000 4300 50
 $EndSheet
 $Comp
@@
 Wire Wire Line
 	9800 4650 10000 4650
-Wire Wire Line
-	10000 4500 9750 4500
-Wire Wire Line
-	9750 4500 9750 4350
-Wire Wire Line
-	9750 4350 10000 4350
-Wire Wire Line
-	9750 4350 9400 4350
-Connection ~ 9750 4350
-Text Label 9450 4350 0    50   ~ 0
+Text Label 9450 4500 0    50   ~ 0
 3.3V
 Wire Wire Line
@@
 Text Label 5650 2100 0    50   ~ 0
 SCK_BUF
+Wire Wire Line
+	9400 4500 10000 4500
+Wire Wire Line
+	10000 4300 9400 4300
+Text Label 9450 4300 0    50   ~ 0
+5V
 $EndSCHEMATC

Commit message: Added dual themocouple pins. You'll have to sacrifice the controllable extruder cooling fans via jumpers.
Parts:
- added J31: TC1, Connector_PinHeader_2.54mm:PinHeader_1x06_P2.54mm_Vertical, symbol Connector_Generic:Conn_01x06
- added J32: TC2, Connector_PinHeader_2.54mm:PinHeader_1x06_P2.54mm_Vertical, symbol Connector_Generic:Conn_01x06
- added JP2: E1_TC2, Connector_PinHeader_2.54mm:PinHeader_1x03_P2.54mm_Vertical, symbol Jumper:Jumper_3_Bridged12
- added JP3: E0_TC1, Connector_PinHeader_2.54mm:PinHeader_1x03_P2.54mm_Vertical, symbol Jumper:Jumper_3_Bridged12
Connections:
- net labels added: E0_COOL_TC1, E1_COOL_TC2, ~TC1_CS, ~TC2_CS
- wire segments 254 -> 290
Changed lines of the file:
@@
 	1750 6150 1000 6150
-Wire Wire Line
-	1750 6250 1000 6250
 Wire Wire Line
 	1750 6350 1000 6350
@@
 Text Label 3650 5350 0    50   ~ 0
 Y_STEP
-Text Label 3450 5250 0    50   ~ 0
+Text Label 3600 4850 0    50   ~ 0
 E0_COOL_PWM
 Text Label 1050 5650 0    50   ~ 0
@@
 Text Label 1050 6150 0    50   ~ 0
 E1_DIR
-Text Label 1050 6250 0    50   ~ 0
-E1_COOL_PWM
 Text Label 1050 6350 0    50   ~ 0
 SCK
@@
 	3400 3700 3400 6050
 Wire Wire Line
-	3250 5250 3950 5250
-Wire Wire Line
 	3250 3400 4400 3400
 Connection ~ 4400 3400
@@
 Text Label 9450 4300 0    50   ~ 0
 5V
+$Comp
+L Connector_Generic:Conn_01x06 J31
+U 1 1 5B0DCBB0
+P 10400 6000
+F 0 "J31" H 10450 5950 50  0000 L CNN
+F 1 "TC1" H 10350 6550 50  0000 L CNN
+F 2 "Connector_PinHeader_2.54mm:PinHeader_1x06_P2.54mm_Vertical" H 10400 6000 50  0001 C CNN
+F 3 "~" H 10400 6000 50  0001 C CNN
+	1    10400 6000
+	1    0    0    -1
+$EndComp
+$Comp
+L Connector_Generic:Conn_01x06 J32
+U 1 1 5B0DCCBB
+P 10900 6000
+F 0 "J32" H 10950 5950 50  0000 L CNN
+F 1 "TC2" H 10850 6550 50  0000 L CNN
+F 2 "Connector_PinHeader_2.54mm:PinHeader_1x06_P2.54mm_Vertical" H 10900 6000 50  0001 C CNN
+F 3 "~" H 10900 6000 50  0001 C CNN
+	1    10900 6000
+	1    0    0    -1
+$EndComp
+Wire Wire Line
+	10700 6000 10600 6000
+Wire Wire Line
+	10600 6000 10600 5700
+Wire Wire Line
+	10600 5700 10100 5700
+Wire Wire Line
+	10100 5700 10100 6000
+Wire Wire Line
+	10100 6000 10200 6000
+Wire Wire Line
+	10700 5900 10650 5900
+Wire Wire Line
+	10650 5900 10650 5650
+Wire Wire Line
+	10650 5650 10150 5650
+Wire Wire Line
+	10150 5650 10150 5900
+Wire Wire Line
+	10150 5900 10200 5900
+Wire Wire Line
+	10700 5800 10700 5600
+Wire Wire Line
+	10700 5600 10200 5600
+Wire Wire Line
+	10200 5600 10200 5800
+Wire Wire Line
+	10700 6100 10600 6100
+Wire Wire Line
+	10600 6100 10600 6400
+Wire Wire Line
+	10600 6400 10100 6400
+Wire Wire Line
+	10100 6400 10100 6100
+Wire Wire Line
+	10100 6100 10200 6100
+Wire Wire Line
+	10700 6200 10650 6200
+Wire Wire Line
+	10650 6200 10650 6450
+Wire Wire Line
+	10650 6450 10150 6450
+Wire Wire Line
+	10150 6450 10150 6200
+Wire Wire Line
+	10150 6200 10200 6200
+Wire Wire Line
+	10700 6300 10700 6500
+Text Label 10350 5600 0    50   ~ 0
+5V
+$Comp
+L power:GND #PWR091
+U 1 1 5B1853F1
+P 11050 5650
+F 0 "#PWR091" H 11050 5400 50  0001 C CNN
+F 1 "GND" H 11055 5477 50  0000 C CNN
+F 2 "" H 11050 5650 50  0001 C CNN
+F 3 "" H 11050 5650 50  0001 C CNN
+	1    11050 5650
+	1    0    0    -1
+$EndComp
+Wire Wire Line
+	10650 5650 11050 5650
+Connection ~ 10650 5650
+Wire Wire Line
+	10100 6000 9650 6000
+Connection ~ 10100 6000
+Wire Wire Line
+	10100 6100 9650 6100
+Connection ~ 10100 6100
+Wire Wire Line
+	10150 6200 9650 6200
+Connection ~ 10150 6200
+Wire Wire Line
+	10200 6300 9650 6300
+Wire Wire Line
+	9650 6500 10700 6500
+Text Label 9650 6000 0    50   ~ 0
+SCK_BUF
+Text Label 9650 6100 0    50   ~ 0
+MOSI_BUF
+Text Label 9650 6200 0    50   ~ 0
+MISO
+Text Label 9650 6300 0    50   ~ 0
+~TC1_CS
+Text Label 9650 6500 0    50   ~ 0
+~TC2_CS
+$Comp
+L Jumper:Jumper_3_Bridged12 JP3
+U 1 1 5B24639E
+P 4200 5250
+F 0 "JP3" V 4154 5317 50  0000 L CNN
+F 1 "E0_TC1" V 4245 5317 50  0000 L CNN
+F 2 "Connector_PinHeader_2.54mm:PinHeader_1x03_P2.54mm_Vertical" H 4200 5250 50  0001 C CNN
+F 3 "~" H 4200 5250 50  0001 C CNN
+	1    4200 5250
+	0    1    1    0
+$EndComp
+$Comp
+L Jumper:Jumper_3_Bridged12 JP2
+U 1 1 5B2464D1
+P 750 6250
+F 0 "JP2" V 796 6316 50  0000 L CNN
+F 1 "E1_TC2" H 300 6350 50  0000 L CNN
+F 2 "Connector_PinHeader_2.54mm:PinHeader_1x03_P2.54mm_Vertical" H 750 6250 50  0001 C CNN
+F 3 "~" H 750 6250 50  0001 C CNN
+	1    750  6250
+	0    -1   -1   0
+$EndComp
+Text Label 900  7200 0    50   ~ 0
+E1_COOL_PWM
+Wire Wire Line
+	750  6500 750  7200
+Wire Wire Line
+	750  7200 1450 7200
+Wire Wire Line
+	900  6250 1750 6250
+Wire Wire Line
+	750  6000 750  5650
+Text Label 750  6000 1    50   ~ 0
+~TC2_CS
+Wire Wire Line
+	4200 5000 4200 4850
+Wire Wire Line
+	4200 4850 3500 4850
+Wire Wire Line
+	3250 5250 4050 5250
+Wire Wire Line
+	4200 5500 4200 5850
+Text Label 4200 5550 3    50   ~ 0
+~TC1_CS
+Text Label 1000 6250 0    50   ~ 0
+E1_COOL_TC2
+Text Label 3450 5250 0    50   ~ 0
+E0_COOL_TC1
 $EndSCHEMATC

Commit message: Updated schematics with the latest features.
Connections:
- wire segments 290 -> 289
Changed lines of the file:
@@
 F39 "E1_TEMP" O L 6050 2350 50
 F40 "E1_PWM" I L 6050 2600 50
-F41 "5V" I L 6050 1350 50
-F42 "MOSI_BUF" O L 6050 2000 50
-F43 "SCK_BUF" O L 6050 2100 50
+F41 "MOSI_BUF" O L 6050 2000 50
+F42 "SCK_BUF" O L 6050 2100 50
 $EndSheet
 $Comp
@@
 $EndComp
 Wire Wire Line
-	6050 1350 5050 1350
-Wire Wire Line
 	4100 1350 4100 1850
 Connection ~ 4100 1850
@@
 	1    0    0    -1
 $EndComp
-Connection ~ 5050 1350
 Wire Wire Line
 	5050 1350 4700 1350

Commit message: Updated the README.md file. Added filtering caps on the 3.3v input as well as the AVREF input.
Updated the board 3D rendering.
Parts:
- added C78, C79: 10uF 10V, Capacitor_SMD:C_0603_1608Metric, symbol Device:C
Connections:
- wire segments 289 -> 291
Changed lines of the file:
@@
 	3400 3700 3400 6050
 Wire Wire Line
-	3250 3400 4400 3400
+	3250 3400 3800 3400
 Connection ~ 4400 3400
 Wire Wire Line
@@
 Text Label 3450 5250 0    50   ~ 0
 E0_COOL_TC1
+$Comp
+L Device:C C78
+U 1 1 5B2D178A
+P 3800 3550
+F 0 "C78" H 3915 3596 50  0000 L CNN
+F 1 "10uF 10V" H 3915 3505 50  0000 L CNN
+F 2 "Capacitor_SMD:C_0603_1608Metric" H 3838 3400 50  0001 C CNN
+F 3 "~" H 3800 3550 50  0001 C CNN
+	1    3800 3550
+	1    0    0    -1
+$EndComp
+Connection ~ 3800 3400
+Wire Wire Line
+	3800 3400 4400 3400
+$Comp
+L power:GND #PWR076
+U 1 1 5B2D196F
+P 3800 3750
+F 0 "#PWR076" H 3800 3500 50  0001 C CNN
+F 1 "GND" H 3950 3700 50  0000 C CNN
+F 2 "" H 3800 3750 50  0001 C CNN
+F 3 "" H 3800 3750 50  0001 C CNN
+	1    3800 3750
+	1    0    0    -1
+$EndComp
+Wire Wire Line
+	3800 3750 3800 3700
+$Comp
+L Device:C C79
+U 1 1 5B2ECF11
+P 5950 3900
+F 0 "C79" H 6065 3946 50  0000 L CNN
+F 1 "10uF 10V" H 6065 3855 50  0000 L CNN
+F 2 "Capacitor_SMD:C_0603_1608Metric" H 5988 3750 50  0001 C CNN
+F 3 "~" H 5950 3900 50  0001 C CNN
+	1    5950 3900
+	1    0    0    -1
+$EndComp
+Connection ~ 5950 3750
+$Comp
+L power:GND #PWR077
+U 1 1 5B2ECFE1
+P 5950 4050
+F 0 "#PWR077" H 5950 3800 50  0001 C CNN
+F 1 "GND" H 5955 3877 50  0000 C CNN
+F 2 "" H 5950 4050 50  0001 C CNN
+F 3 "" H 5950 4050 50  0001 C CNN
+	1    5950 4050
+	1    0    0    -1
+$EndComp
 $EndSCHEMATC

Commit message: Cleanup paths and library names.
Parts:
- U2: symbol Logic_74xx:74HCT02 -> 74ls02:74HCT02
Changed lines of the file:
@@
 5V
 $Comp
-L Logic_74xx:74HCT02 U2
+L 74ls02:74HCT02 U2
 U 1 1 5AB9C30F
 P 5750 6750
@@
 $EndComp
 $Comp
-L Logic_74xx:74HCT02 U2
+L 74ls02:74HCT02 U2
 U 2 1 5AB9E04D
 P 5750 5200
@@
 $EndComp
 $Comp
-L Logic_74xx:74HCT02 U2
+L 74ls02:74HCT02 U2
 U 3 1 5AB9E0C5
 P 5750 5750
@@
 $EndComp
 $Comp
-L Logic_74xx:74HCT02 U2
+L 74ls02:74HCT02 U2
 U 4 1 5AB9E15A
 P 5750 6250
@@
 $EndComp
 $Comp
-L Logic_74xx:74HCT02 U2
+L 74ls02:74HCT02 U2
 U 5 1 5AB9E1C8
 P 7650 5600

Commit message: Add more filtering caps.
Parts:
- added C80: 1000pF, Capacitor_SMD:C_0603_1608Metric, symbol Device:C
Connections:
- wire segments 291 -> 295
Changed lines of the file:
@@
 L Device:C C2
 U 1 1 5ABB120D
-P 7150 5600
-F 0 "C2" H 7265 5646 50  0000 L CNN
-F 1 "0.1uF" H 7265 5555 50  0000 L CNN
-F 2 "Capacitor_SMD:C_0603_1608Metric" H 7188 5450 50  0001 C CNN
-F 3 "~" H 7150 5600 50  0001 C CNN
-	1    7150 5600
-	1    0    0    -1
-$EndComp
-Wire Wire Line
-	7150 5750 7150 6150
-Wire Wire Line
-	7150 6150 7650 6150
+P 7200 5600
+F 0 "C2" H 7250 5500 50  0000 L CNN
+F 1 "0.1uF" H 7200 5400 50  0000 L CNN
+F 2 "Capacitor_SMD:C_0603_1608Metric" H 7238 5450 50  0001 C CNN
+F 3 "~" H 7200 5600 50  0001 C CNN
+	1    7200 5600
+	1    0    0    -1
+$EndComp
+Wire Wire Line
+	7200 5750 7200 6150
+Wire Wire Line
+	7200 6150 7650 6150
 Connection ~ 7650 6150
 Wire Wire Line
 	7650 6150 7650 6200
 Wire Wire Line
-	7150 5450 7150 5100
+	7200 5450 7200 5100
 $Comp
 L PrntrBoardV1-rescue:Screw_Terminal_01x02-Connector_Specialized J8
@@
 E0_COOL_PWM
 Wire Wire Line
-	7150 5100 7650 5100
+	7200 5100 7650 5100
 Wire Wire Line
 	7350 1050 7800 1050
@@
 	6400 4700 6400 5100
 Wire Wire Line
-	6400 5100 6750 5100
-Connection ~ 7150 5100
+	6400 5100 6600 5100
+Connection ~ 7200 5100
 Wire Wire Line
 	3400 6050 3400 6650
@@
 L Device:LED D20
 U 1 1 5AF9C705
-P 6750 5250
-F 0 "D20" V 6788 5133 50  0000 R CNN
-F 1 "LED" V 6697 5133 50  0000 R CNN
-F 2 "PrntrBoardV1:LED_0603_1608Metric" H 6750 5250 50  0001 C CNN
-F 3 "~" H 6750 5250 50  0001 C CNN
-	1    6750 5250
+P 6600 5250
+F 0 "D20" V 6638 5133 50  0000 R CNN
+F 1 "LED" V 6547 5133 50  0000 R CNN
+F 2 "PrntrBoardV1:LED_0603_1608Metric" H 6600 5250 50  0001 C CNN
+F 3 "~" H 6600 5250 50  0001 C CNN
+	1    6600 5250
 	0    -1   -1   0
 $EndComp
@@
 L Device:R R31
 U 1 1 5AF9C901
-P 6750 5600
-F 0 "R31" H 6820 5646 50  0000 L CNN
-F 1 "10k" H 6820 5555 50  0000 L CNN
-F 2 "Resistor_SMD:R_0603_1608Metric" V 6680 5600 50  0001 C CNN
-F 3 "~" H 6750 5600 50  0001 C CNN
-	1    6750 5600
+P 6600 5600
+F 0 "R31" H 6670 5646 50  0000 L CNN
+F 1 "10k" H 6670 5555 50  0000 L CNN
+F 2 "Resistor_SMD:R_0603_1608Metric" V 6530 5600 50  0001 C CNN
+F 3 "~" H 6600 5600 50  0001 C CNN
+	1    6600 5600
 	1    0    0    -1
 $EndComp
@@
 	3000 1100 3000 1150
 Wire Wire Line
-	6750 5400 6750 5450
+	6600 5400 6600 5450
 $Comp
 L power:GND #PWR087
 U 1 1 5AFEB104
-P 6750 5800
-F 0 "#PWR087" H 6750 5550 50  0001 C CNN
-F 1 "GND" H 6755 5627 50  0000 C CNN
-F 2 "" H 6750 5800 50  0001 C CNN
-F 3 "" H 6750 5800 50  0001 C CNN
-	1    6750 5800
+P 6600 5800
+F 0 "#PWR087" H 6600 5550 50  0001 C CNN
+F 1 "GND" H 6605 5627 50  0000 C CNN
+F 2 "" H 6600 5800 50  0001 C CNN
+F 3 "" H 6600 5800 50  0001 C CNN
+	1    6600 5800
 	1    0    0    -1
 $EndComp
@@
 	10750 1900 10750 1950
 Wire Wire Line
-	6750 5750 6750 5800
+	6600 5750 6600 5800
 Wire Wire Line
 	3000 1450 3000 1500
-Connection ~ 6750 5100
-Wire Wire Line
-	6750 5100 7150 5100
 Wire Wire Line
 	3850 1950 4700 1950
@@
 	1    0    0    -1
 $EndComp
+Connection ~ 6600 5100
+Wire Wire Line
+	6600 5100 6950 5100
+$Comp
+L Device:C C80
+U 1 1 5B36B308
+P 6950 5600
+F 0 "C80" H 7000 5500 50  0000 L CNN
+F 1 "1000pF" H 6650 5400 50  0000 L CNN
+F 2 "Capacitor_SMD:C_0603_1608Metric" H 6988 5450 50  0001 C CNN
+F 3 "~" H 6950 5600 50  0001 C CNN
+	1    6950 5600
+	1    0    0    -1
+$EndComp
+Wire Wire Line
+	6950 5750 6950 6150
+Wire Wire Line
+	6950 6150 7200 6150
+Connection ~ 7200 6150
+Wire Wire Line
+	6950 5450 6950 5100
+Connection ~ 6950 5100
+Wire Wire Line
+	6950 5100 7200 5100
 $EndSCHEMATC
