File: PrntrBoardV1.sch (KiCad schematic (older format))
At the start: 48 parts, among them J1 EXT 5V, J2 Bed Heater, J29 12-24V, J3 Z Probe, J31 TC1, J32 TC2, J4 E0 Cool, J5 E0 Part, J6 E1 Cool, J7 E1 Part, J8 Always On Fan 1, J9 Always On Fan 2, U1 4078, U11 NUCLEO-64, U2 74HCT02

Commit message: Carry over schematics updates from 2130 branch:   - fix z stop input resistor   - add extra fan connectors
Parts:
- added J33: XF1, Connector_PinHeader_2.54mm:PinHeader_1x02_P2.54mm_Vertical, symbol Connector_Generic:Conn_01x02
- added J34: XF2, Connector_PinHeader_2.54mm:PinHeader_1x02_P2.54mm_Vertical, symbol Connector_Generic:Conn_01x02
- added J35: XF3, Connector_PinHeader_2.54mm:PinHeader_1x02_P2.54mm_Vertical, symbol Connector_Generic:Conn_01x02
- added J36: XF4, Connector_PinHeader_2.54mm:PinHeader_1x02_P2.54mm_Vertical, symbol Connector_Generic:Conn_01x02
- R1: value 10k -> 1k
Connections:
- wire segments 295 -> 310
Changed lines of the file:
@@
 5V
 Wire Wire Line
-	5900 800  3350 800
+	5900 800  4100 800
 Connection ~ 5900 800
 $Comp
@@
 P 9050 5200
 F 0 "R1" V 9150 5150 50  0000 C CNN
-F 1 "10k" V 9150 5300 50  0000 C CNN
+F 1 "1k" V 9150 5300 50  0000 C CNN
 F 2 "Resistor_SMD:R_0603_1608Metric" V 8980 5200 50  0001 C CNN
 F 3 "~" H 9050 5200 50  0001 C CNN
@@
 	4100 2900 4100 4150
 Wire Wire Line
-	4100 4150 5850 4150
+	4100 4150 5050 4150
 Wire Wire Line
 	5850 4150 5850 4700
@@
 U 1 1 5AF4F08D
 P 3350 1350
-F 0 "JP8" V 3304 1448 50  0000 L CNN
-F 1 "Use VIn" V 3395 1448 50  0000 L CNN
+F 0 "JP8" V 3400 1450 50  0000 L CNN
+F 1 "Use VIn" V 3500 1450 50  0000 L CNN
 F 2 "Connector_PinHeader_2.54mm:PinHeader_1x02_P2.54mm_Vertical" H 3350 1350 50  0001 C CNN
 F 3 "~" H 3350 1350 50  0001 C CNN
@@
 Wire Wire Line
 	6950 5100 7200 5100
+$Comp
+L Connector_Generic:Conn_01x02 J33
+U 1 1 5B5B23D5
+P 3850 1000
+F 0 "J33" H 3929 992 50  0000 L CNN
+F 1 "XF1" H 3929 901 50  0000 L CNN
+F 2 "Connector_PinHeader_2.54mm:PinHeader_1x02_P2.54mm_Vertical" H 3850 1000 50  0001 C CNN
+F 3 "~" H 3850 1000 50  0001 C CNN
+	1    3850 1000
+	1    0    0    -1
+$EndComp
+$Comp
+L Connector_Generic:Conn_01x02 J34
+U 1 1 5B5B249F
+P 4300 1000
+F 0 "J34" H 4379 992 50  0000 L CNN
+F 1 "XF2" H 4379 901 50  0000 L CNN
+F 2 "Connector_PinHeader_2.54mm:PinHeader_1x02_P2.54mm_Vertical" H 4300 1000 50  0001 C CNN
+F 3 "~" H 4300 1000 50  0001 C CNN
+	1    4300 1000
+	1    0    0    -1
+$EndComp
+Wire Wire Line
+	3650 1000 3650 800
+Connection ~ 3650 800
+Wire Wire Line
+	3650 800  3350 800
+Wire Wire Line
+	4100 1000 4100 800
+Connection ~ 4100 800
+Wire Wire Line
+	4100 800  3650 800
+Wire Wire Line
+	4100 1100 4100 1200
+Wire Wire Line
+	4100 1200 3650 1200
+Wire Wire Line
+	3650 1200 3650 1100
+$Comp
+L power:GND #PWR078
+U 1 1 5B623979
+P 3650 1200
+F 0 "#PWR078" H 3650 950 50  0001 C CNN
+F 1 "GND" H 3800 1150 50  0000 C CNN
+F 2 "" H 3650 1200 50  0001 C CNN
+F 3 "" H 3650 1200 50  0001 C CNN
+	1    3650 1200
+	1    0    0    -1
+$EndComp
+Connection ~ 3650 1200
+$Comp
+L Connector_Generic:Conn_01x02 J35
+U 1 1 5B6240A6
+P 5250 4250
+F 0 "J35" H 4850 4150 50  0000 L CNN
+F 1 "XF3" H 4850 4250 50  0000 L CNN
+F 2 "Connector_PinHeader_2.54mm:PinHeader_1x02_P2.54mm_Vertical" H 5250 4250 50  0001 C CNN
+F 3 "~" H 5250 4250 50  0001 C CNN
+	1    5250 4250
+	1    0    0    -1
+$EndComp
+$Comp
+L Connector_Generic:Conn_01x02 J36
+U 1 1 5B62417C
+P 5650 4250
+F 0 "J36" H 5700 4150 50  0000 L CNN
+F 1 "XF4" H 5650 4050 50  0000 L CNN
+F 2 "Connector_PinHeader_2.54mm:PinHeader_1x02_P2.54mm_Vertical" H 5650 4250 50  0001 C CNN
+F 3 "~" H 5650 4250 50  0001 C CNN
+	1    5650 4250
+	1    0    0    -1
+$EndComp
+$Comp
+L power:GND #PWR079
+U 1 1 5B624259
+P 5350 4500
+F 0 "#PWR079" H 5350 4250 50  0001 C CNN
+F 1 "GND" H 5355 4327 50  0000 C CNN
+F 2 "" H 5350 4500 50  0001 C CNN
+F 3 "" H 5350 4500 50  0001 C CNN
+	1    5350 4500
+	1    0    0    -1
+$EndComp
+Wire Wire Line
+	5450 4250 5450 4150
+Connection ~ 5450 4150
+Wire Wire Line
+	5450 4150 5850 4150
+Wire Wire Line
+	5050 4250 5050 4150
+Connection ~ 5050 4150
+Wire Wire Line
+	5050 4150 5450 4150
+Wire Wire Line
+	5050 4350 5050 4500
+Wire Wire Line
+	5050 4500 5350 4500
+Wire Wire Line
+	5450 4350 5450 4500
+Wire Wire Line
+	5450 4500 5350 4500
+Connection ~ 5350 4500
 $EndSCHEMATC

Commit message: Update FID footprint.
Parts:
- FID1, FID2, FID3, FID4: footprint Fiducial:Fiducial_1mm_Dia_2.54mm_Outer_CopperTop -> PrntrBoardV1:Fiducial_1mm_Dia_2.54mm_Outer_CopperTop
Changed lines of the file:
@@
 F 0 "FID1" H 2050 1646 50  0000 L CNN
 F 1 "Fiducial" H 2050 1555 50  0000 L CNN
-F 2 "Fiducial:Fiducial_1mm_Dia_2.54mm_Outer_CopperTop" H 1950 1600 50  0001 C CNN
+F 2 "PrntrBoardV1:Fiducial_1mm_Dia_2.54mm_Outer_CopperTop" H 1950 1600 50  0001 C CNN
 F 3 "" H 1950 1600 50  0001 C CNN
 	1    1950 1600
@@
 F 0 "FID2" H 2050 1896 50  0000 L CNN
 F 1 "Fiducial" H 2050 1805 50  0000 L CNN
-F 2 "Fiducial:Fiducial_1mm_Dia_2.54mm_Outer_CopperTop" H 1950 1850 50  0001 C CNN
+F 2 "PrntrBoardV1:Fiducial_1mm_Dia_2.54mm_Outer_CopperTop" H 1950 1850 50  0001 C CNN
 F 3 "" H 1950 1850 50  0001 C CNN
 	1    1950 1850
@@
 F 0 "FID3" H 2050 2146 50  0000 L CNN
 F 1 "Fiducial" H 2050 2055 50  0000 L CNN
-F 2 "Fiducial:Fiducial_1mm_Dia_2.54mm_Outer_CopperTop" H 1950 2100 50  0001 C CNN
+F 2 "PrntrBoardV1:Fiducial_1mm_Dia_2.54mm_Outer_CopperTop" H 1950 2100 50  0001 C CNN
 F 3 "" H 1950 2100 50  0001 C CNN
 	1    1950 2100
@@
 F 0 "FID4" H 2050 1446 50  0000 L CNN
 F 1 "Fiducial" H 2050 1355 50  0000 L CNN
-F 2 "Fiducial:Fiducial_1mm_Dia_2.54mm_Outer_CopperTop" H 1950 1400 50  0001 C CNN
+F 2 "PrntrBoardV1:Fiducial_1mm_Dia_2.54mm_Outer_CopperTop" H 1950 1400 50  0001 C CNN
 F 3 "" H 1950 1400 50  0001 C CNN
 	1    1950 1400

Commit message: Update annotations.
Parts:
- removed FID1, FID2, FID3, FID4: Fiducial, PrntrBoardV1:Fiducial_1mm_Dia_2.54mm_Outer_CopperTop, symbol Mechanical:Mounting_Hole
- removed MK1, MK2, MK3: Mounting_Hole_3mm, MountingHole:MountingHole_3.2mm_M3, symbol Mechanical:Mounting_Hole
- removed MK4: Mounting_Hole, MountingHole:MountingHole_3.2mm_M3, symbol Mechanical:Mounting_Hole
- added FID1, FID2, FID3, FID4: Fiducial, PrntrBoardV1:Fiducial_1mm_Dia_2.54mm_Outer_CopperTop, symbol Mechanical:Fiducial
- added MK1, MK2, MK3, MK4: Mounting_Hole-Mechanical, symbol PrntrBoardV1-rescue:Mounting_Hole-Mechanical
Changed lines of the file:
@@
 EESchema Schematic File Version 4
 LIBS:PrntrBoardV1-cache
-EELAYER 26 0
+EELAYER 29 0
 EELAYER END
 $Descr A4 11693 8268
@@
 	3850 1950 3700 1950
 $Comp
-L Mechanical:Mounting_Hole MK1
-U 1 1 5ACC3347
-P 1000 1600
-F 0 "MK1" H 1100 1646 50  0000 L CNN
-F 1 "Mounting_Hole_3mm" H 1100 1555 50  0000 L CNN
-F 2 "MountingHole:MountingHole_3.2mm_M3" H 1000 1600 50  0001 C CNN
-F 3 "" H 1000 1600 50  0001 C CNN
-	1    1000 1600
-	1    0    0    -1
-$EndComp
-$Comp
-L Mechanical:Mounting_Hole MK2
-U 1 1 5ACC33D5
-P 1000 1850
-F 0 "MK2" H 1100 1896 50  0000 L CNN
-F 1 "Mounting_Hole_3mm" H 1100 1805 50  0000 L CNN
-F 2 "MountingHole:MountingHole_3.2mm_M3" H 1000 1850 50  0001 C CNN
-F 3 "" H 1000 1850 50  0001 C CNN
-	1    1000 1850
-	1    0    0    -1
-$EndComp
-$Comp
-L Mechanical:Mounting_Hole MK3
-U 1 1 5ACC3448
-P 1000 2100
-F 0 "MK3" H 1100 2146 50  0000 L CNN
-F 1 "Mounting_Hole_3mm" H 1100 2055 50  0000 L CNN
-F 2 "MountingHole:MountingHole_3.2mm_M3" H 1000 2100 50  0001 C CNN
-F 3 "" H 1000 2100 50  0001 C CNN
-	1    1000 2100
-	1    0    0    -1
-$EndComp
-NoConn ~ 1000 1600
-NoConn ~ 1000 1850
-NoConn ~ 1000 2100
-$Comp
-L Mechanical:Mounting_Hole FID1
-U 1 1 5ACF4B85
-P 1950 1600
-F 0 "FID1" H 2050 1646 50  0000 L CNN
-F 1 "Fiducial" H 2050 1555 50  0000 L CNN
-F 2 "PrntrBoardV1:Fiducial_1mm_Dia_2.54mm_Outer_CopperTop" H 1950 1600 50  0001 C CNN
-F 3 "" H 1950 1600 50  0001 C CNN
-	1    1950 1600
-	1    0    0    -1
-$EndComp
-$Comp
-L Mechanical:Mounting_Hole FID2
-U 1 1 5ACF4C64
-P 1950 1850
-F 0 "FID2" H 2050 1896 50  0000 L CNN
-F 1 "Fiducial" H 2050 1805 50  0000 L CNN
-F 2 "PrntrBoardV1:Fiducial_1mm_Dia_2.54mm_Outer_CopperTop" H 1950 1850 50  0001 C CNN
-F 3 "" H 1950 1850 50  0001 C CNN
-	1    1950 1850
-	1    0    0    -1
-$EndComp
-$Comp
-L Mechanical:Mounting_Hole FID3
-U 1 1 5ACF4CE0
-P 1950 2100
-F 0 "FID3" H 2050 2146 50  0000 L CNN
-F 1 "Fiducial" H 2050 2055 50  0000 L CNN
-F 2 "PrntrBoardV1:Fiducial_1mm_Dia_2.54mm_Outer_CopperTop" H 1950 2100 50  0001 C CNN
-F 3 "" H 1950 2100 50  0001 C CNN
-	1    1950 2100
-	1    0    0    -1
-$EndComp
-NoConn ~ 1950 1600
-NoConn ~ 1950 1850
-NoConn ~ 1950 2100
-$Comp
-L Mechanical:Mounting_Hole FID4
-U 1 1 5AD38017
-P 1950 1400
-F 0 "FID4" H 2050 1446 50  0000 L CNN
-F 1 "Fiducial" H 2050 1355 50  0000 L CNN
-F 2 "PrntrBoardV1:Fiducial_1mm_Dia_2.54mm_Outer_CopperTop" H 1950 1400 50  0001 C CNN
-F 3 "" H 1950 1400 50  0001 C CNN
-	1    1950 1400
-	1    0    0    -1
-$EndComp
-NoConn ~ 1950 1400
-$Comp
 L PrntrBoardV1-rescue:Screw_Terminal_01x02-Connector_Specialized J1
 U 1 1 5AEDA4A7
@@
 	5050 1950 4700 1950
 Connection ~ 4700 1950
-$Comp
-L Mechanical:Mounting_Hole MK4
-U 1 1 5AE11BDF
-P 1000 1350
-F 0 "MK4" H 1100 1396 50  0000 L CNN
-F 1 "Mounting_Hole" H 1100 1305 50  0000 L CNN
-F 2 "MountingHole:MountingHole_3.2mm_M3" H 1000 1350 50  0001 C CNN
-F 3 "" H 1000 1350 50  0001 C CNN
-	1    1000 1350
-	1    0    0    -1
-$EndComp
-NoConn ~ 1000 1350
 $Comp
 L Jumper:Jumper_2_Open JP8
@@
 	5450 4500 5350 4500
 Connection ~ 5350 4500
+$Comp
+L PrntrBoardV1-rescue:Mounting_Hole-Mechanical MK1
+U 1 1 5C45D06F
+P 750 1250
+F 0 "MK1" H 850 1296 50  0000 L CNN
+F 1 "Mounting_Hole-Mechanical" H 850 1205 50  0000 L CNN
+F 2 "" H 750 1250 50  0001 C CNN
+F 3 "" H 750 1250 50  0001 C CNN
+	1    750  1250
+	1    0    0    -1
+$EndComp
+$Comp
+L PrntrBoardV1-rescue:Mounting_Hole-Mechanical MK2
+U 1 1 5C45DD4F
+P 750 1500
+F 0 "MK2" H 850 1546 50  0000 L CNN
+F 1 "Mounting_Hole-Mechanical" H 850 1455 50  0000 L CNN
+F 2 "" H 750 1500 50  0001 C CNN
+F 3 "" H 750 1500 50  0001 C CNN
+	1    750  1500
+	1    0    0    -1
+$EndComp
+$Comp
+L PrntrBoardV1-rescue:Mounting_Hole-Mechanical MK3
+U 1 1 5C45E6B4
+P 750 1750
+F 0 "MK3" H 850 1796 50  0000 L CNN
+F 1 "Mounting_Hole-Mechanical" H 850 1705 50  0000 L CNN
+F 2 "" H 750 1750 50  0001 C CNN
+F 3 "" H 750 1750 50  0001 C CNN
+	1    750  1750
+	1    0    0    -1
+$EndComp
+$Comp
+L PrntrBoardV1-rescue:Mounting_Hole-Mechanical MK4
+U 1 1 5C45F2D3
+P 750 2000
+F 0 "MK4" H 850 2046 50  0000 L CNN
+F 1 "Mounting_Hole-Mechanical" H 850 1955 50  0000 L CNN
+F 2 "" H 750 2000 50  0001 C CNN
+F 3 "" H 750 2000 50  0001 C CNN
+	1    750  2000
+	1    0    0    -1
+$EndComp
+$Comp
+L Mechanical:Fiducial FID1
+U 1 1 5C45FEDB
+P 2100 1300
+F 0 "FID1" H 2185 1346 50  0000 L CNN
+F 1 "Fiducial" H 2185 1255 50  0000 L CNN
+F 2 "PrntrBoardV1:Fiducial_1mm_Dia_2.54mm_Outer_CopperTop" H 2100 1300 50  0001 C CNN
+F 3 "~" H 2100 1300 50  0001 C CNN
+	1    2100 1300
+	1    0    0    -1
+$EndComp
+$Comp
+L Mechanical:Fiducial FID2
+U 1 1 5C460A81
+P 2100 1550
+F 0 "FID2" H 2185 1596 50  0000 L CNN
+F 1 "Fiducial" H 2185 1505 50  0000 L CNN
+F 2 "PrntrBoardV1:Fiducial_1mm_Dia_2.54mm_Outer_CopperTop" H 2100 1550 50  0001 C CNN
+F 3 "~" H 2100 1550 50  0001 C CNN
+	1    2100 1550
+	1    0    0    -1
+$EndComp
+$Comp
+L Mechanical:Fiducial FID3
+U 1 1 5C461405
+P 2100 1800
+F 0 "FID3" H 2185 1846 50  0000 L CNN
+F 1 "Fiducial" H 2185 1755 50  0000 L CNN
+F 2 "PrntrBoardV1:Fiducial_1mm_Dia_2.54mm_Outer_CopperTop" H 2100 1800 50  0001 C CNN
+F 3 "~" H 2100 1800 50  0001 C CNN
+	1    2100 1800
+	1    0    0    -1
+$EndComp
+$Comp
+L Mechanical:Fiducial FID4
+U 1 1 5C4620C1
+P 2100 2050
+F 0 "FID4" H 2185 2096 50  0000 L CNN
+F 1 "Fiducial" H 2185 2005 50  0000 L CNN
+F 2 "PrntrBoardV1:Fiducial_1mm_Dia_2.54mm_Outer_CopperTop" H 2100 2050 50  0001 C CNN
+F 3 "~" H 2100 2050 50  0001 C CNN
+	1    2100 2050
+	1    0    0    -1
+$EndComp
+NoConn ~ 2100 1300
+NoConn ~ 2100 1550
+NoConn ~ 2100 1800
+NoConn ~ 2100 2050
+NoConn ~ 750  2000
+NoConn ~ 750  1750
+NoConn ~ 750  1500
+NoConn ~ 750  1250
 $EndSCHEMATC

Commit message: Add missing files from the TMC2130 branch.
Parts:
- C1, C2, C89: footprint Capacitor_SMD:C_0603_1608Metric -> PrntrBoardV1:C_0603_1608Metric
- R1, R22, R23, R28, R29, R30, R31, R36, R37: footprint Resistor_SMD:R_0603_1608Metric -> PrntrBoardV1:R_0603_1608Metric
Changed lines of the file:
@@
 F 0 "C1" H 4950 2350 50  0000 L CNN
 F 1 "0.1uF" H 4850 2250 50  0000 L CNN
-F 2 "Capacitor_SMD:C_0603_1608Metric" H 5188 2150 50  0001 C CNN
+F 2 "PrntrBoardV1:C_0603_1608Metric" H 5188 2150 50  0001 C CNN
 F 3 "~" H 5150 2300 50  0001 C CNN
 	1    5150 2300
@@
 F 0 "C2" H 7250 5500 50  0000 L CNN
 F 1 "0.1uF" H 7200 5400 50  0000 L CNN
-F 2 "Capacitor_SMD:C_0603_1608Metric" H 7238 5450 50  0001 C CNN
+F 2 "PrntrBoardV1:C_0603_1608Metric" H 7238 5450 50  0001 C CNN
 F 3 "~" H 7200 5600 50  0001 C CNN
 	1    7200 5600
@@
 F 0 "R1" V 9150 5150 50  0000 C CNN
 F 1 "1k" V 9150 5300 50  0000 C CNN
-F 2 "Resistor_SMD:R_0603_1608Metric" V 8980 5200 50  0001 C CNN
+F 2 "PrntrBoardV1:R_0603_1608Metric" V 8980 5200 50  0001 C CNN
 F 3 "~" H 9050 5200 50  0001 C CNN
 	1    9050 5200
@@
 F 0 "C89" H 5165 1546 50  0000 L CNN
 F 1 "1000pF" H 5050 1400 50  0000 L CNN
-F 2 "Capacitor_SMD:C_0603_1608Metric" H 5088 1350 50  0001 C CNN
+F 2 "PrntrBoardV1:C_0603_1608Metric" H 5088 1350 50  0001 C CNN
 F 3 "~" H 5050 1500 50  0001 C CNN
 	1    5050 1500
@@
 F 0 "R29" H 4970 4946 50  0000 L CNN
 F 1 "10k" H 4970 4855 50  0000 L CNN
-F 2 "Resistor_SMD:R_0603_1608Metric" V 4830 4900 50  0001 C CNN
+F 2 "PrntrBoardV1:R_0603_1608Metric" V 4830 4900 50  0001 C CNN
 F 3 "~" H 4900 4900 50  0001 C CNN
 	1    4900 4900
@@
 F 0 "R23" H 4920 5646 50  0000 L CNN
 F 1 "10k" H 4920 5555 50  0000 L CNN
-F 2 "Resistor_SMD:R_0603_1608Metric" V 4780 5600 50  0001 C CNN
+F 2 "PrntrBoardV1:R_0603_1608Metric" V 4780 5600 50  0001 C CNN
 F 3 "~" H 4850 5600 50  0001 C CNN
 	1    4850 5600
@@
 F 0 "R28" H 4920 6146 50  0000 L CNN
 F 1 "10k" H 4920 6055 50  0000 L CNN
-F 2 "Resistor_SMD:R_0603_1608Metric" V 4780 6100 50  0001 C CNN
+F 2 "PrntrBoardV1:R_0603_1608Metric" V 4780 6100 50  0001 C CNN
 F 3 "~" H 4850 6100 50  0001 C CNN
 	1    4850 6100
@@
 F 0 "R22" H 4820 6696 50  0000 L CNN
 F 1 "10k" H 4820 6605 50  0000 L CNN
-F 2 "Resistor_SMD:R_0603_1608Metric" V 4680 6650 50  0001 C CNN
+F 2 "PrntrBoardV1:R_0603_1608Metric" V 4680 6650 50  0001 C CNN
 F 3 "~" H 4750 6650 50  0001 C CNN
 	1    4750 6650
@@
 F 0 "R31" H 6670 5646 50  0000 L CNN
 F 1 "10k" H 6670 5555 50  0000 L CNN
-F 2 "Resistor_SMD:R_0603_1608Metric" V 6530 5600 50  0001 C CNN
+F 2 "PrntrBoardV1:R_0603_1608Metric" V 6530 5600 50  0001 C CNN
 F 3 "~" H 6600 5600 50  0001 C CNN
 	1    6600 5600
@@
 F 0 "R30" H 3070 1346 50  0000 L CNN
 F 1 "10k" H 3070 1255 50  0000 L CNN
-F 2 "Resistor_SMD:R_0603_1608Metric" V 2930 1300 50  0001 C CNN
+F 2 "PrntrBoardV1:R_0603_1608Metric" V 2930 1300 50  0001 C CNN
 F 3 "~" H 3000 1300 50  0001 C CNN
 	1    3000 1300
@@
 F 0 "R36" H 10820 1796 50  0000 L CNN
 F 1 "10k" H 10820 1705 50  0000 L CNN
-F 2 "Resistor_SMD:R_0603_1608Metric" V 10680 1750 50  0001 C CNN
+F 2 "PrntrBoardV1:R_0603_1608Metric" V 10680 1750 50  0001 C CNN
 F 3 "~" H 10750 1750 50  0001 C CNN
 	1    10750 1750
@@
 F 0 "R37" H 4500 2450 50  0000 L CNN
 F 1 "1k" H 4550 2350 50  0000 L CNN
-F 2 "Resistor_SMD:R_0603_1608Metric" V 4630 2350 50  0001 C CNN
+F 2 "PrntrBoardV1:R_0603_1608Metric" V 4630 2350 50  0001 C CNN
 F 3 "~" H 4700 2350 50  0001 C CNN
 	1    4700 2350

Commit message: Update schematics to match rev3 of tmc2130 branch.
Parts:
- removed C78, C79: 10uF 10V, Capacitor_SMD:C_0603_1608Metric, symbol Device:C
- removed C80: 1000pF, Capacitor_SMD:C_0603_1608Metric, symbol Device:C
- removed FID1, FID2, FID3, FID4: Fiducial, PrntrBoardV1:Fiducial_1mm_Dia_2.54mm_Outer_CopperTop, symbol Mechanical:Fiducial
- removed MK1, MK2, MK3, MK4: Mounting_Hole-Mechanical, symbol PrntrBoardV1-rescue:Mounting_Hole-Mechanical
- added C91, C92: 10uF 10V, PrntrBoardV1:C_0603_1608Metric, symbol Device:C
- added C93: 1000pF, PrntrBoardV1:C_0603_1608Metric, symbol Device:C
- added FID1, FID2, FID3, FID4: Fiducial, PrntrBoardV1:Fiducial_1mm_Dia_2.54mm_Outer_CopperTop, symbol Mechanical:MountingHole
- added MK1, MK2, MK3: Mounting_Hole_3mm, MountingHole:MountingHole_3.2mm_M3, symbol Mechanical:MountingHole
- added MK4: Mounting_Hole, MountingHole:MountingHole_3.2mm_M3, symbol Mechanical:MountingHole
- J33: value XF1 -> Vin
- J34: value XF2 -> Vin
- J35: value XF3 -> 5V
- J36: value XF4 -> 5V
Connections:
- net labels added: BTN_IN, ENC_A, ENC_B
- wire segments 310 -> 318
- no-connect marks 30 -> 27
Other:
- moved on the sheet: C2, D20, R31

Commit message: Reset schematics for tmc2660. Clean the board layout.
Parts:
- renumbered C91 to C1, C88 to C2, C89 to C3, C1 to C4, C92 to C5, C93 to C6, C2 to C7, D19 to D1, D22 to D2, D20 to D3, D21 to D4, FID4 to FID1, FID1 to FID2, FID2 to FID3, FID3 to FID4, J29 to J1, J5 to J10, J6 to J11, J7 to J12, J8 to J13, J9 to J14, J31 to J15, J32 to J16, J1 to J2, J33 to J3, J34 to J4, J35 to J5, J36 to J6, J2 to J7, J3 to J8, J4 to J9, JP2 to JP1, JP8 to JP2, JP9 to JP3, JP3 to JP4, JP1 to JP5, MK4 to MK1, MK1 to MK2, MK2 to MK3, MK3 to MK4, R30 to R1, R37 to R2, R22 to R3, R23 to R4, R28 to R5, R29 to R6, R31 to R7, R1 to R8, R36 to R9, U11 to U1, U1 to U2, U2 to U3
Connections:
- wire segments 318 -> 317

Commit message: Added OSHW logo.
Parts:
- added LOGO1: Logo_Open_Hardware_Large, Symbol:OSHW-Logo2_7.3x6mm_SilkScreen, symbol Graphic:Logo_Open_Hardware_Large
Changed lines of the file:
@@
 Text Label 9450 4600 0    50   ~ 0
 ENC_B
+$Comp
+L Graphic:Logo_Open_Hardware_Large LOGO1
+U 1 1 5C473C23
+P 4400 7300
+F 0 "LOGO1" H 4400 7800 50  0001 C CNN
+F 1 "Logo_Open_Hardware_Large" H 4400 6900 50  0001 C CNN
+F 2 "Symbol:OSHW-Logo2_7.3x6mm_SilkScreen" H 4400 7300 50  0001 C CNN
+F 3 "~" H 4400 7300 50  0001 C CNN
+	1    4400 7300
+	1    0    0    -1
+$EndComp
 $EndSCHEMATC

Commit message: Add two fuses.
Parts:
- added F1: 10A, Fuse:Fuseholder_Blade_Mini_Keystone_3568, symbol Device:Fuse
- added F2: 15A, Fuse:Fuseholder_Blade_Mini_Keystone_3568, symbol Device:Fuse
Connections:
- net labels added: Vin
- wire segments 317 -> 320
Other:
- moved on the sheet: J1
Changed lines of the file:
@@
 Wire Wire Line
 	5900 800  7900 800
-Connection ~ 7900 3950
 Wire Wire Line
 	6050 1250 5950 1250
@@
 	1    0    0    -1
 $EndComp
-Connection ~ 7900 1050
-Wire Wire Line
-	7900 1050 7900 3950
 Wire Wire Line
 	8950 1200 8950 1250
@@
 L PrntrBoardV1-rescue:Screw_Terminal_01x02-Connector_Specialized J1
 U 1 1 5ACB9063
-P 2350 900
-F 0 "J1" H 2270 575 50  0000 C CNN
-F 1 "12-24V" H 2270 666 50  0000 C CNN
-F 2 "PrntrBoardV1:TerminalBlock_Phoenix_MKDS-1,5-2-5.08_1x02_P5.08mm_Horizontal" H 2350 900 50  0001 C CNN
-F 3 "~" H 2350 900 50  0001 C CNN
-	1    2350 900
+P 1600 900
+F 0 "J1" H 1520 575 50  0000 C CNN
+F 1 "12-24V" H 1520 666 50  0000 C CNN
+F 2 "PrntrBoardV1:TerminalBlock_Phoenix_MKDS-1,5-2-5.08_1x02_P5.08mm_Horizontal" H 1600 900 50  0001 C CNN
+F 3 "~" H 1600 900 50  0001 C CNN
+	1    1600 900
 	-1   0    0    1
 $EndComp
@@
 L power:GND #PWR02
 U 1 1 5ACB9195
-P 2600 950
-F 0 "#PWR02" H 2600 700 50  0001 C CNN
-F 1 "GND" H 2605 777 50  0000 C CNN
-F 2 "" H 2600 950 50  0001 C CNN
-F 3 "" H 2600 950 50  0001 C CNN
-	1    2600 950
-	1    0    0    -1
-$EndComp
-Wire Wire Line
-	2600 950  2600 900
-Wire Wire Line
-	2600 900  2550 900
+P 1850 950
+F 0 "#PWR02" H 1850 700 50  0001 C CNN
+F 1 "GND" H 1855 777 50  0000 C CNN
+F 2 "" H 1850 950 50  0001 C CNN
+F 3 "" H 1850 950 50  0001 C CNN
+	1    1850 950
+	1    0    0    -1
+$EndComp
 Wire Wire Line
 	3700 1850 4100 1850
@@
 	1    0    0    -1
 $EndComp
+$Comp
+L Device:Fuse F2
+U 1 1 5C49EAB2
+P 7900 3700
+F 0 "F2" H 7960 3746 50  0000 L CNN
+F 1 "15A" H 7960 3655 50  0000 L CNN
+F 2 "Fuse:Fuseholder_Blade_Mini_Keystone_3568" V 7830 3700 50  0001 C CNN
+F 3 "~" H 7900 3700 50  0001 C CNN
+	1    7900 3700
+	1    0    0    -1
+$EndComp
+Wire Wire Line
+	7900 3850 7900 3950
+Connection ~ 7900 3950
+Wire Wire Line
+	7900 3550 7900 3500
+Wire Wire Line
+	7900 3500 7500 3500
+Text Label 7650 3500 0    50   ~ 0
+Vin
+Wire Wire Line
+	1850 950  1850 900
+Wire Wire Line
+	1850 900  1800 900
+Text Label 1850 800  0    50   ~ 0
+Vin
+$Comp
+L Device:Fuse F1
+U 1 1 5C5249D8
+P 2400 800
+F 0 "F1" V 2203 800 50  0000 C CNN
+F 1 "10A" V 2294 800 50  0000 C CNN
+F 2 "Fuse:Fuseholder_Blade_Mini_Keystone_3568" V 2330 800 50  0001 C CNN
+F 3 "~" H 2400 800 50  0001 C CNN
+	1    2400 800
+	0    1    1    0
+$EndComp
+Wire Wire Line
+	1800 800  2250 800
 $EndSCHEMATC
