File: BedHeater.sch (KiCad schematic (older format))
At the start: 9 parts, among them J13 Thermistor

Commit message: Split the bed heater in separate schematics.
Other:
- moved on the sheet: C71, C72, D11, J28, R46, R47, R48, R49, TR3

Commit message: Assigned footprints for all components. Inductors are approximate size. MOSFETs dont agree with the footprints. Saved pcb netlist report as report.txt.
Parts:
- C16: footprint (none) -> Capacitor_SMD:C_0603_1608Metric
- C17: footprint (none) -> Capacitor_SMD:CP_Elec_4x5.3
- D2: footprint (none) -> LED_SMD:LED_0603_1608Metric
- J13: footprint (none) -> Connector_PinHeader_2.54mm:PinHeader_1x02_P2.54mm_Vertical
- R10, R11, R8, R9: footprint (none) -> Resistor_SMD:R_0603_1608Metric
- TR1: value IPD036N04L -> BSC011N03LS; footprint (none) -> Package_SON:Texas_S-PVSON-N8_ThermalVias
Changed lines of the file:
@@
 F 0 "J28" V 4054 4280 50  0000 L CNN
 F 1 "Thermistor" V 4145 4280 50  0000 L CNN
-F 2 "" H 4050 4200 50  0001 C CNN
+F 2 "Connector_PinHeader_2.54mm:PinHeader_1x02_P2.54mm_Vertical" H 4050 4200 50  0001 C CNN
 F 3 "~" H 4050 4200 50  0001 C CNN
 	1    4050 4200
@@
 F 0 "R46" H 3900 3550 50  0000 L CNN
 F 1 "4k7 1%" H 3700 3450 50  0000 L CNN
-F 2 "" V 3980 3500 50  0001 C CNN
+F 2 "Resistor_SMD:R_0603_1608Metric" V 3980 3500 50  0001 C CNN
 F 3 "~" H 4050 3500 50  0001 C CNN
 	1    4050 3500
@@
 F 0 "R47" V 4243 3800 50  0000 C CNN
 F 1 "10k" V 4334 3800 50  0000 C CNN
-F 2 "" V 4380 3800 50  0001 C CNN
+F 2 "Resistor_SMD:R_0603_1608Metric" V 4380 3800 50  0001 C CNN
 F 3 "~" H 4450 3800 50  0001 C CNN
 	1    4450 3800
@@
 F 0 "C71" H 4865 4146 50  0000 L CNN
 F 1 "1000pF" H 4865 4055 50  0000 L CNN
-F 2 "" H 4788 3950 50  0001 C CNN
+F 2 "Capacitor_SMD:C_0603_1608Metric" H 4788 3950 50  0001 C CNN
 F 3 "~" H 4750 4100 50  0001 C CNN
 	1    4750 4100
@@
 F 0 "R48" V 5693 3800 50  0000 C CNN
 F 1 "180R" V 5784 3800 50  0000 C CNN
-F 2 "" V 5830 3800 50  0001 C CNN
+F 2 "Resistor_SMD:R_0603_1608Metric" V 5830 3800 50  0001 C CNN
 F 3 "~" H 5900 3800 50  0001 C CNN
 	1    5900 3800
@@
 AR Path="/5AB8F10D/5AD51003" Ref="TR3"  Part="1"
 F 0 "TR3" H 6727 3853 70  0000 L CNN
-F 1 "IPD036N04L" H 6727 3739 60  0000 L CNN
-F 2 "" H 6500 3800 60  0000 C CNN
+F 1 "BSC011N03LS" H 6727 3739 60  0000 L CNN
+F 2 "Package_SON:Texas_S-PVSON-N8_ThermalVias" H 6500 3800 60  0001 C CNN
 F 3 "" H 6500 3800 60  0000 C CNN
 	1    6500 3800
@@
 F 0 "C72" H 5850 3050 50  0000 L CNN
 F 1 "10uF 35V" H 5600 2950 50  0000 L CNN
-F 2 "" H 6050 3000 50  0001 C CNN
+F 2 "Capacitor_SMD:CP_Elec_4x5.3" H 6050 3000 50  0001 C CNN
 F 3 "~" H 6050 3000 50  0001 C CNN
 	1    6050 3000
@@
 F 0 "R49" H 6420 2846 50  0000 L CNN
 F 1 "10k" H 6420 2755 50  0000 L CNN
-F 2 "" V 6280 2800 50  0001 C CNN
+F 2 "Resistor_SMD:R_0603_1608Metric" V 6280 2800 50  0001 C CNN
 F 3 "~" H 6350 2800 50  0001 C CNN
 	1    6350 2800
@@
 F 0 "D11" V 6450 3150 50  0000 R CNN
 F 1 "HEATER" V 6550 3150 50  0000 R CNN
-F 2 "" H 6350 3200 50  0001 C CNN
+F 2 "LED_SMD:LED_0603_1608Metric" H 6350 3200 50  0001 C CNN
 F 3 "~" H 6350 3200 50  0001 C CNN
 	1    6350 3200

Commit message: Updated components. Removed power supply. Component layout on PCB.
Parts:
- TR1: footprint Package_SON:Texas_S-PVSON-N8_ThermalVias -> PrntrBoardV1:Texas_S-PVSON-N8_ThermalVias
Changed lines of the file:
@@
 $Descr A4 11693 8268
 encoding utf-8
-Sheet 30 35
+Sheet 30 34
 Title ""
 Date ""
@@
 $Comp
 L Device:C C16
-U 1 1 5AD4D569
+U 1 1 5ACEEAAF
 P 4750 4100
-AR Path="/5AC337B6/5ACBE919/5AD4D269/5AD4D569" Ref="C16"  Part="1"
-AR Path="/5AC337B6/5AD9F95A/5AD4D269/5AD4D569" Ref="C69"  Part="1"
-AR Path="/5AB8F10D/5AD4D569" Ref="C71"  Part="1"
+AR Path="/5AC337B6/5ACBE919/5AD4D269/5ACEEAAF" Ref="C16"  Part="1"
+AR Path="/5AC337B6/5AD9F95A/5AD4D269/5ACEEAAF" Ref="C69"  Part="1"
+AR Path="/5AB8F10D/5ACEEAAF" Ref="C71"  Part="1"
 F 0 "C71" H 4865 4146 50  0000 L CNN
 F 1 "1000pF" H 4865 4055 50  0000 L CNN
@@
 $Comp
 L ipd036n04l:IPD036N04L TR1
-U 1 1 5AD51003
+U 1 1 5ACEEAB1
 P 6500 3800
-AR Path="/5AC337B6/5ACBE919/5AD4D269/5AD51003" Ref="TR1"  Part="1"
-AR Path="/5AC337B6/5AD9F95A/5AD4D269/5AD51003" Ref="TR2"  Part="1"
-AR Path="/5AB8F10D/5AD51003" Ref="TR3"  Part="1"
+AR Path="/5AC337B6/5ACBE919/5AD4D269/5ACEEAB1" Ref="TR1"  Part="1"
+AR Path="/5AC337B6/5AD9F95A/5AD4D269/5ACEEAB1" Ref="TR2"  Part="1"
+AR Path="/5AB8F10D/5ACEEAB1" Ref="TR3"  Part="1"
 F 0 "TR3" H 6727 3853 70  0000 L CNN
 F 1 "BSC011N03LS" H 6727 3739 60  0000 L CNN
-F 2 "Package_SON:Texas_S-PVSON-N8_ThermalVias" H 6500 3800 60  0001 C CNN
+F 2 "PrntrBoardV1:Texas_S-PVSON-N8_ThermalVias" H 6500 3800 60  0001 C CNN
 F 3 "" H 6500 3800 60  0000 C CNN
 	1    6500 3800
@@
 $Comp
 L power:GND #PWR022
-U 1 1 5AD51105
+U 1 1 5ACEEAB2
 P 6650 4300
-AR Path="/5AC337B6/5ACBE919/5AD4D269/5AD51105" Ref="#PWR022"  Part="1"
-AR Path="/5AC337B6/5AD9F95A/5AD4D269/5AD51105" Ref="#PWR067"  Part="1"
-AR Path="/5AB8F10D/5AD51105" Ref="#PWR070"  Part="1"
+AR Path="/5AC337B6/5ACBE919/5AD4D269/5ACEEAB2" Ref="#PWR022"  Part="1"
+AR Path="/5AC337B6/5AD9F95A/5AD4D269/5ACEEAB2" Ref="#PWR067"  Part="1"
+AR Path="/5AB8F10D/5ACEEAB2" Ref="#PWR070"  Part="1"
 F 0 "#PWR070" H 6650 4050 50  0001 C CNN
 F 1 "GND" H 6655 4127 50  0000 C CNN
@@
 $Comp
 L Device:CP1_Small C17
-U 1 1 5AD51206
+U 1 1 5ACEEAB3
 P 6050 3000
-AR Path="/5AC337B6/5ACBE919/5AD4D269/5AD51206" Ref="C17"  Part="1"
-AR Path="/5AC337B6/5AD9F95A/5AD4D269/5AD51206" Ref="C70"  Part="1"
-AR Path="/5AB8F10D/5AD51206" Ref="C72"  Part="1"
+AR Path="/5AC337B6/5ACBE919/5AD4D269/5ACEEAB3" Ref="C17"  Part="1"
+AR Path="/5AC337B6/5AD9F95A/5AD4D269/5ACEEAB3" Ref="C70"  Part="1"
+AR Path="/5AB8F10D/5ACEEAB3" Ref="C72"  Part="1"
 F 0 "C72" H 5850 3050 50  0000 L CNN
 F 1 "10uF 35V" H 5600 2950 50  0000 L CNN
@@
 $Comp
 L Device:R R11
-U 1 1 5AD512CE
+U 1 1 5ACEEAB4
 P 6350 2800
-AR Path="/5AC337B6/5ACBE919/5AD4D269/5AD512CE" Ref="R11"  Part="1"
-AR Path="/5AC337B6/5AD9F95A/5AD4D269/5AD512CE" Ref="R45"  Part="1"
-AR Path="/5AB8F10D/5AD512CE" Ref="R49"  Part="1"
+AR Path="/5AC337B6/5ACBE919/5AD4D269/5ACEEAB4" Ref="R11"  Part="1"
+AR Path="/5AC337B6/5AD9F95A/5AD4D269/5ACEEAB4" Ref="R45"  Part="1"
+AR Path="/5AB8F10D/5ACEEAB4" Ref="R49"  Part="1"
 F 0 "R49" H 6420 2846 50  0000 L CNN
 F 1 "10k" H 6420 2755 50  0000 L CNN

Commit message: Update schematics to use TMC5130/TMC2130 drivers.
Parts:
- added D18: 1N4148, Diode_SMD:D_SOD-323F, symbol Device:D
Connections:
- net HEATER: now also D18.2 (A)
- net V_HEAT: now also D18.1 (K)
Changed lines of the file:
@@
 Connection ~ 6350 2500
 Wire Wire Line
-	6350 2500 7050 2500
+	6350 2500 6700 2500
 Wire Wire Line
 	6350 2950 6350 3050
@@
 HEATER
 Wire Wire Line
-	6750 3100 6650 3100
+	6750 3100 6700 3100
+$Comp
+L Device:D D18
+U 1 1 5ACE7777
+P 6700 2850
+F 0 "D18" V 6654 2929 50  0000 L CNN
+F 1 "1N4148" V 6745 2929 50  0000 L CNN
+F 2 "Diode_SMD:D_SOD-323F" H 6700 2850 50  0001 C CNN
+F 3 "~" H 6700 2850 50  0001 C CNN
+	1    6700 2850
+	0    1    1    0
+$EndComp
+Wire Wire Line
+	6700 2500 6700 2700
+Connection ~ 6700 2500
+Wire Wire Line
+	6700 2500 7050 2500
+Wire Wire Line
+	6700 3000 6700 3100
+Connection ~ 6700 3100
+Wire Wire Line
+	6700 3100 6650 3100
 $EndSCHEMATC

Commit message: Switched to local foorprints for terminals and LED. Switched to local foorprint for the printer driver ship - it has larger thermal pad ares.
Placement V1 complete.
Parts:
- D2: footprint LED_SMD:LED_0603_1608Metric -> PrntrBoardV1:LED_0603_1608Metric
Changed lines of the file:
@@
 F 0 "D11" V 6450 3150 50  0000 R CNN
 F 1 "HEATER" V 6550 3150 50  0000 R CNN
-F 2 "LED_SMD:LED_0603_1608Metric" H 6350 3200 50  0001 C CNN
+F 2 "PrntrBoardV1:LED_0603_1608Metric" H 6350 3200 50  0001 C CNN
 F 3 "~" H 6350 3200 50  0001 C CNN
 	1    6350 3200

Commit message: Change 10uF capacitor footprints to 1206.
Parts:
- C17: value 10uF 35V -> 10uF 50V; footprint Capacitor_SMD:CP_Elec_4x5.3 -> Capacitor_SMD:C_1206_3216Metric; symbol Device:CP1_Small -> Device:C
Changed lines of the file:
@@
 	6650 4150 6650 4300
 $Comp
-L Device:CP1_Small C17
+L Device:C C17
 U 1 1 5ACEEAB3
-P 6050 3000
+P 6050 2950
 AR Path="/5AC337B6/5ACBE919/5AD4D269/5ACEEAB3" Ref="C17"  Part="1"
 AR Path="/5AC337B6/5AD9F95A/5AD4D269/5ACEEAB3" Ref="C70"  Part="1"
 AR Path="/5AB8F10D/5ACEEAB3" Ref="C72"  Part="1"
 F 0 "C72" H 5850 3050 50  0000 L CNN
-F 1 "10uF 35V" H 5600 2950 50  0000 L CNN
-F 2 "Capacitor_SMD:CP_Elec_4x5.3" H 6050 3000 50  0001 C CNN
-F 3 "~" H 6050 3000 50  0001 C CNN
-	1    6050 3000
+F 1 "10uF 50V" H 5650 2850 50  0000 L CNN
+F 2 "Capacitor_SMD:C_1206_3216Metric" H 6050 2950 50  0001 C CNN
+F 3 "~" H 6050 2950 50  0001 C CNN
+	1    6050 2950
 	1    0    0    -1
 $EndComp
@@
 	6050 3100 6050 3250
 Wire Wire Line
-	6050 2900 6050 2500
+	6050 2800 6050 2500
 Wire Wire Line
 	6050 2500 6350 2500

Commit message: Updated TR3 foor print and re-routed tracks.
Parts:
- D18: footprint Diode_SMD:D_SOD-323F -> Diode_SMD:D_SOD-323_HandSoldering
- TR1: footprint PrntrBoardV1:Texas_S-PVSON-N8_ThermalVias -> PrntrBoardV1:PG-TDSON-8-FL
Changed lines of the file:
@@
 F 0 "TR3" H 6727 3853 70  0000 L CNN
 F 1 "BSC011N03LS" H 6727 3739 60  0000 L CNN
-F 2 "PrntrBoardV1:Texas_S-PVSON-N8_ThermalVias" H 6500 3800 60  0001 C CNN
+F 2 "PrntrBoardV1:PG-TDSON-8-FL" H 6500 3800 60  0001 C CNN
 F 3 "" H 6500 3800 60  0000 C CNN
 	1    6500 3800
@@
 F 0 "D18" V 6654 2929 50  0000 L CNN
 F 1 "1N4148" V 6745 2929 50  0000 L CNN
-F 2 "Diode_SMD:D_SOD-323F" H 6700 2850 50  0001 C CNN
+F 2 "Diode_SMD:D_SOD-323_HandSoldering" H 6700 2850 50  0001 C CNN
 F 3 "~" H 6700 2850 50  0001 C CNN
 	1    6700 2850
