File: BedHeater.sch (KiCad schematic (older format))
At the start: 10 parts, among them J13 Thermistor

Commit message: Change LED value to LED from HEATER.
Parts:
- D2: value HEATER -> LED
Changed lines of the file:
@@
 AR Path="/5AB8F10D/5AD513CB" Ref="D11"  Part="1"
 F 0 "D11" V 6450 3150 50  0000 R CNN
-F 1 "HEATER" V 6550 3150 50  0000 R CNN
+F 1 "LED" V 6550 3150 50  0000 R CNN
 F 2 "PrntrBoardV1:LED_0603_1608Metric" H 6350 3200 50  0001 C CNN
 F 3 "~" H 6350 3200 50  0001 C CNN

Commit message: Switch away from rounded rect pads. The PCB boar house had issues making the board.
Parts:
- C16: footprint Capacitor_SMD:C_0603_1608Metric -> PrntrBoardV1:C_0603_1608Metric
- C17: footprint Capacitor_SMD:C_1206_3216Metric -> PrntrBoardV1:C_1206_3216Metric
- R10, R11, R8, R9: footprint Resistor_SMD:R_0603_1608Metric -> PrntrBoardV1:R_0603_1608Metric
Changed lines of the file:
@@
 F 0 "R46" H 3900 3550 50  0000 L CNN
 F 1 "4k7 1%" H 3700 3450 50  0000 L CNN
-F 2 "Resistor_SMD:R_0603_1608Metric" V 3980 3500 50  0001 C CNN
+F 2 "PrntrBoardV1:R_0603_1608Metric" V 3980 3500 50  0001 C CNN
 F 3 "~" H 4050 3500 50  0001 C CNN
 	1    4050 3500
@@
 F 0 "R47" V 4243 3800 50  0000 C CNN
 F 1 "10k" V 4334 3800 50  0000 C CNN
-F 2 "Resistor_SMD:R_0603_1608Metric" V 4380 3800 50  0001 C CNN
+F 2 "PrntrBoardV1:R_0603_1608Metric" V 4380 3800 50  0001 C CNN
 F 3 "~" H 4450 3800 50  0001 C CNN
 	1    4450 3800
@@
 F 0 "C71" H 4865 4146 50  0000 L CNN
 F 1 "1000pF" H 4865 4055 50  0000 L CNN
-F 2 "Capacitor_SMD:C_0603_1608Metric" H 4788 3950 50  0001 C CNN
+F 2 "PrntrBoardV1:C_0603_1608Metric" H 4788 3950 50  0001 C CNN
 F 3 "~" H 4750 4100 50  0001 C CNN
 	1    4750 4100
@@
 F 0 "R48" V 5693 3800 50  0000 C CNN
 F 1 "180R" V 5784 3800 50  0000 C CNN
-F 2 "Resistor_SMD:R_0603_1608Metric" V 5830 3800 50  0001 C CNN
+F 2 "PrntrBoardV1:R_0603_1608Metric" V 5830 3800 50  0001 C CNN
 F 3 "~" H 5900 3800 50  0001 C CNN
 	1    5900 3800
@@
 F 0 "C72" H 5850 3050 50  0000 L CNN
 F 1 "10uF 50V" H 5650 2850 50  0000 L CNN
-F 2 "Capacitor_SMD:C_1206_3216Metric" H 6050 2950 50  0001 C CNN
+F 2 "PrntrBoardV1:C_1206_3216Metric" H 6050 2950 50  0001 C CNN
 F 3 "~" H 6050 2950 50  0001 C CNN
 	1    6050 2950
@@
 F 0 "R49" H 6420 2846 50  0000 L CNN
 F 1 "10k" H 6420 2755 50  0000 L CNN
-F 2 "Resistor_SMD:R_0603_1608Metric" V 6280 2800 50  0001 C CNN
+F 2 "PrntrBoardV1:R_0603_1608Metric" V 6280 2800 50  0001 C CNN
 F 3 "~" H 6350 2800 50  0001 C CNN
 	1    6350 2800

Commit message: Update thermistor filter capacitor values.
Parts:
- C16: value 1000pF -> 2.2uF
Changed lines of the file:
@@
 AR Path="/5AB8F10D/5ACEEAAF" Ref="C71"  Part="1"
 F 0 "C71" H 4865 4146 50  0000 L CNN
-F 1 "1000pF" H 4865 4055 50  0000 L CNN
+F 1 "2.2uF" H 4865 4055 50  0000 L CNN
 F 2 "PrntrBoardV1:C_0603_1608Metric" H 4788 3950 50  0001 C CNN
 F 3 "~" H 4750 4100 50  0001 C CNN
