File: MotorDriver_TMC5130.sch (KiCad schematic (older format))
At the start: 18 parts, among them U8 TMC5130

Commit message: Movet top FID to the top right corner. Added PCB origin. Switched 0.1uF 50V cpas to 0402 size.
Parts:
- C6, C86, C87: footprint Capacitor_SMD:C_0603_1608Metric -> Capacitor_SMD:C_0402_1005Metric
Changed lines of the file:
@@
 AR Path="/5AC337B6/5ACE1C6D/5ACC0B66/5AC33A94" Ref="C46"  Part="1"
 AR Path="/5AC337B6/5AD9F95A/5AD4B0F5/5AC33A94" Ref="C59"  Part="1"
-F 0 "C59" H 6000 2650 50  0000 L CNN
+F 0 "C33" H 6000 2650 50  0000 L CNN
 F 1 "0.1uF 50V" H 5700 2400 50  0000 L CNN
-F 2 "Capacitor_SMD:C_0603_1608Metric" H 5988 2400 50  0001 C CNN
+F 2 "Capacitor_SMD:C_0402_1005Metric" H 5988 2400 50  0001 C CNN
 F 3 "~" H 5950 2550 50  0001 C CNN
 	1    5950 2550
@@
 AR Path="/5AC337B6/5ACE1C6D/5ACC0B66/5AC33B3C" Ref="C44"  Part="1"
 AR Path="/5AC337B6/5AD9F95A/5AD4B0F5/5AC33B3C" Ref="C57"  Part="1"
-F 0 "C57" H 3050 1750 50  0000 L CNN
+F 0 "C31" H 3050 1750 50  0000 L CNN
 F 1 "10uF 50V" H 2850 1650 50  0000 L CNN
 F 2 "Capacitor_SMD:C_1206_3216Metric" H 3338 1550 50  0001 C CNN
@@
 AR Path="/5AC337B6/5ACE1C6D/5ACC0B66/5AC33B85" Ref="C47"  Part="1"
 AR Path="/5AC337B6/5AD9F95A/5AD4B0F5/5AC33B85" Ref="C60"  Part="1"
-F 0 "C60" H 5250 1800 50  0000 C CNN
+F 0 "C34" H 5250 1800 50  0000 C CNN
 F 1 "0.47uF" H 5200 1700 50  0000 C CNN
 F 2 "Capacitor_SMD:C_0603_1608Metric" H 5488 1650 50  0001 C CNN
@@
 AR Path="/5AC337B6/5ACE1C6D/5ACC0B66/5AC33C56" Ref="C48"  Part="1"
 AR Path="/5AC337B6/5AD9F95A/5AD4B0F5/5AC33C56" Ref="C61"  Part="1"
-F 0 "C61" H 4315 2096 50  0000 L CNN
+F 0 "C35" H 4315 2096 50  0000 L CNN
 F 1 "0.1uF" H 4315 2005 50  0000 L CNN
 F 2 "Capacitor_SMD:C_0603_1608Metric" H 4238 1900 50  0001 C CNN
@@
 AR Path="/5AC337B6/5ACE1C6D/5ACC0B66/5AC33CA1" Ref="C50"  Part="1"
 AR Path="/5AC337B6/5AD9F95A/5AD4B0F5/5AC33CA1" Ref="C63"  Part="1"
-F 0 "C63" V 7650 3450 50  0000 C CNN
+F 0 "C37" V 7650 3450 50  0000 C CNN
 F 1 "1000pF >50V" V 7750 3550 50  0000 C CNN
 F 2 "Capacitor_SMD:C_0603_1608Metric" H 7588 3450 50  0001 C CNN
@@
 AR Path="/5AC337B6/5ACE1C6D/5ACC0B66/5AC33D6E" Ref="C51"  Part="1"
 AR Path="/5AC337B6/5AD9F95A/5AD4B0F5/5AC33D6E" Ref="C64"  Part="1"
-F 0 "C64" V 6250 3150 50  0000 C CNN
+F 0 "C38" V 6250 3150 50  0000 C CNN
 F 1 "1000pF >50V" V 6250 3550 50  0000 C CNN
 F 2 "Capacitor_SMD:C_0603_1608Metric" H 6438 3150 50  0001 C CNN
@@
 AR Path="/5AC337B6/5ACE1C6D/5ACC0B66/5AC33DC1" Ref="C52"  Part="1"
 AR Path="/5AC337B6/5AD9F95A/5AD4B0F5/5AC33DC1" Ref="C65"  Part="1"
-F 0 "C65" V 6200 3700 50  0000 C CNN
+F 0 "C39" V 6200 3700 50  0000 C CNN
 F 1 "1000pF >50V" V 6200 4100 50  0000 C CNN
 F 2 "Capacitor_SMD:C_0603_1608Metric" H 6438 3650 50  0001 C CNN
@@
 AR Path="/5AC337B6/5ACE1C6D/5ACC0B66/5AC33E6E" Ref="C53"  Part="1"
 AR Path="/5AC337B6/5AD9F95A/5AD4B0F5/5AC33E6E" Ref="C66"  Part="1"
-F 0 "C66" V 6600 4650 50  0000 C CNN
+F 0 "C40" V 6600 4650 50  0000 C CNN
 F 1 "1000pF >50V" V 6700 4850 50  0000 C CNN
 F 2 "Capacitor_SMD:C_0603_1608Metric" H 6638 3950 50  0001 C CNN
@@
 AR Path="/5AC337B6/5ACE1C6D/5ACC0B66/5AC34593" Ref="#PWR049"  Part="1"
 AR Path="/5AC337B6/5AD9F95A/5AD4B0F5/5AC34593" Ref="#PWR059"  Part="1"
-F 0 "#PWR059" H 5450 1950 50  0001 C CNN
+F 0 "#PWR038" H 5450 1950 50  0001 C CNN
 F 1 "GND" H 5455 2027 50  0000 C CNN
 F 2 "" H 5450 2200 50  0001 C CNN
@@
 AR Path="/5AC337B6/5ACE1C6D/5ACC0B66/5AC345D6" Ref="#PWR048"  Part="1"
 AR Path="/5AC337B6/5AD9F95A/5AD4B0F5/5AC345D6" Ref="#PWR058"  Part="1"
-F 0 "#PWR058" H 3300 1800 50  0001 C CNN
+F 0 "#PWR037" H 3300 1800 50  0001 C CNN
 F 1 "GND" H 3305 1877 50  0000 C CNN
 F 2 "" H 3300 2050 50  0001 C CNN
@@
 AR Path="/5AC337B6/5ACE1C6D/5ACC0B66/5AC34619" Ref="#PWR050"  Part="1"
 AR Path="/5AC337B6/5AD9F95A/5AD4B0F5/5AC34619" Ref="#PWR060"  Part="1"
-F 0 "#PWR060" H 7800 3350 50  0001 C CNN
+F 0 "#PWR039" H 7800 3350 50  0001 C CNN
 F 1 "GND" H 7900 3600 50  0000 C CNN
 F 2 "" H 7800 3600 50  0001 C CNN
@@
 AR Path="/5AC337B6/5ACE1C6D/5ACC0B66/5AC3465C" Ref="#PWR051"  Part="1"
 AR Path="/5AC337B6/5AD9F95A/5AD4B0F5/5AC3465C" Ref="#PWR061"  Part="1"
-F 0 "#PWR061" H 6650 3050 50  0001 C CNN
+F 0 "#PWR040" H 6650 3050 50  0001 C CNN
 F 1 "GND" H 6750 3200 50  0000 C CNN
 F 2 "" H 6650 3300 50  0001 C CNN
@@
 AR Path="/5AC337B6/5ACE1C6D/5ACC0B66/5AC3469F" Ref="#PWR052"  Part="1"
 AR Path="/5AC337B6/5AD9F95A/5AD4B0F5/5AC3469F" Ref="#PWR062"  Part="1"
-F 0 "#PWR062" H 6650 3550 50  0001 C CNN
+F 0 "#PWR041" H 6650 3550 50  0001 C CNN
 F 1 "GND" H 6750 3800 50  0000 C CNN
 F 2 "" H 6650 3800 50  0001 C CNN
@@
 AR Path="/5AC337B6/5ACE1C6D/5ACC0B66/5AC346E2" Ref="#PWR053"  Part="1"
 AR Path="/5AC337B6/5AD9F95A/5AD4B0F5/5AC346E2" Ref="#PWR063"  Part="1"
-F 0 "#PWR063" H 6850 3850 50  0001 C CNN
+F 0 "#PWR042" H 6850 3850 50  0001 C CNN
 F 1 "GND" H 6950 4100 50  0000 C CNN
 F 2 "" H 6850 4100 50  0001 C CNN
@@
 AR Path="/5AC337B6/5ACE1C6D/5ACC0B66/5AC34725" Ref="#PWR047"  Part="1"
 AR Path="/5AC337B6/5AD9F95A/5AD4B0F5/5AC34725" Ref="#PWR057"  Part="1"
-F 0 "#PWR057" H 5350 5550 50  0001 C CNN
+F 0 "#PWR036" H 5350 5550 50  0001 C CNN
 F 1 "GND" H 5355 5627 50  0000 C CNN
 F 2 "" H 5350 5800 50  0001 C CNN
@@
 AR Path="/5AC337B6/5ACE1C6D/5ACC0B66/5AC55FA7" Ref="C45"  Part="1"
 AR Path="/5AC337B6/5AD9F95A/5AD4B0F5/5AC55FA7" Ref="C58"  Part="1"
-F 0 "C58" H 3700 1900 50  0000 L CNN
+F 0 "C32" H 3700 1900 50  0000 L CNN
 F 1 "100uF 35V" H 3700 1800 50  0000 L CNN
 F 2 "Capacitor_SMD:CP_Elec_6.3x7.7" H 3650 1700 50  0001 C CNN
@@
 AR Path="/5AC337B6/5ACE1C6D/5ACC0B66/5ACA36B2" Ref="C76"  Part="1"
 AR Path="/5AC337B6/5AD9F95A/5AD4B0F5/5ACA36B2" Ref="C77"  Part="1"
-F 0 "C77" H 2715 1746 50  0000 L CNN
+F 0 "C75" H 2715 1746 50  0000 L CNN
 F 1 "10uF 50V" H 2650 1550 50  0000 L CNN
 F 2 "Capacitor_SMD:C_1206_3216Metric" H 2638 1550 50  0001 C CNN
@@
 AR Path="/5AC337B6/5ACCA309/5ACC0B66/5ACFA54E" Ref="U6"  Part="1"
 AR Path="/5AC337B6/5ACE1C6D/5ACC0B66/5ACFA54E" Ref="U7"  Part="1"
-F 0 "U8" H 4900 1714 50  0000 C CNN
+F 0 "U6" H 4900 1714 50  0000 C CNN
 F 1 "TMC5130" H 4900 1623 50  0000 C CNN
 F 2 "PrntrBoardV1:tmc5130-nc" H 4900 3700 50  0001 C CNN
@@
 AR Path="/5AC337B6/5ACCA309/5ACC0B66/5AD3397E" Ref="#PWR081"  Part="1"
 AR Path="/5AC337B6/5ACE1C6D/5ACC0B66/5AD3397E" Ref="#PWR083"  Part="1"
-F 0 "#PWR085" H 4200 2000 50  0001 C CNN
+F 0 "#PWR081" H 4200 2000 50  0001 C CNN
 F 1 "GND" H 4205 2077 50  0000 C CNN
 F 2 "" H 4200 2250 50  0001 C CNN
@@
 AR Path="/5AC337B6/5ACCA309/5ACC0B66/5AD37DE9" Ref="C67"  Part="1"
 AR Path="/5AC337B6/5ACE1C6D/5ACC0B66/5AD37DE9" Ref="C81"  Part="1"
-F 0 "C85" H 5000 2350 50  0000 L CNN
+F 0 "C67" H 5000 2350 50  0000 L CNN
 F 1 "0.1uF" H 4900 2250 50  0000 L CNN
 F 2 "Capacitor_SMD:C_0603_1608Metric" H 5188 2000 50  0001 C CNN
@@
 AR Path="/5AC337B6/5ACCA309/5ACC0B66/5AD494C8" Ref="C62"  Part="1"
 AR Path="/5AC337B6/5ACE1C6D/5ACC0B66/5AD494C8" Ref="C80"  Part="1"
-F 0 "C84" V 3750 5200 50  0000 C CNN
+F 0 "C62" V 3750 5200 50  0000 C CNN
 F 1 "0.022uF 50V" V 3750 4750 50  0000 C CNN
 F 2 "Capacitor_SMD:C_0603_1608Metric" H 3638 4900 50  0001 C CNN
@@
 AR Path="/5AC337B6/5ACCA309/5ACC0B66/5AD5670C" Ref="#PWR080"  Part="1"
 AR Path="/5AC337B6/5ACE1C6D/5ACC0B66/5AD5670C" Ref="#PWR082"  Part="1"
-F 0 "#PWR084" H 3600 3900 50  0001 C CNN
+F 0 "#PWR080" H 3600 3900 50  0001 C CNN
 F 1 "GND" H 3605 3977 50  0000 C CNN
 F 2 "" H 3600 4150 50  0001 C CNN
@@
 AR Path="/5AC337B6/5ACCA309/5ACC0B66/5AD66FAA" Ref="R12"  Part="1"
 AR Path="/5AC337B6/5ACE1C6D/5ACC0B66/5AD66FAA" Ref="R14"  Part="1"
-F 0 "R20" H 6370 4996 50  0000 L CNN
+F 0 "R12" H 6370 4996 50  0000 L CNN
 F 1 "0R15 0.5W" H 6100 4800 50  0000 L CNN
 F 2 "Resistor_SMD:R_1206_3216Metric" V 6230 4950 50  0001 C CNN
@@
 AR Path="/5AC337B6/5ACCA309/5ACC0B66/5AD67008" Ref="R13"  Part="1"
 AR Path="/5AC337B6/5ACE1C6D/5ACC0B66/5AD67008" Ref="R15"  Part="1"
-F 0 "R21" H 6970 5046 50  0000 L CNN
+F 0 "R13" H 6970 5046 50  0000 L CNN
 F 1 "0R15 0.5W" H 6970 4955 50  0000 L CNN
 F 2 "Resistor_SMD:R_1206_3216Metric" V 6830 5000 50  0001 C CNN
@@
 AR Path="/5AC337B6/5ACCA309/5ACC0B66/5AD6F856" Ref="C79"  Part="1"
 AR Path="/5AC337B6/5ACE1C6D/5ACC0B66/5AD6F856" Ref="C83"  Part="1"
-F 0 "C87" H 7665 5146 50  0000 L CNN
+F 0 "C79" H 7665 5146 50  0000 L CNN
 F 1 "0.1uF 50V" H 7665 5055 50  0000 L CNN
-F 2 "Capacitor_SMD:C_0603_1608Metric" H 7588 4950 50  0001 C CNN
+F 2 "Capacitor_SMD:C_0402_1005Metric" H 7588 4950 50  0001 C CNN
 F 3 "~" H 7550 5100 50  0001 C CNN
 	1    7550 5100
@@
 AR Path="/5AC337B6/5ACCA309/5ACC0B66/5AD6F966" Ref="C78"  Part="1"
 AR Path="/5AC337B6/5ACE1C6D/5ACC0B66/5AD6F966" Ref="C82"  Part="1"
-F 0 "C86" H 6715 5246 50  0000 L CNN
+F 0 "C78" H 6715 5246 50  0000 L CNN
 F 1 "0.1uF 50V" H 6350 5050 50  0000 L CNN
-F 2 "Capacitor_SMD:C_0603_1608Metric" H 6638 5050 50  0001 C CNN
+F 2 "Capacitor_SMD:C_0402_1005Metric" H 6638 5050 50  0001 C CNN
 F 3 "~" H 6600 5200 50  0001 C CNN
 	1    6600 5200
@@
 AR Path="/5AC337B6/5ACC0AA2/5ACC0B66/5AEA3C62" Ref="JP4"  Part="1"
 AR Path="/5AC337B6/5ACE1C6D/5ACC0B66/5AEA3C62" Ref="JP6"  Part="1"
-F 0 "JP7" V 8104 5198 50  0000 L CNN
+F 0 "JP5" V 8104 5198 50  0000 L CNN
 F 1 "Clock Disable" V 8195 5198 50  0000 L CNN
 F 2 "Jumper:SolderJumper-2_P1.3mm_Open_Pad1.0x1.5mm" H 8150 5100 50  0001 C CNN

Commit message: Some useless changes, I'll remove the SD_MODE wire soon.
Connections:
- net labels added: SD_MODE
- wire segments 107 -> 106
Changed lines of the file:
@@
 Wire Wire Line
 	3600 4050 3600 4150
-Wire Wire Line
-	3850 3800 3600 3800
-Wire Wire Line
-	3600 3800 3600 4050
-Connection ~ 3600 4050
 NoConn ~ 3850 3700
 NoConn ~ 3850 3900
@@
 	8150 5600 7550 5600
 Connection ~ 7550 5600
+Text HLabel 3100 3800 0    50   Input ~ 0
+SD_MODE
+Wire Wire Line
+	3100 3800 3850 3800
 $EndSCHEMATC

Commit message: Removed SD_MODE wire. Added motor clock oscillator. Wired the clock on the internal layer to reduce EMI.
Parts:
- removed JP5: Clock Disable, Jumper:SolderJumper-2_P1.3mm_Open_Pad1.0x1.5mm, symbol Jumper:Jumper_2_Open
Connections:
- net labels removed: SD_MODE
- wire segments 106 -> 101
- no-connect marks 6 -> 7
Changed lines of the file:
@@
 $Descr A4 11693 8268
 encoding utf-8
-Sheet 9 34
+Sheet 17 34
 Title ""
 Date ""
@@
 	6050 4950 5950 4950
 Connection ~ 5950 4950
-Wire Wire Line
-	5950 4700 8150 4700
 Text HLabel 8350 4700 2    50   Input ~ 0
 CLOCK
-$Comp
-L Jumper:Jumper_2_Open JP5
-U 1 1 5AEA3C62
-P 8150 5100
-AR Path="/5AC337B6/5ACCA309/5ACC0B66/5AEA3C62" Ref="JP5"  Part="1"
-AR Path="/5AC337B6/5AD9F95A/5AD4B0F5/5AEA3C62" Ref="JP7"  Part="1"
-AR Path="/5AC337B6/5ACBE919/5AD4B0F5/5AEA3C62" Ref="JP3"  Part="1"
-AR Path="/5AC337B6/5ACC0AA2/5ACC0B66/5AEA3C62" Ref="JP4"  Part="1"
-AR Path="/5AC337B6/5ACE1C6D/5ACC0B66/5AEA3C62" Ref="JP6"  Part="1"
-F 0 "JP7" V 8104 5198 50  0000 L CNN
-F 1 "Clock Disable" V 8195 5198 50  0000 L CNN
-F 2 "Jumper:SolderJumper-2_P1.3mm_Open_Pad1.0x1.5mm" H 8150 5100 50  0001 C CNN
-F 3 "~" H 8150 5100 50  0001 C CNN
-	1    8150 5100
-	0    1    1    0
-$EndComp
-Wire Wire Line
-	8150 4900 8150 4700
-Connection ~ 8150 4700
-Wire Wire Line
-	8150 4700 8350 4700
-Wire Wire Line
-	8150 5300 8150 5600
-Wire Wire Line
-	8150 5600 7550 5600
-Connection ~ 7550 5600
-Text HLabel 3100 3800 0    50   Input ~ 0
-SD_MODE
-Wire Wire Line
-	3100 3800 3850 3800
+NoConn ~ 3850 3800
+Wire Wire Line
+	5950 4700 8350 4700
 $EndSCHEMATC
