File: Endstop.sch (KiCad schematic (older format))
At the start: 4 parts

Commit message: Switched to local foorprints for terminals and LED. Switched to local foorprint for the printer driver ship - it has larger thermal pad ares.
Placement V1 complete.
Parts:
- D1: footprint LED_SMD:LED_0603_1608Metric -> PrntrBoardV1:LED_0603_1608Metric
Changed lines of the file:
@@
 F 0 "D9" V 4388 2433 50  0000 R CNN
 F 1 "LED" V 4297 2433 50  0000 R CNN
-F 2 "LED_SMD:LED_0603_1608Metric" H 4350 2550 50  0001 C CNN
+F 2 "PrntrBoardV1:LED_0603_1608Metric" H 4350 2550 50  0001 C CNN
 F 3 "~" H 4350 2550 50  0001 C CNN
 	1    4350 2550
