File: PrntrBoardV1.kicad_pcb (KiCad board)
At the start: 4 copper layers, 99 x 99 mm, 238 parts, among them J1 EXT 5V, J10 Probe, J11 Extruder Heater, J12 Stepper, J13 Thermistor, J14 Max, J15 Min, J16 Max, J17 Min, J18 Max, J19 Min, J2 Bed Heater, J20 Stepper, J21 Stepper, J22 Stepper, J23 Stepper, J24 Probe, J25 Extruder Heater, J26 Stepper, J27 Thermistor, J28 Thermistor, J29 12-24V, J3 Z Probe, J30 LCD, J31 TC1, J32 TC2, J33 Vin, J34 Vin, J35 5V, J36 5V, J4 E0 Cool, J5 E0 Part, J6 E1 Cool, J7 E1 Part, J8 Always On Fan 1, J9 Always On Fan 2, U1 4078, U11 NUCLEO-64, U2 74HCT02, U3 74LVC125, U4 TMC5130, U5 TMC5130, U6 TMC5130, U7 TMC5130, U8 TMC5130, X1 16MHz

Commit message: Update back labels.
Other:
- board text added: "A0"
- board text added: "MOSI"
- board text added: "~RESET"
Changed lines of the file:
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@@
   (general
     (thickness 1.6)
-    (drawings 109)
+    (drawings 120)
     (tracks 2521)
     (zones 0)
@@
   )
   (setup
-    (last_trace_width 0.5)
+    (last_trace_width 0.1524)
     (user_trace_width 0.1524)
     (user_trace_width 0.2032)
@@
     )
   )
+  (gr_text LCD (at 63.25 93.4 90) (layer B.SilkS)
+    (effects (font (size 1.5 1.5) (thickness 0.3)) (justify mirror))
+  )
+  (gr_text GND (at 50.5 97.65 90) (layer B.SilkS)
+    (effects (font (size 1 1) (thickness 0.15)) (justify mirror))
+  )
+  (gr_text GND (at 53 97.65 90) (layer B.SilkS)
+    (effects (font (size 1 1) (thickness 0.15)) (justify mirror))
+  )
+  (gr_text GND (at 55.55 97.65 90) (layer B.SilkS)
+    (effects (font (size 1 1) (thickness 0.15)) (justify mirror))
+  )
+  (gr_text 3.3V (at 58.25 97.65 90) (layer B.SilkS)
+    (effects (font (size 1 1) (thickness 0.15)) (justify mirror))
+  )
+  (gr_text 5V (at 60.7 96.8 90) (layer B.SilkS)
+    (effects (font (size 1 1) (thickness 0.15)) (justify mirror))
+  )
+  (gr_text MOSI (at 60.7 89.25 90) (layer B.SilkS)
+    (effects (font (size 1 1) (thickness 0.15)) (justify mirror))
+  )
+  (gr_text SCK (at 58.05 89.6 90) (layer B.SilkS)
+    (effects (font (size 1 1) (thickness 0.15)) (justify mirror))
+  )
+  (gr_text A0 (at 55.55 90.35 90) (layer B.SilkS)
+    (effects (font (size 1 1) (thickness 0.15)) (justify mirror))
+  )
+  (gr_text ~RESET (at 53.15 88.95 90) (layer B.SilkS)
+    (effects (font (size 1 1) (thickness 0.15)) (justify mirror))
+  )
+  (gr_text ~CS (at 50.55 90.05 90) (layer B.SilkS)
+    (effects (font (size 1 1) (thickness 0.15)) (justify mirror))
+  )
   (gr_text "+ -" (at 94.45 46.95 270) (layer F.SilkS)
     (effects (font (size 1.5 1.5) (thickness 0.3)))
@@
     (effects (font (size 0.8 0.8) (thickness 0.1)))
   )
-  (gr_text "Bed level\nprobe" (at 47.1 85.05 90) (layer B.SilkS)
+  (gr_text "Bed level\nprobe" (at 46.55 83.85 90) (layer B.SilkS)
     (effects (font (size 1.5 1.5) (thickness 0.3)) (justify mirror))
   )
-  (gr_text "Temp\nE0" (at 71.8 90.3) (layer B.SilkS)
+  (gr_text "Temp\nE0" (at 72.15 91.8) (layer B.SilkS)
     (effects (font (size 1.5 1.5) (thickness 0.3)) (justify mirror))
   )
-  (gr_text "Temp\nE1" (at 71.95 97) (layer B.SilkS)
+  (gr_text "Temp\nE1" (at 72.45 98.05) (layer B.SilkS)
     (effects (font (size 1.5 1.5) (thickness 0.3)) (justify mirror))
   )
-  (gr_text "Temp\nBeb" (at 71.8 103.5) (layer B.SilkS)
+  (gr_text "Temp\nBeb" (at 72.35 104.6) (layer B.SilkS)
     (effects (font (size 1.5 1.5) (thickness 0.3)) (justify mirror))
   )
-  (gr_text "E1 Filament\nDetect" (at 33.55 80.75) (layer B.SilkS)
+  (gr_text "E1 Filament\nDetect" (at 34.8 74.1) (layer B.SilkS)
     (effects (font (size 1.5 1.5) (thickness 0.3)) (justify mirror))
   )
@@
     (effects (font (size 1.5 1.5) (thickness 0.3)) (justify mirror))
   )
-  (gr_text "E0 Filament\nDetect" (at 70.5 78.35) (layer B.SilkS)
+  (gr_text "E0 Filament\nDetect" (at 71.95 85.45) (layer B.SilkS)
     (effects (font (size 1.5 1.5) (thickness 0.3)) (justify mirror))
   )
@@
     (effects (font (size 1.5 1.5) (thickness 0.3)) (justify mirror))
   )
-  (gr_text "E1\n+  -" (at 62.103 28.1305) (layer B.SilkS)
+  (gr_text "E1\n+  -" (at 62.4 28.25) (layer B.SilkS)
     (effects (font (size 1.5 1.5) (thickness 0.3)) (justify mirror))
   )
