File: Nucleo-64-407.sch (KiCad schematic (older format))
At the start: 70 parts, among them J1 SWD, J3 USB_B_Micro, J4 Serial 0, J5 EXP1, J6 EXP2, J7 EXP3, J8 EXP4, SW1 RESET, SW2 BOOT, U1 STM32F407VETx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

Commit message: Rename LED values.
Parts:
- D2: value B0 -> RED
- D3: value B1 -> RED
- D4: value VIN -> RED
- D5: value 3.3V -> RED
- D6: value 5V -> RED
Changed lines of the file:
@@
 P 8100 5050
 F 0 "D4" V 8139 4932 50  0000 R CNN
-F 1 "VIN" V 8048 4932 50  0000 R CNN
+F 1 "RED" V 8048 4932 50  0000 R CNN
 F 2 "PrntrBoardV1:D_0603_1608Metric" H 8100 5050 50  0001 C CNN
 F 3 "~" H 8100 5050 50  0001 C CNN
@@
 P 8450 5050
 F 0 "D5" V 8489 4933 50  0000 R CNN
-F 1 "3.3V" V 8398 4933 50  0000 R CNN
+F 1 "RED" V 8398 4933 50  0000 R CNN
 F 2 "PrntrBoardV1:D_0603_1608Metric" H 8450 5050 50  0001 C CNN
 F 3 "~" H 8450 5050 50  0001 C CNN
@@
 P 8800 5050
 F 0 "D6" V 8839 4932 50  0000 R CNN
-F 1 "5V" V 8748 4932 50  0000 R CNN
+F 1 "RED" V 8748 4932 50  0000 R CNN
 F 2 "PrntrBoardV1:D_0603_1608Metric" H 8800 5050 50  0001 C CNN
 F 3 "~" H 8800 5050 50  0001 C CNN
@@
 P 7600 5800
 F 0 "D2" V 7547 5878 50  0000 L CNN
-F 1 "B0" V 7638 5878 50  0000 L CNN
+F 1 "RED" V 7638 5878 50  0000 L CNN
 F 2 "PrntrBoardV1:D_0603_1608Metric" H 7600 5800 50  0001 C CNN
 F 3 "~" H 7600 5800 50  0001 C CNN
@@
 P 7900 5800
 F 0 "D3" V 7847 5878 50  0000 L CNN
-F 1 "B1" V 7938 5878 50  0000 L CNN
+F 1 "RED" V 7938 5878 50  0000 L CNN
 F 2 "PrntrBoardV1:D_0603_1608Metric" H 7900 5800 50  0001 C CNN
 F 3 "~" H 7900 5800 50  0001 C CNN
