File: ST7735 LCD.sch (KiCad schematic (older format))
At the start: 1 part, among them J30 LCD

Commit message: Started rev 3. Added encoder iand button input. Re-routed LCD A0 and RESET to be connected to the HW I2C pins.
Parts:
- removed J30: LCD, Connector_IDC:IDC-Header_2x05_P2.54mm_Vertical, symbol Connector_Generic:Conn_02x05_Odd_Even
- added J30: LCD, Connector_IDC:IDC-Header_2x06_P2.54mm_Vertical, symbol Connector_Generic:Conn_02x06_Odd_Even
Connections:
- net labels added: BTN_IN, ENC_A, ENC_B
- wire segments 12 -> 13
Changed lines of the file:
@@
 L power:GND #PWR090
 U 1 1 5AFA6291
-P 4100 2350
-F 0 "#PWR090" H 4100 2100 50  0001 C CNN
-F 1 "GND" H 4105 2177 50  0000 C CNN
-F 2 "" H 4100 2350 50  0001 C CNN
-F 3 "" H 4100 2350 50  0001 C CNN
-	1    4100 2350
+P 3450 2400
+F 0 "#PWR090" H 3450 2150 50  0001 C CNN
+F 1 "GND" H 3455 2227 50  0000 C CNN
+F 2 "" H 3450 2400 50  0001 C CNN
+F 3 "" H 3450 2400 50  0001 C CNN
+	1    3450 2400
 	1    0    0    -1
 $EndComp
-Wire Wire Line
-	4100 2150 4000 2150
 Wire Wire Line
 	4100 2050 4000 2050
@@
 Text HLabel 3450 2250 0    50   Input ~ 0
 ~CS
+Wire Wire Line
+	3450 2250 3500 2250
+Text HLabel 4100 2150 2    50   Input ~ 0
+BTN_IN
+Wire Wire Line
+	4100 2150 4000 2150
 $Comp
-L Connector_Generic:Conn_02x05_Odd_Even J30
-U 1 1 5B08E113
+L Connector_Generic:Conn_02x06_Odd_Even J30
+U 1 1 5B6CF880
 P 3700 2050
 F 0 "J30" H 3750 2467 50  0000 C CNN
 F 1 "LCD" H 3750 2376 50  0000 C CNN
-F 2 "Connector_IDC:IDC-Header_2x05_P2.54mm_Vertical" H 3700 2050 50  0001 C CNN
+F 2 "Connector_IDC:IDC-Header_2x06_P2.54mm_Vertical" H 3700 2050 50  0001 C CNN
 F 3 "~" H 3700 2050 50  0001 C CNN
 	1    3700 2050
@@
 $EndComp
 Wire Wire Line
-	3450 2250 3500 2250
+	3500 2350 3450 2350
 Wire Wire Line
-	4000 2250 4100 2250
+	3450 2350 3450 2400
+Text HLabel 4100 2250 2    50   Input ~ 0
+ENC_A
+Text HLabel 4100 2350 2    50   Input ~ 0
+ENC_B
 Wire Wire Line
-	4100 2250 4100 2350
+	4100 2250 4000 2250
 Wire Wire Line
-	4100 2150 4100 2250
-Connection ~ 4100 2250
+	4100 2350 4000 2350
 $EndSCHEMATC
