File: Nucleo-64-407.kicad_pcb (KiCad board)
At the start: 2 copper layers, 70 x 81 mm, 72 parts, among them J1 SWD, J3 USB_B_Micro, J4 Serial 0, J5 EXP1, J6 EXP2, J7 EXP3, J8 EXP4, SW1 RESET, SW2 BOOT, U1 STM32F407VETx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

Commit message: Switched nuc-f407 to rev 3.
Other:
- board text added: "Rev 3"
- board text removed: "Rev 2"
Changed lines of the file:
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@@
     (effects (font (size 1 1) (thickness 0.15)) (justify mirror))
   )
-  (gr_text "Rev 2" (at 114.2 42) (layer B.SilkS)
+  (gr_text "Rev 3" (at 114.2 42) (layer B.SilkS)
     (effects (font (size 1.5 1.5) (thickness 0.3)) (justify mirror))
   )

Commit message: Update ground routing for the MCU.
Routing:
- net /3.3V: track 315.2 -> 313.5 mm, vias 9 -> 8
- net GND: track 67.3 -> 68.9 mm
- net /SPI2_MISO: track 58.0 -> 57.2 mm
Other:
- board text added: "(c) iQury.us Jun 2019"
- board text added: "Rev 4"
- board text removed: "(c) iQury.us Dec 2018"
- board text removed: "Rev 3"
