File: MotorDriver_TMC2660.sch (KiCad schematic (older format))
At the start: 17 parts, among them U5 TMC2660

Commit message: Updated sense resistors to 1210 size. Moved heater LEDs to the center. Moved fan voltage LED to the rest of the power indicator LEDs.
Parts:
- R11, R13: footprint PrntrBoardV1:R_1206_3216Metric -> Resistor_SMD:R_1210_3225Metric
Changed lines of the file:
@@
 $Descr A4 11693 8268
 encoding utf-8
-Sheet 9 35
+Sheet 26 35
 Title ""
 Date ""
@@
 F 0 "R45" H 6320 5396 50  0000 L CNN
 F 1 "0R051" H 6320 5305 50  0000 L CNN
-F 2 "PrntrBoardV1:R_1206_3216Metric" V 6180 5350 50  0001 C CNN
+F 2 "Resistor_SMD:R_1210_3225Metric" V 6180 5350 50  0001 C CNN
 F 3 "~" H 6250 5350 50  0001 C CNN
 	1    6250 5350
@@
 F 0 "R47" H 7570 5196 50  0000 L CNN
 F 1 "0R051" H 7570 5105 50  0000 L CNN
-F 2 "PrntrBoardV1:R_1206_3216Metric" V 7430 5150 50  0001 C CNN
+F 2 "Resistor_SMD:R_1210_3225Metric" V 7430 5150 50  0001 C CNN
 F 3 "~" H 7500 5150 50  0001 C CNN
 	1    7500 5150
