File: EExtruder/EExtruder.sch (KiCad schematic (older format))
At the start: 35 parts, among them J1 20A 50V, J11 Conn_01x03_Male, J2 AudioJack4_Ground, U1 STM32F030C8Tx, U2 DCBuck, Y1 8MHz

Commit message: Component layout complete.
Parts:
- J2: footprint Connector_Audio:Jack_3.5mm_PJ320D_Horizontal -> PJ320D:Jack_3.5mm_PJ320D_Horizontal
- U2: footprint (none) -> DCBuck:Buck2217
- Y1: footprint Crystal:Crystal_SMD_HC49-SD_HandSoldering -> Crystal:Crystal_SMD_HC49-SD
Connections:
- wire segments 227 -> 231
Changed lines of the file:
@@
 F 0 "Y1" V 5696 2319 50  0000 R CNN
 F 1 "8MHz" V 5605 2319 50  0000 R CNN
-F 2 "Crystal:Crystal_SMD_HC49-SD_HandSoldering" H 5650 2450 50  0001 C CNN
+F 2 "Crystal:Crystal_SMD_HC49-SD" H 5650 2450 50  0001 C CNN
 F 3 "~" H 5650 2450 50  0001 C CNN
 	1    5650 2450
@@
 Text Label 2050 4250 0    50   ~ 0
 3.3V
-$Comp
-L BuckConverter:DCBuck U2
-U 1 1 5C1F761F
-P 1450 4400
-F 0 "U2" H 1450 4865 50  0000 C CNN
-F 1 "DCBuck" H 1450 4774 50  0000 C CNN
-F 2 "" H 1450 4400 50  0001 C CNN
-F 3 "" H 1450 4400 50  0001 C CNN
-	1    1450 4400
-	1    0    0    -1
-$EndComp
 Wire Wire Line
 	1800 4800 1800 5000
-Wire Wire Line
-	1100 4700 1100 5000
 $Comp
 L Connector:AudioJack4_Ground J2
@@
 F 0 "J2" H 1868 5892 50  0000 C CNN
 F 1 "AudioJack4_Ground" H 1868 5801 50  0000 C CNN
-F 2 "Connector_Audio:Jack_3.5mm_PJ320D_Horizontal" H 1900 5550 50  0001 C CNN
+F 2 "PJ320D:Jack_3.5mm_PJ320D_Horizontal" H 1900 5550 50  0001 C CNN
 F 3 "~" H 1900 5550 50  0001 C CNN
 	1    1900 5550
 	1    0    0    -1
 $EndComp
+$Comp
+L BuckConverter:DCBuck U2
+U 1 1 5BC116EF
+P 1450 4400
+F 0 "U2" H 1450 4865 50  0000 C CNN
+F 1 "DCBuck" H 1450 4774 50  0000 C CNN
+F 2 "DCBuck:Buck2217" H 1450 4400 50  0001 C CNN
+F 3 "" H 1450 4400 50  0001 C CNN
+	1    1450 4400
+	1    0    0    -1
+$EndComp
+Wire Wire Line
+	1100 4800 1100 5000
+Wire Wire Line
+	1100 4250 1100 4350
+Connection ~ 1100 4250
+Wire Wire Line
+	1800 4350 1800 4250
+Connection ~ 1800 4250
+Wire Wire Line
+	1800 4700 1800 4800
+Connection ~ 1800 4800
+Wire Wire Line
+	1100 4700 1100 4800
+Connection ~ 1100 4800
 $EndSCHEMATC

Commit message: Ready to manufacture.
Parts:
- added H1, H2: MountingHole, MountingHole:MountingHole_3.2mm_M3, symbol Mechanical:MountingHole
Changed lines of the file:
@@
 	1100 4700 1100 4800
 Connection ~ 1100 4800
+$Comp
+L Mechanical:MountingHole H1
+U 1 1 5BC3C6F1
+P 8700 5450
+F 0 "H1" H 8800 5496 50  0000 L CNN
+F 1 "MountingHole" H 8800 5405 50  0000 L CNN
+F 2 "MountingHole:MountingHole_3.2mm_M3" H 8700 5450 50  0001 C CNN
+F 3 "~" H 8700 5450 50  0001 C CNN
+	1    8700 5450
+	1    0    0    -1
+$EndComp
+$Comp
+L Mechanical:MountingHole H2
+U 1 1 5BC42E42
+P 9450 5450
+F 0 "H2" H 9550 5496 50  0000 L CNN
+F 1 "MountingHole" H 9550 5405 50  0000 L CNN
+F 2 "MountingHole:MountingHole_3.2mm_M3" H 9450 5450 50  0001 C CNN
+F 3 "~" H 9450 5450 50  0001 C CNN
+	1    9450 5450
+	1    0    0    -1
+$EndComp
 $EndSCHEMATC

Commit message: Select correct terminals. Use old style square footprints.
Parts:
- C1, C10, C2, C3, C4, C5, C6, C7, C8, C9: footprint Capacitor_SMD:C_0603_1608Metric -> Local:C_0603_1608Metric
- J1: footprint Connector_Phoenix_MC:PhoenixContact_MCV_1,5_2-G-3.5_1x02_P3.50mm_Vertical -> Local:TerminalBlock_Phoenix_PT-1,5-2-3.5-H_1x02_P3.50mm_Horizontal
- R1, R2, R3, R4, R5, R6, R7, R8: footprint Resistor_SMD:R_0603_1608Metric -> Local:R_0603_1608Metric
- SWD1, TC0, TC1: footprint Connector_PinSocket_2.54mm:PinSocket_1x05_P2.54mm_Vertical -> Connector_PinHeader_2.54mm:PinHeader_1x05_P2.54mm_Vertical
Changed lines of the file:
@@
 F 0 "R6" V 6600 2200 50  0000 C CNN
 F 1 "10k" V 6600 2050 50  0000 C CNN
-F 2 "Resistor_SMD:R_0603_1608Metric" V 6430 2050 50  0001 C CNN
+F 2 "Local:R_0603_1608Metric" V 6430 2050 50  0001 C CNN
 F 3 "~" H 6500 2050 50  0001 C CNN
 	1    6500 2050
@@
 F 0 "R8" V 7293 1050 50  0000 C CNN
 F 1 "1R5" V 7384 1050 50  0000 C CNN
-F 2 "Resistor_SMD:R_0603_1608Metric" V 7430 1050 50  0001 C CNN
+F 2 "Local:R_0603_1608Metric" V 7430 1050 50  0001 C CNN
 F 3 "~" H 7500 1050 50  0001 C CNN
 	1    7500 1050
@@
 F 0 "C9" H 8065 1246 50  0000 L CNN
 F 1 "1uF" H 8065 1155 50  0000 L CNN
-F 2 "Capacitor_SMD:C_0603_1608Metric" H 7988 1050 50  0001 C CNN
+F 2 "Local:C_0603_1608Metric" H 7988 1050 50  0001 C CNN
 F 3 "~" H 7950 1200 50  0001 C CNN
 	1    7950 1200
@@
 F 0 "C10" H 8415 1246 50  0000 L CNN
 F 1 "10nF" H 8415 1155 50  0000 L CNN
-F 2 "Capacitor_SMD:C_0603_1608Metric" H 8338 1050 50  0001 C CNN
+F 2 "Local:C_0603_1608Metric" H 8338 1050 50  0001 C CNN
 F 3 "~" H 8300 1200 50  0001 C CNN
 	1    8300 1200
@@
 F 0 "C7" H 6050 1750 50  0000 L CNN
 F 1 "100nF" H 5950 1650 50  0000 L CNN
-F 2 "Capacitor_SMD:C_0603_1608Metric" H 6338 1550 50  0001 C CNN
+F 2 "Local:C_0603_1608Metric" H 6338 1550 50  0001 C CNN
 F 3 "~" H 6300 1700 50  0001 C CNN
 	1    6300 1700
@@
 F 0 "C2" H 5165 1596 50  0000 L CNN
 F 1 "100nF" H 5100 1450 50  0000 L CNN
-F 2 "Capacitor_SMD:C_0603_1608Metric" H 5088 1400 50  0001 C CNN
+F 2 "Local:C_0603_1608Metric" H 5088 1400 50  0001 C CNN
 F 3 "~" H 5050 1550 50  0001 C CNN
 	1    5050 1550
@@
 F 0 "C5" H 5515 1596 50  0000 L CNN
 F 1 "100nF" H 5450 1450 50  0000 L CNN
-F 2 "Capacitor_SMD:C_0603_1608Metric" H 5438 1400 50  0001 C CNN
+F 2 "Local:C_0603_1608Metric" H 5438 1400 50  0001 C CNN
 F 3 "~" H 5400 1550 50  0001 C CNN
 	1    5400 1550
@@
 F 0 "C6" H 5815 1596 50  0000 L CNN
 F 1 "100nF" H 5750 1450 50  0000 L CNN
-F 2 "Capacitor_SMD:C_0603_1608Metric" H 5738 1400 50  0001 C CNN
+F 2 "Local:C_0603_1608Metric" H 5738 1400 50  0001 C CNN
 F 3 "~" H 5700 1550 50  0001 C CNN
 	1    5700 1550
@@
 F 0 "C1" H 4865 1596 50  0000 L CNN
 F 1 "10uF" H 4800 1450 50  0000 L CNN
-F 2 "Capacitor_SMD:C_0603_1608Metric" H 4788 1400 50  0001 C CNN
+F 2 "Local:C_0603_1608Metric" H 4788 1400 50  0001 C CNN
 F 3 "~" H 4750 1550 50  0001 C CNN
 	1    4750 1550
@@
 F 0 "R3" V 6050 2250 50  0000 C CNN
 F 1 "0" V 6050 2350 50  0000 C CNN
-F 2 "Resistor_SMD:R_0603_1608Metric" V 5880 2250 50  0001 C CNN
+F 2 "Local:R_0603_1608Metric" V 5880 2250 50  0001 C CNN
 F 3 "~" H 5950 2250 50  0001 C CNN
 	1    5950 2250
@@
 F 0 "R4" V 6150 2600 50  0000 C CNN
 F 1 "390" V 6050 2600 50  0000 C CNN
-F 2 "Resistor_SMD:R_0603_1608Metric" V 5880 2600 50  0001 C CNN
+F 2 "Local:R_0603_1608Metric" V 5880 2600 50  0001 C CNN
 F 3 "~" H 5950 2600 50  0001 C CNN
 	1    5950 2600
@@
 F 0 "C3" V 5250 2350 50  0000 C CNN
 F 1 "20pF" V 5500 2250 50  0000 C CNN
-F 2 "Capacitor_SMD:C_0603_1608Metric" H 5388 2100 50  0001 C CNN
+F 2 "Local:C_0603_1608Metric" H 5388 2100 50  0001 C CNN
 F 3 "~" H 5350 2250 50  0001 C CNN
 	1    5350 2250
@@
 F 0 "C4" V 5600 2650 50  0000 C CNN
 F 1 "20pF" V 5500 2600 50  0000 C CNN
-F 2 "Capacitor_SMD:C_0603_1608Metric" H 5388 2450 50  0001 C CNN
+F 2 "Local:C_0603_1608Metric" H 5388 2450 50  0001 C CNN
 F 3 "~" H 5350 2600 50  0001 C CNN
 	1    5350 2600
@@
 F 0 "R1" H 2520 5246 50  0000 L CNN
 F 1 "10k" H 2520 5155 50  0000 L CNN
-F 2 "Resistor_SMD:R_0603_1608Metric" V 2380 5200 50  0001 C CNN
+F 2 "Local:R_0603_1608Metric" V 2380 5200 50  0001 C CNN
 F 3 "~" H 2450 5200 50  0001 C CNN
 	1    2450 5200
@@
 F 0 "R2" H 2770 5246 50  0000 L CNN
 F 1 "10k" H 2770 5155 50  0000 L CNN
-F 2 "Resistor_SMD:R_0603_1608Metric" V 2630 5200 50  0001 C CNN
+F 2 "Local:R_0603_1608Metric" V 2630 5200 50  0001 C CNN
 F 3 "~" H 2700 5200 50  0001 C CNN
 	1    2700 5200
@@
 L Connector:Screw_Terminal_01x02 J1
 U 1 1 5BC959F9
-P 1350 950
-F 0 "J1" H 1268 625 50  0000 C CNN
-F 1 "20A 50V" H 1268 716 50  0000 C CNN
-F 2 "Connector_Phoenix_MC:PhoenixContact_MCV_1,5_2-G-3.5_1x02_P3.50mm_Vertical" H 1350 950 50  0001 C CNN
-F 3 "~" H 1350 950 50  0001 C CNN
-	1    1350 950
-	-1   0    0    1
+P 1350 850
+F 0 "J1" H 1350 550 50  0000 C CNN
+F 1 "20A 50V" H 1400 650 50  0000 C CNN
+F 2 "Local:TerminalBlock_Phoenix_PT-1,5-2-3.5-H_1x02_P3.50mm_Horizontal" H 1350 850 50  0001 C CNN
+F 3 "~" H 1350 850 50  0001 C CNN
+	1    1350 850
+	-1   0    0    -1
 $EndComp
 Wire Wire Line
@@
 F 0 "TC1" H 5108 5131 50  0000 C CNN
 F 1 "Conn_01x05_Male" H 5108 5040 50  0000 C CNN
-F 2 "Connector_PinSocket_2.54mm:PinSocket_1x05_P2.54mm_Vertical" H 5000 4750 50  0001 C CNN
+F 2 "Connector_PinHeader_2.54mm:PinHeader_1x05_P2.54mm_Vertical" H 5000 4750 50  0001 C CNN
 F 3 "~" H 5000 4750 50  0001 C CNN
 	1    5000 4750
@@
 F 0 "TC0" H 5100 5100 50  0000 C CNN
 F 1 "Conn_01x05_Male" H 5250 5200 50  0000 C CNN
-F 2 "Connector_PinSocket_2.54mm:PinSocket_1x05_P2.54mm_Vertical" H 5000 5450 50  0001 C CNN
+F 2 "Connector_PinHeader_2.54mm:PinHeader_1x05_P2.54mm_Vertical" H 5000 5450 50  0001 C CNN
 F 3 "~" H 5000 5450 50  0001 C CNN
 	1    5000 5450
@@
 F 0 "R7" H 7420 5546 50  0000 L CNN
 F 1 "10k" H 7420 5455 50  0000 L CNN
-F 2 "Resistor_SMD:R_0603_1608Metric" V 7280 5500 50  0001 C CNN
+F 2 "Local:R_0603_1608Metric" V 7280 5500 50  0001 C CNN
 F 3 "~" H 7350 5500 50  0001 C CNN
 	1    7350 5500
@@
 F 0 "R5" H 6100 5550 50  0000 L CNN
 F 1 "10k" H 6050 5450 50  0000 L CNN
-F 2 "Resistor_SMD:R_0603_1608Metric" V 6180 5500 50  0001 C CNN
+F 2 "Local:R_0603_1608Metric" V 6180 5500 50  0001 C CNN
 F 3 "~" H 6250 5500 50  0001 C CNN
 	1    6250 5500
@@
 F 0 "C8" H 7315 6396 50  0000 L CNN
 F 1 "1uF" H 7315 6305 50  0000 L CNN
-F 2 "Capacitor_SMD:C_0603_1608Metric" H 7238 6200 50  0001 C CNN
+F 2 "Local:C_0603_1608Metric" H 7238 6200 50  0001 C CNN
 F 3 "~" H 7200 6350 50  0001 C CNN
 	1    7200 6350
@@
 F 0 "SWD1" H 9772 2382 50  0000 R CNN
 F 1 "Conn_01x05_Male" H 9772 2473 50  0000 R CNN
-F 2 "Connector_PinSocket_2.54mm:PinSocket_1x05_P2.54mm_Vertical" H 9800 2450 50  0001 C CNN
+F 2 "Connector_PinHeader_2.54mm:PinHeader_1x05_P2.54mm_Vertical" H 9800 2450 50  0001 C CNN
 F 3 "~" H 9800 2450 50  0001 C CNN
 	1    9800 2450

Commit message: Add solder jumper on the audio jack to avoid ground loops.
Parts:
- added JP2: SolderJumper_2_Open, Jumper:SolderJumper-2_P1.3mm_Open_TrianglePad1.0x1.5mm, symbol Jumper:SolderJumper_2_Open
Changed lines of the file:
@@
 Wire Wire Line
 	2100 5550 2400 5550
-Wire Wire Line
-	2850 5550 2850 5900
 $Comp
 L power:GND #PWR02
@@
 	1    0    0    -1
 $EndComp
+$Comp
+L Jumper:SolderJumper_2_Open JP2
+U 1 1 5BC4D384
+P 2850 5700
+F 0 "JP2" V 2804 5768 50  0000 L CNN
+F 1 "SolderJumper_2_Open" V 2895 5768 50  0000 L CNN
+F 2 "Jumper:SolderJumper-2_P1.3mm_Open_TrianglePad1.0x1.5mm" H 2850 5700 50  0001 C CNN
+F 3 "~" H 2850 5700 50  0001 C CNN
+	1    2850 5700
+	0    1    1    0
+$EndComp
+Wire Wire Line
+	2850 5850 2850 5900
 $EndSCHEMATC

Commit message: Add fiducials.
Parts:
- added FID1, FID2: Fiducial, Local:Fiducial_1mm_Dia_2.54mm_Outer_CopperTop, symbol Mechanical:MountingHole
Changed lines of the file:
@@
 Wire Wire Line
 	2850 5850 2850 5900
+$Comp
+L Mechanical:MountingHole FID1
+U 1 1 5BC5F696
+P 8700 5900
+F 0 "FID1" H 8800 5946 50  0000 L CNN
+F 1 "Fiducial" H 8800 5855 50  0000 L CNN
+F 2 "Local:Fiducial_1mm_Dia_2.54mm_Outer_CopperTop" H 8700 5900 50  0001 C CNN
+F 3 "~" H 8700 5900 50  0001 C CNN
+	1    8700 5900
+	1    0    0    -1
+$EndComp
+$Comp
+L Mechanical:MountingHole FID2
+U 1 1 5BC636A0
+P 9450 5900
+F 0 "FID2" H 9550 5946 50  0000 L CNN
+F 1 "Fiducial" H 9550 5855 50  0000 L CNN
+F 2 "Local:Fiducial_1mm_Dia_2.54mm_Outer_CopperTop" H 9450 5900 50  0001 C CNN
+F 3 "~" H 9450 5900 50  0001 C CNN
+	1    9450 5900
+	1    0    0    -1
+$EndComp
 $EndSCHEMATC
