File: EExtruder/Heater.sch (KiCad schematic (older format))
At the start: 10 parts, among them J3 6A 50V, Q1 DTC124E, Q2 PSMN7R0-30YL

Commit message: Component layout complete.
Changed lines of the file:
@@
 AR Path="/5BBB311C/5BBB34F6" Ref="Q2"  Part="1"
 AR Path="/5BBB43B6/5BBB34F6" Ref="Q4"  Part="1"
-F 0 "Q2" H 5956 3196 50  0000 L CNN
+F 0 "Q4" H 5956 3196 50  0000 L CNN
 F 1 "PSMN7R0-30YL" H 5956 3105 50  0000 L CNN
 F 2 "Package_TO_SOT_SMD:LFPAK56" H 5900 3150 50  0001 C CNN
@@
 AR Path="/5BBB311C/5BBB34FD" Ref="Q1"  Part="1"
 AR Path="/5BBB43B6/5BBB34FD" Ref="Q3"  Part="1"
-F 0 "Q1" H 5237 3346 50  0000 L CNN
+F 0 "Q3" H 5237 3346 50  0000 L CNN
 F 1 "DTC124E" H 4750 3500 50  0000 L CNN
 F 2 "Package_TO_SOT_SMD:SOT-23" H 5050 3300 50  0001 L CNN
@@
 AR Path="/5BBB311C/5BBB3504" Ref="R11"  Part="1"
 AR Path="/5BBB43B6/5BBB3504" Ref="R15"  Part="1"
-F 0 "R11" H 5470 3396 50  0000 L CNN
+F 0 "R15" H 5470 3396 50  0000 L CNN
 F 1 "10K" H 5470 3305 50  0000 L CNN
 F 2 "Resistor_SMD:R_0603_1608Metric" V 5330 3350 50  0001 C CNN
@@
 AR Path="/5BBB311C/5BBB350B" Ref="R10"  Part="1"
 AR Path="/5BBB43B6/5BBB350B" Ref="R14"  Part="1"
-F 0 "R10" H 5330 2654 50  0000 R CNN
+F 0 "R14" H 5330 2654 50  0000 R CNN
 F 1 "10K" H 5330 2745 50  0000 R CNN
 F 2 "Resistor_SMD:R_0603_1608Metric" V 5330 2700 50  0001 C CNN
@@
 AR Path="/5BBB311C/5BBB3512" Ref="R12"  Part="1"
 AR Path="/5BBB43B6/5BBB3512" Ref="R16"  Part="1"
-F 0 "R12" H 5920 2446 50  0000 L CNN
+F 0 "R16" H 5920 2446 50  0000 L CNN
 F 1 "10K" H 5920 2355 50  0000 L CNN
 F 2 "Resistor_SMD:R_0603_1608Metric" V 5780 2400 50  0001 C CNN
@@
 AR Path="/5BBB311C/5BBB3519" Ref="D1"  Part="1"
 AR Path="/5BBB43B6/5BBB3519" Ref="D3"  Part="1"
-F 0 "D1" V 5888 2632 50  0000 R CNN
+F 0 "D3" V 5888 2632 50  0000 R CNN
 F 1 "RED" V 5797 2632 50  0000 R CNN
 F 2 "Diode_SMD:D_0603_1608Metric" H 5850 2750 50  0001 C CNN
@@
 AR Path="/5BBB311C/5BBB3520" Ref="D2"  Part="1"
 AR Path="/5BBB43B6/5BBB3520" Ref="D4"  Part="1"
-F 0 "D2" V 6154 2729 50  0000 L CNN
+F 0 "D4" V 6154 2729 50  0000 L CNN
 F 1 "1N4148" V 6245 2729 50  0000 L CNN
 F 2 "Diode_SMD:D_SOD-323_HandSoldering" H 6200 2475 50  0001 C CNN
@@
 AR Path="/5BBB311C/5BBB3527" Ref="C11"  Part="1"
 AR Path="/5BBB43B6/5BBB3527" Ref="C12"  Part="1"
-F 0 "C11" H 5015 2596 50  0000 L CNN
+F 0 "C12" H 5015 2596 50  0000 L CNN
 F 1 "10uF 50V" H 5015 2505 50  0000 L CNN
 F 2 "Capacitor_SMD:C_1206_3216Metric" H 4938 2400 50  0001 C CNN
@@
 AR Path="/5BBB311C/5BBB353A" Ref="#PWR010"  Part="1"
 AR Path="/5BBB43B6/5BBB353A" Ref="#PWR012"  Part="1"
-F 0 "#PWR010" H 5750 3400 50  0001 C CNN
+F 0 "#PWR012" H 5750 3400 50  0001 C CNN
 F 1 "GND" H 5755 3477 50  0000 C CNN
 F 2 "" H 5750 3650 50  0001 C CNN
@@
 AR Path="/5BBB311C/5BBB3540" Ref="#PWR09"  Part="1"
 AR Path="/5BBB43B6/5BBB3540" Ref="#PWR011"  Part="1"
-F 0 "#PWR09" H 4900 2500 50  0001 C CNN
+F 0 "#PWR011" H 4900 2500 50  0001 C CNN
 F 1 "GND" H 4905 2577 50  0000 C CNN
 F 2 "" H 4900 2750 50  0001 C CNN
@@
 AR Path="/5BBB311C/5BBB355D" Ref="R9"  Part="1"
 AR Path="/5BBB43B6/5BBB355D" Ref="R13"  Part="1"
-F 0 "R9" H 4570 3096 50  0000 L CNN
+F 0 "R13" H 4570 3096 50  0000 L CNN
 F 1 "10k" H 4570 3005 50  0000 L CNN
 F 2 "Resistor_SMD:R_0603_1608Metric" V 4430 3050 50  0001 C CNN
@@
 AR Path="/5BBB311C/5BBED217" Ref="J3"  Part="1"
 AR Path="/5BBB43B6/5BBED217" Ref="J4"  Part="1"
-F 0 "J3" H 7230 2792 50  0000 L CNN
+F 0 "J4" H 7230 2792 50  0000 L CNN
 F 1 "6A 50V" H 7230 2701 50  0000 L CNN
 F 2 "Connector_Phoenix_MC:PhoenixContact_MCV_1,5_2-G-3.5_1x02_P3.50mm_Vertical" H 7150 2800 50  0001 C CNN

Commit message: Select correct terminals. Use old style square footprints.
Parts:
- C11: footprint Capacitor_SMD:C_1206_3216Metric -> Local:C_1206_3216Metric
- J3: footprint Connector_Phoenix_MC:PhoenixContact_MCV_1,5_2-G-3.5_1x02_P3.50mm_Vertical -> Local:TerminalBlock_Phoenix_PT-1,5-2-3.5-H_1x02_P3.50mm_Horizontal
- R10, R11, R12, R9: footprint Resistor_SMD:R_0603_1608Metric -> Local:R_0603_1608Metric
Connections:
- net VIN: now also J3.2 (Pin_2); no longer J3.1 (Pin_1)
- net at D1.1 (K), D2.2 (A), Q2.5 (D): now also J3.1 (Pin_1); no longer J3.2 (Pin_2)
Changed lines of the file:
@@
 AR Path="/5BBB311C/5BBB34F6" Ref="Q2"  Part="1"
 AR Path="/5BBB43B6/5BBB34F6" Ref="Q4"  Part="1"
-F 0 "Q4" H 5956 3196 50  0000 L CNN
+F 0 "Q2" H 5956 3196 50  0000 L CNN
 F 1 "PSMN7R0-30YL" H 5956 3105 50  0000 L CNN
 F 2 "Package_TO_SOT_SMD:LFPAK56" H 5900 3150 50  0001 C CNN
@@
 AR Path="/5BBB311C/5BBB34FD" Ref="Q1"  Part="1"
 AR Path="/5BBB43B6/5BBB34FD" Ref="Q3"  Part="1"
-F 0 "Q3" H 5237 3346 50  0000 L CNN
+F 0 "Q1" H 5237 3346 50  0000 L CNN
 F 1 "DTC124E" H 4750 3500 50  0000 L CNN
 F 2 "Package_TO_SOT_SMD:SOT-23" H 5050 3300 50  0001 L CNN
@@
 AR Path="/5BBB311C/5BBB3504" Ref="R11"  Part="1"
 AR Path="/5BBB43B6/5BBB3504" Ref="R15"  Part="1"
-F 0 "R15" H 5470 3396 50  0000 L CNN
+F 0 "R11" H 5470 3396 50  0000 L CNN
 F 1 "10K" H 5470 3305 50  0000 L CNN
-F 2 "Resistor_SMD:R_0603_1608Metric" V 5330 3350 50  0001 C CNN
+F 2 "Local:R_0603_1608Metric" V 5330 3350 50  0001 C CNN
 F 3 "~" H 5400 3350 50  0001 C CNN
 	1    5400 3350
@@
 AR Path="/5BBB311C/5BBB350B" Ref="R10"  Part="1"
 AR Path="/5BBB43B6/5BBB350B" Ref="R14"  Part="1"
-F 0 "R14" H 5330 2654 50  0000 R CNN
+F 0 "R10" H 5330 2654 50  0000 R CNN
 F 1 "10K" H 5330 2745 50  0000 R CNN
-F 2 "Resistor_SMD:R_0603_1608Metric" V 5330 2700 50  0001 C CNN
+F 2 "Local:R_0603_1608Metric" V 5330 2700 50  0001 C CNN
 F 3 "~" H 5400 2700 50  0001 C CNN
 	1    5400 2700
@@
 AR Path="/5BBB311C/5BBB3512" Ref="R12"  Part="1"
 AR Path="/5BBB43B6/5BBB3512" Ref="R16"  Part="1"
-F 0 "R16" H 5920 2446 50  0000 L CNN
+F 0 "R12" H 5920 2446 50  0000 L CNN
 F 1 "10K" H 5920 2355 50  0000 L CNN
-F 2 "Resistor_SMD:R_0603_1608Metric" V 5780 2400 50  0001 C CNN
+F 2 "Local:R_0603_1608Metric" V 5780 2400 50  0001 C CNN
 F 3 "~" H 5850 2400 50  0001 C CNN
 	1    5850 2400
@@
 AR Path="/5BBB311C/5BBB3519" Ref="D1"  Part="1"
 AR Path="/5BBB43B6/5BBB3519" Ref="D3"  Part="1"
-F 0 "D3" V 5888 2632 50  0000 R CNN
+F 0 "D1" V 5888 2632 50  0000 R CNN
 F 1 "RED" V 5797 2632 50  0000 R CNN
 F 2 "Diode_SMD:D_0603_1608Metric" H 5850 2750 50  0001 C CNN
@@
 AR Path="/5BBB311C/5BBB3520" Ref="D2"  Part="1"
 AR Path="/5BBB43B6/5BBB3520" Ref="D4"  Part="1"
-F 0 "D4" V 6154 2729 50  0000 L CNN
+F 0 "D2" V 6154 2729 50  0000 L CNN
 F 1 "1N4148" V 6245 2729 50  0000 L CNN
 F 2 "Diode_SMD:D_SOD-323_HandSoldering" H 6200 2475 50  0001 C CNN
@@
 AR Path="/5BBB311C/5BBB3527" Ref="C11"  Part="1"
 AR Path="/5BBB43B6/5BBB3527" Ref="C12"  Part="1"
-F 0 "C12" H 5015 2596 50  0000 L CNN
+F 0 "C11" H 5015 2596 50  0000 L CNN
 F 1 "10uF 50V" H 5015 2505 50  0000 L CNN
-F 2 "Capacitor_SMD:C_1206_3216Metric" H 4938 2400 50  0001 C CNN
+F 2 "Local:C_1206_3216Metric" H 4938 2400 50  0001 C CNN
 F 3 "~" H 4900 2550 50  0001 C CNN
 	1    4900 2550
@@
 AR Path="/5BBB311C/5BBB353A" Ref="#PWR010"  Part="1"
 AR Path="/5BBB43B6/5BBB353A" Ref="#PWR012"  Part="1"
-F 0 "#PWR012" H 5750 3400 50  0001 C CNN
+F 0 "#PWR010" H 5750 3400 50  0001 C CNN
 F 1 "GND" H 5755 3477 50  0000 C CNN
 F 2 "" H 5750 3650 50  0001 C CNN
@@
 AR Path="/5BBB311C/5BBB3540" Ref="#PWR09"  Part="1"
 AR Path="/5BBB43B6/5BBB3540" Ref="#PWR011"  Part="1"
-F 0 "#PWR011" H 4900 2500 50  0001 C CNN
+F 0 "#PWR09" H 4900 2500 50  0001 C CNN
 F 1 "GND" H 4905 2577 50  0000 C CNN
 F 2 "" H 4900 2750 50  0001 C CNN
@@
 AR Path="/5BBB311C/5BBB355D" Ref="R9"  Part="1"
 AR Path="/5BBB43B6/5BBB355D" Ref="R13"  Part="1"
-F 0 "R13" H 4570 3096 50  0000 L CNN
+F 0 "R9" H 4570 3096 50  0000 L CNN
 F 1 "10k" H 4570 3005 50  0000 L CNN
-F 2 "Resistor_SMD:R_0603_1608Metric" V 4430 3050 50  0001 C CNN
+F 2 "Local:R_0603_1608Metric" V 4430 3050 50  0001 C CNN
 F 3 "~" H 4500 3050 50  0001 C CNN
 	1    4500 3050
@@
 L Connector:Screw_Terminal_01x02 J3
 U 1 1 5BBED217
-P 7150 2800
+P 7150 2900
 AR Path="/5BBB311C/5BBED217" Ref="J3"  Part="1"
 AR Path="/5BBB43B6/5BBED217" Ref="J4"  Part="1"
-F 0 "J4" H 7230 2792 50  0000 L CNN
-F 1 "6A 50V" H 7230 2701 50  0000 L CNN
-F 2 "Connector_Phoenix_MC:PhoenixContact_MCV_1,5_2-G-3.5_1x02_P3.50mm_Vertical" H 7150 2800 50  0001 C CNN
-F 3 "~" H 7150 2800 50  0001 C CNN
-	1    7150 2800
-	1    0    0    -1
+F 0 "J3" H 7230 2892 50  0000 L CNN
+F 1 "6A 50V" H 7230 2801 50  0000 L CNN
+F 2 "Local:TerminalBlock_Phoenix_PT-1,5-2-3.5-H_1x02_P3.50mm_Horizontal" H 7150 2900 50  0001 C CNN
+F 3 "~" H 7150 2900 50  0001 C CNN
+	1    7150 2900
+	1    0    0    1
 $EndComp
 $EndSCHEMATC

Commit message: Add solder jumper on the audio jack to avoid ground loops.
Changed lines of the file:
@@
 AR Path="/5BBB311C/5BBB34F6" Ref="Q2"  Part="1"
 AR Path="/5BBB43B6/5BBB34F6" Ref="Q4"  Part="1"
-F 0 "Q2" H 5956 3196 50  0000 L CNN
+F 0 "Q4" H 5956 3196 50  0000 L CNN
 F 1 "PSMN7R0-30YL" H 5956 3105 50  0000 L CNN
 F 2 "Package_TO_SOT_SMD:LFPAK56" H 5900 3150 50  0001 C CNN
@@
 AR Path="/5BBB311C/5BBB34FD" Ref="Q1"  Part="1"
 AR Path="/5BBB43B6/5BBB34FD" Ref="Q3"  Part="1"
-F 0 "Q1" H 5237 3346 50  0000 L CNN
+F 0 "Q3" H 5237 3346 50  0000 L CNN
 F 1 "DTC124E" H 4750 3500 50  0000 L CNN
 F 2 "Package_TO_SOT_SMD:SOT-23" H 5050 3300 50  0001 L CNN
@@
 AR Path="/5BBB311C/5BBB3504" Ref="R11"  Part="1"
 AR Path="/5BBB43B6/5BBB3504" Ref="R15"  Part="1"
-F 0 "R11" H 5470 3396 50  0000 L CNN
+F 0 "R15" H 5470 3396 50  0000 L CNN
 F 1 "10K" H 5470 3305 50  0000 L CNN
 F 2 "Local:R_0603_1608Metric" V 5330 3350 50  0001 C CNN
@@
 AR Path="/5BBB311C/5BBB350B" Ref="R10"  Part="1"
 AR Path="/5BBB43B6/5BBB350B" Ref="R14"  Part="1"
-F 0 "R10" H 5330 2654 50  0000 R CNN
+F 0 "R14" H 5330 2654 50  0000 R CNN
 F 1 "10K" H 5330 2745 50  0000 R CNN
 F 2 "Local:R_0603_1608Metric" V 5330 2700 50  0001 C CNN
@@
 AR Path="/5BBB311C/5BBB3512" Ref="R12"  Part="1"
 AR Path="/5BBB43B6/5BBB3512" Ref="R16"  Part="1"
-F 0 "R12" H 5920 2446 50  0000 L CNN
+F 0 "R16" H 5920 2446 50  0000 L CNN
 F 1 "10K" H 5920 2355 50  0000 L CNN
 F 2 "Local:R_0603_1608Metric" V 5780 2400 50  0001 C CNN
@@
 AR Path="/5BBB311C/5BBB3519" Ref="D1"  Part="1"
 AR Path="/5BBB43B6/5BBB3519" Ref="D3"  Part="1"
-F 0 "D1" V 5888 2632 50  0000 R CNN
+F 0 "D3" V 5888 2632 50  0000 R CNN
 F 1 "RED" V 5797 2632 50  0000 R CNN
 F 2 "Diode_SMD:D_0603_1608Metric" H 5850 2750 50  0001 C CNN
@@
 AR Path="/5BBB311C/5BBB3520" Ref="D2"  Part="1"
 AR Path="/5BBB43B6/5BBB3520" Ref="D4"  Part="1"
-F 0 "D2" V 6154 2729 50  0000 L CNN
+F 0 "D4" V 6154 2729 50  0000 L CNN
 F 1 "1N4148" V 6245 2729 50  0000 L CNN
 F 2 "Diode_SMD:D_SOD-323_HandSoldering" H 6200 2475 50  0001 C CNN
@@
 AR Path="/5BBB311C/5BBB3527" Ref="C11"  Part="1"
 AR Path="/5BBB43B6/5BBB3527" Ref="C12"  Part="1"
-F 0 "C11" H 5015 2596 50  0000 L CNN
+F 0 "C12" H 5015 2596 50  0000 L CNN
 F 1 "10uF 50V" H 5015 2505 50  0000 L CNN
 F 2 "Local:C_1206_3216Metric" H 4938 2400 50  0001 C CNN
@@
 AR Path="/5BBB311C/5BBB353A" Ref="#PWR010"  Part="1"
 AR Path="/5BBB43B6/5BBB353A" Ref="#PWR012"  Part="1"
-F 0 "#PWR010" H 5750 3400 50  0001 C CNN
+F 0 "#PWR012" H 5750 3400 50  0001 C CNN
 F 1 "GND" H 5755 3477 50  0000 C CNN
 F 2 "" H 5750 3650 50  0001 C CNN
@@
 AR Path="/5BBB311C/5BBB3540" Ref="#PWR09"  Part="1"
 AR Path="/5BBB43B6/5BBB3540" Ref="#PWR011"  Part="1"
-F 0 "#PWR09" H 4900 2500 50  0001 C CNN
+F 0 "#PWR011" H 4900 2500 50  0001 C CNN
 F 1 "GND" H 4905 2577 50  0000 C CNN
 F 2 "" H 4900 2750 50  0001 C CNN
@@
 AR Path="/5BBB311C/5BBB355D" Ref="R9"  Part="1"
 AR Path="/5BBB43B6/5BBB355D" Ref="R13"  Part="1"
-F 0 "R9" H 4570 3096 50  0000 L CNN
+F 0 "R13" H 4570 3096 50  0000 L CNN
 F 1 "10k" H 4570 3005 50  0000 L CNN
 F 2 "Local:R_0603_1608Metric" V 4430 3050 50  0001 C CNN
@@
 AR Path="/5BBB311C/5BBED217" Ref="J3"  Part="1"
 AR Path="/5BBB43B6/5BBED217" Ref="J4"  Part="1"
-F 0 "J3" H 7230 2892 50  0000 L CNN
+F 0 "J4" H 7230 2892 50  0000 L CNN
 F 1 "6A 50V" H 7230 2801 50  0000 L CNN
 F 2 "Local:TerminalBlock_Phoenix_PT-1,5-2-3.5-H_1x02_P3.50mm_Horizontal" H 7150 2900 50  0001 C CNN

Commit message: Added 3.3V LDO, updated TC connectors to 6 pins. Re-arranged the layout.
Changed lines of the file:
@@
 EESchema Schematic File Version 4
 LIBS:EExtruder-cache
-EELAYER 28 0
+EELAYER 29 0
 EELAYER END
 $Descr A4 11693 8268
@@
 AR Path="/5BBB311C/5BBB34F6" Ref="Q2"  Part="1"
 AR Path="/5BBB43B6/5BBB34F6" Ref="Q4"  Part="1"
-F 0 "Q4" H 5956 3196 50  0000 L CNN
+F 0 "Q2" H 5956 3196 50  0000 L CNN
 F 1 "PSMN7R0-30YL" H 5956 3105 50  0000 L CNN
 F 2 "Package_TO_SOT_SMD:LFPAK56" H 5900 3150 50  0001 C CNN
@@
 AR Path="/5BBB311C/5BBB34FD" Ref="Q1"  Part="1"
 AR Path="/5BBB43B6/5BBB34FD" Ref="Q3"  Part="1"
-F 0 "Q3" H 5237 3346 50  0000 L CNN
+F 0 "Q1" H 5237 3346 50  0000 L CNN
 F 1 "DTC124E" H 4750 3500 50  0000 L CNN
 F 2 "Package_TO_SOT_SMD:SOT-23" H 5050 3300 50  0001 L CNN
@@
 AR Path="/5BBB311C/5BBB3504" Ref="R11"  Part="1"
 AR Path="/5BBB43B6/5BBB3504" Ref="R15"  Part="1"
-F 0 "R15" H 5470 3396 50  0000 L CNN
+F 0 "R11" H 5470 3396 50  0000 L CNN
 F 1 "10K" H 5470 3305 50  0000 L CNN
 F 2 "Local:R_0603_1608Metric" V 5330 3350 50  0001 C CNN
@@
 AR Path="/5BBB311C/5BBB350B" Ref="R10"  Part="1"
 AR Path="/5BBB43B6/5BBB350B" Ref="R14"  Part="1"
-F 0 "R14" H 5330 2654 50  0000 R CNN
+F 0 "R10" H 5330 2654 50  0000 R CNN
 F 1 "10K" H 5330 2745 50  0000 R CNN
 F 2 "Local:R_0603_1608Metric" V 5330 2700 50  0001 C CNN
@@
 AR Path="/5BBB311C/5BBB3512" Ref="R12"  Part="1"
 AR Path="/5BBB43B6/5BBB3512" Ref="R16"  Part="1"
-F 0 "R16" H 5920 2446 50  0000 L CNN
+F 0 "R12" H 5920 2446 50  0000 L CNN
 F 1 "10K" H 5920 2355 50  0000 L CNN
 F 2 "Local:R_0603_1608Metric" V 5780 2400 50  0001 C CNN
@@
 AR Path="/5BBB311C/5BBB3519" Ref="D1"  Part="1"
 AR Path="/5BBB43B6/5BBB3519" Ref="D3"  Part="1"
-F 0 "D3" V 5888 2632 50  0000 R CNN
+F 0 "D1" V 5888 2632 50  0000 R CNN
 F 1 "RED" V 5797 2632 50  0000 R CNN
 F 2 "Diode_SMD:D_0603_1608Metric" H 5850 2750 50  0001 C CNN
@@
 AR Path="/5BBB311C/5BBB3520" Ref="D2"  Part="1"
 AR Path="/5BBB43B6/5BBB3520" Ref="D4"  Part="1"
-F 0 "D4" V 6154 2729 50  0000 L CNN
+F 0 "D2" V 6154 2729 50  0000 L CNN
 F 1 "1N4148" V 6245 2729 50  0000 L CNN
 F 2 "Diode_SMD:D_SOD-323_HandSoldering" H 6200 2475 50  0001 C CNN
@@
 AR Path="/5BBB311C/5BBB3527" Ref="C11"  Part="1"
 AR Path="/5BBB43B6/5BBB3527" Ref="C12"  Part="1"
-F 0 "C12" H 5015 2596 50  0000 L CNN
+F 0 "C11" H 5015 2596 50  0000 L CNN
 F 1 "10uF 50V" H 5015 2505 50  0000 L CNN
 F 2 "Local:C_1206_3216Metric" H 4938 2400 50  0001 C CNN
@@
 AR Path="/5BBB311C/5BBB355D" Ref="R9"  Part="1"
 AR Path="/5BBB43B6/5BBB355D" Ref="R13"  Part="1"
-F 0 "R13" H 4570 3096 50  0000 L CNN
+F 0 "R9" H 4570 3096 50  0000 L CNN
 F 1 "10k" H 4570 3005 50  0000 L CNN
 F 2 "Local:R_0603_1608Metric" V 4430 3050 50  0001 C CNN
@@
 AR Path="/5BBB311C/5BBED217" Ref="J3"  Part="1"
 AR Path="/5BBB43B6/5BBED217" Ref="J4"  Part="1"
-F 0 "J4" H 7230 2892 50  0000 L CNN
+F 0 "J3" H 7230 2892 50  0000 L CNN
 F 1 "6A 50V" H 7230 2801 50  0000 L CNN
 F 2 "Local:TerminalBlock_Phoenix_PT-1,5-2-3.5-H_1x02_P3.50mm_Horizontal" H 7150 2900 50  0001 C CNN

Commit message: Added voltage selector for the fans.
Changed lines of the file:
@@
 AR Path="/5BBB311C/5BBB34F6" Ref="Q2"  Part="1"
 AR Path="/5BBB43B6/5BBB34F6" Ref="Q4"  Part="1"
-F 0 "Q2" H 5956 3196 50  0000 L CNN
+F 0 "Q4" H 5956 3196 50  0000 L CNN
 F 1 "PSMN7R0-30YL" H 5956 3105 50  0000 L CNN
 F 2 "Package_TO_SOT_SMD:LFPAK56" H 5900 3150 50  0001 C CNN
@@
 AR Path="/5BBB311C/5BBB34FD" Ref="Q1"  Part="1"
 AR Path="/5BBB43B6/5BBB34FD" Ref="Q3"  Part="1"
-F 0 "Q1" H 5237 3346 50  0000 L CNN
+F 0 "Q3" H 5237 3346 50  0000 L CNN
 F 1 "DTC124E" H 4750 3500 50  0000 L CNN
 F 2 "Package_TO_SOT_SMD:SOT-23" H 5050 3300 50  0001 L CNN
@@
 AR Path="/5BBB311C/5BBB3504" Ref="R11"  Part="1"
 AR Path="/5BBB43B6/5BBB3504" Ref="R15"  Part="1"
-F 0 "R11" H 5470 3396 50  0000 L CNN
+F 0 "R15" H 5470 3396 50  0000 L CNN
 F 1 "10K" H 5470 3305 50  0000 L CNN
 F 2 "Local:R_0603_1608Metric" V 5330 3350 50  0001 C CNN
@@
 AR Path="/5BBB311C/5BBB350B" Ref="R10"  Part="1"
 AR Path="/5BBB43B6/5BBB350B" Ref="R14"  Part="1"
-F 0 "R10" H 5330 2654 50  0000 R CNN
+F 0 "R14" H 5330 2654 50  0000 R CNN
 F 1 "10K" H 5330 2745 50  0000 R CNN
 F 2 "Local:R_0603_1608Metric" V 5330 2700 50  0001 C CNN
@@
 AR Path="/5BBB311C/5BBB3512" Ref="R12"  Part="1"
 AR Path="/5BBB43B6/5BBB3512" Ref="R16"  Part="1"
-F 0 "R12" H 5920 2446 50  0000 L CNN
+F 0 "R16" H 5920 2446 50  0000 L CNN
 F 1 "10K" H 5920 2355 50  0000 L CNN
 F 2 "Local:R_0603_1608Metric" V 5780 2400 50  0001 C CNN
@@
 AR Path="/5BBB311C/5BBB3519" Ref="D1"  Part="1"
 AR Path="/5BBB43B6/5BBB3519" Ref="D3"  Part="1"
-F 0 "D1" V 5888 2632 50  0000 R CNN
+F 0 "D3" V 5888 2632 50  0000 R CNN
 F 1 "RED" V 5797 2632 50  0000 R CNN
 F 2 "Diode_SMD:D_0603_1608Metric" H 5850 2750 50  0001 C CNN
@@
 AR Path="/5BBB311C/5BBB3520" Ref="D2"  Part="1"
 AR Path="/5BBB43B6/5BBB3520" Ref="D4"  Part="1"
-F 0 "D2" V 6154 2729 50  0000 L CNN
+F 0 "D4" V 6154 2729 50  0000 L CNN
 F 1 "1N4148" V 6245 2729 50  0000 L CNN
 F 2 "Diode_SMD:D_SOD-323_HandSoldering" H 6200 2475 50  0001 C CNN
@@
 AR Path="/5BBB311C/5BBB3527" Ref="C11"  Part="1"
 AR Path="/5BBB43B6/5BBB3527" Ref="C12"  Part="1"
-F 0 "C11" H 5015 2596 50  0000 L CNN
+F 0 "C12" H 5015 2596 50  0000 L CNN
 F 1 "10uF 50V" H 5015 2505 50  0000 L CNN
 F 2 "Local:C_1206_3216Metric" H 4938 2400 50  0001 C CNN
@@
 AR Path="/5BBB311C/5BBB355D" Ref="R9"  Part="1"
 AR Path="/5BBB43B6/5BBB355D" Ref="R13"  Part="1"
-F 0 "R9" H 4570 3096 50  0000 L CNN
+F 0 "R13" H 4570 3096 50  0000 L CNN
 F 1 "10k" H 4570 3005 50  0000 L CNN
 F 2 "Local:R_0603_1608Metric" V 4430 3050 50  0001 C CNN
@@
 AR Path="/5BBB311C/5BBED217" Ref="J3"  Part="1"
 AR Path="/5BBB43B6/5BBED217" Ref="J4"  Part="1"
-F 0 "J3" H 7230 2892 50  0000 L CNN
+F 0 "J4" H 7230 2892 50  0000 L CNN
 F 1 "6A 50V" H 7230 2801 50  0000 L CNN
 F 2 "Local:TerminalBlock_Phoenix_PT-1,5-2-3.5-H_1x02_P3.50mm_Horizontal" H 7150 2900 50  0001 C CNN
